File: hp_breakout/hp_breakout.kicad_pcb (KiCad board)
At the start: 2 copper layers, 21 x 35.6 mm, 20 parts, among them J1 AudioJack2_Ground_Switch, J10 Conn_01x05_Male, J11 AudioJack2_Ground_Switch, J12 AudioJack2_Ground_Switch, J13 AudioJack2_Ground_Switch, J14 AudioJack2_Ground_Switch, J15 AudioJack2_Ground_Switch, J16 Conn_01x05_Male, J17 Conn_01x05_Male, J18 Conn_01x05_Male, J19 Conn_01x05_Male, J2 Conn_01x05_Male, J20 Conn_01x05_Male, J3 AudioJack2_Ground_Switch, J4 AudioJack2_Ground_Switch, J5 AudioJack2_Ground_Switch, J6 AudioJack2_Ground_Switch, J7 Conn_01x05_Male, J8 Conn_01x05_Male, J9 Conn_01x05_Male

Commit message: 10 identical boards
Parts:
- J1, J11, J13, J15, J3, J5: footprint KiCad/kicad-footprints/Connector_Audio.pretty:Jack_3.5mm_Ledino_KB3SPRS_Horizontal -> hp_breakout:Jack_3.5mm_Ledino_KB3SPRS_Horizontal
- J12, J14, J4, J6: value AudioJack2_Ground_Switch -> Conn_01x05_Male; footprint KiCad/kicad-footprints/Connector_Audio.pretty:Jack_3.5mm_Ledino_KB3SPRS_Horizontal -> KiCad/kicad-footprints/Connector_PinHeader_2.54mm.pretty:PinHeader_1x05_P2.54mm_Vertical
- J17, J19, J7, J9: value Conn_01x05_Male -> AudioJack2_Ground_Switch; footprint KiCad/kicad-footprints/Connector_PinHeader_2.54mm.pretty:PinHeader_1x05_P2.54mm_Vertical -> hp_breakout:Jack_3.5mm_Ledino_KB3SPRS_Horizontal
- moved J17 137.8 mm to (48.6, 91.8)
- moved J20 123.9 mm to (61.0, 48.9)
- moved J16 122.8 mm to (67.3, 108.6), turned to 180 degrees
- moved J19 121.1 mm to (48.6, 58.8)
- moved J15 112.5 mm to (79.6, 98.7), turned to 180 degrees
- moved J5 109.9 mm to (48.6, 108.3)
- moved J8 106.5 mm to (67.3, 75.6), turned to 180 degrees
- moved J18 105.3 mm to (61.0, 81.9)
- moved J12 99.9 mm to (61.0, 65.4)
- moved J10 96.7 mm to (67.3, 92.1), turned to 180 degrees
- moved J14 93.3 mm to (67.3, 42.5), turned to 180 degrees
- moved J11 91.6 mm to (48.6, 75.3)
- moved J9 77.8 mm to (79.6, 82.2), turned to 180 degrees
- moved J13 72.8 mm to (79.6, 32.6), turned to 180 degrees
- moved J7 71.3 mm to (79.6, 65.7), turned to 180 degrees
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Connections:
- J1 pad R: Net-(J1-PadR) -> /U?/R
- J1 pad RN: Net-(J1-PadRN) -> /U?/RN
- J1 pad S: Net-(J1-PadS) -> /U?/S
- J1 pad T: Net-(J1-PadT) -> /U?/T
- J1 pad TN: Net-(J1-PadTN) -> /U?/TN
- J10 pad 1: Net-(J10-Pad1) -> /sheet5E6F47F3/S
- J10 pad 2: Net-(J10-Pad2) -> /sheet5E6F47F3/R
- J10 pad 3: Net-(J10-Pad3) -> /sheet5E6F47F3/RN
- J10 pad 4: Net-(J10-Pad4) -> /sheet5E6F47F3/T
- J10 pad 5: Net-(J10-Pad5) -> /sheet5E6F47F3/TN
- J11 pad R: Net-(J11-PadR) -> /sheet5E6F4A68/R
- J11 pad RN: Net-(J11-PadRN) -> /sheet5E6F4A68/RN
- J11 pad S: Net-(J11-PadS) -> /sheet5E6F4A68/S
- J11 pad T: Net-(J11-PadT) -> /sheet5E6F4A68/T
- J11 pad TN: Net-(J11-PadTN) -> /sheet5E6F4A68/TN
- J13 pad R: Net-(J13-PadR) -> /sheet5E6F4A6A/R
- J13 pad RN: Net-(J13-PadRN) -> /sheet5E6F4A6A/RN
- J13 pad S: Net-(J13-PadS) -> /sheet5E6F4A6A/S
- J13 pad T: Net-(J13-PadT) -> /sheet5E6F4A6A/T
- J13 pad TN: Net-(J13-PadTN) -> /sheet5E6F4A6A/TN
- J15 pad R: Net-(J15-PadR) -> /sheet5E6F4A6C/R
- J15 pad RN: Net-(J15-PadRN) -> /sheet5E6F4A6C/RN
- J15 pad S: Net-(J15-PadS) -> /sheet5E6F4A6C/S
- J15 pad T: Net-(J15-PadT) -> /sheet5E6F4A6C/T
- J15 pad TN: Net-(J15-PadTN) -> /sheet5E6F4A6C/TN
- J16 pad 1: Net-(J11-PadR) -> /sheet5E6F4A6C/S
- J16 pad 2: Net-(J11-PadTN) -> /sheet5E6F4A6C/R
- J16 pad 3: Net-(J11-PadT) -> /sheet5E6F4A6C/RN
- J16 pad 4: Net-(J11-PadS) -> /sheet5E6F4A6C/T
- J16 pad 5: Net-(J11-PadRN) -> /sheet5E6F4A6C/TN
- J18 pad 1: Net-(J13-PadR) -> /sheet5E6F4A6E/S
- J18 pad 2: Net-(J13-PadTN) -> /sheet5E6F4A6E/R
- J18 pad 3: Net-(J13-PadT) -> /sheet5E6F4A6E/RN
- J18 pad 4: Net-(J13-PadS) -> /sheet5E6F4A6E/T
- J18 pad 5: Net-(J13-PadRN) -> /sheet5E6F4A6E/TN
- J2 pad 1: Net-(J1-PadR) -> /U?/S
- J2 pad 2: Net-(J1-PadTN) -> /U?/R
- J2 pad 3: Net-(J1-PadT) -> /U?/RN
- J2 pad 4: Net-(J1-PadS) -> /U?/T
- J2 pad 5: Net-(J1-PadRN) -> /U?/TN
- J20 pad 1: Net-(J15-PadR) -> /sheet5E6F4A70/S
- J20 pad 2: Net-(J15-PadTN) -> /sheet5E6F4A70/R
- J20 pad 3: Net-(J15-PadT) -> /sheet5E6F4A70/RN
- J20 pad 4: Net-(J15-PadS) -> /sheet5E6F4A70/T
- J20 pad 5: Net-(J15-PadRN) -> /sheet5E6F4A70/TN
- J3 pad R: Net-(J3-PadR) -> /sheet5E6F4684/R
- J3 pad RN: Net-(J3-PadRN) -> /sheet5E6F4684/RN
- J3 pad S: Net-(J3-PadS) -> /sheet5E6F4684/S
- J3 pad T: Net-(J3-PadT) -> /sheet5E6F4684/T
- J3 pad TN: Net-(J3-PadTN) -> /sheet5E6F4684/TN
- J5 pad R: Net-(J5-PadR) -> /sheet5E6F46C9/R
- J5 pad RN: Net-(J5-PadRN) -> /sheet5E6F46C9/RN
- J5 pad S: Net-(J5-PadS) -> /sheet5E6F46C9/S
- J5 pad T: Net-(J5-PadT) -> /sheet5E6F46C9/T
- J5 pad TN: Net-(J5-PadTN) -> /sheet5E6F46C9/TN
- J8 pad 1: Net-(J4-PadR) -> /sheet5E6F46CB/S
- J8 pad 2: Net-(J4-PadTN) -> /sheet5E6F46CB/R
- J8 pad 3: Net-(J4-PadT) -> /sheet5E6F46CB/RN
- J8 pad 4: Net-(J4-PadS) -> /sheet5E6F46CB/T
- J8 pad 5: Net-(J4-PadRN) -> /sheet5E6F46CB/TN
Routing:
- net Net-(J1-PadR): track 18.2 -> 0.00 mm, vias 1 -> 0
- net Net-(J1-PadS): track 17.0 -> 0.00 mm
- net Net-(J1-PadT): track 15.3 -> 0.00 mm
- net /sheet5E6F4A68/T: track 0.00 -> 15.2 mm
- net /sheet5E6F4A70/T: track 0.00 -> 15.2 mm
- net /sheet5E6F46CB/T: track 0.00 -> 15.2 mm
- net /U?/T: track 0.00 -> 15.2 mm
- net /sheet5E6F4A6E/T: track 0.00 -> 15.2 mm
- net /sheet5E6F4A6A/T: track 0.00 -> 15.2 mm
- net /sheet5E6F4A6C/T: track 0.00 -> 15.2 mm
- net /sheet5E6F4684/T: track 0.00 -> 15.2 mm
- net /sheet5E6F46C9/T: track 0.00 -> 15.2 mm
- net /sheet5E6F47F3/T: track 0.00 -> 15.2 mm
- net /sheet5E6F4A6E/RN: track 0.00 -> 10.4 mm
- net /sheet5E6F4A6C/RN: track 0.00 -> 10.4 mm
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- added copper zone on B.Cu, net /U?/S
- added copper zone on B.Cu, net /sheet5E6F4684/S
- added copper zone on B.Cu, net /sheet5E6F46C9/S
- added copper zone on B.Cu, net /sheet5E6F46CB/S
- added copper zone on B.Cu, net /sheet5E6F47F3/S
- added copper zone on B.Cu, net /sheet5E6F4A68/S
- added copper zone on B.Cu, net /sheet5E6F4A6A/S
- added copper zone on B.Cu, net /sheet5E6F4A6C/S
- added copper zone on B.Cu, net /sheet5E6F4A6E/S
- added copper zone on B.Cu, net /sheet5E6F4A70/S
Other:
- board size 21 x 35.6 mm -> 43.2 x 80 mm
- board text added: "R"
- board text added: "RN"
- board text added: "S"
- board text added: "T"
- board text added: "TN"
