File: amp/BVCA.sch (KiCad schematic (older format))
At the start: 19 parts

Commit message: reworked amp sheets and notes
Parts:
- C3: renamed from C?; footprint (none) -> KiCad/Capacitors_ThroughHole.pretty:CP_Radial_D4.0mm_P1.50mm
- C4: renamed from C?; footprint (none) -> KiCad/Capacitors_ThroughHole.pretty:CP_Radial_D6.3mm_P2.50mm
- R14, R15, R16, R17, R18, R19, R20, R21, R22: renamed from R?; footprint (none) -> KiCad/Resistors_ThroughHole.pretty:R_Axial_DIN0204_L3.6mm_D1.6mm_P1.90mm_Vertical
- U2: renamed from U?; footprint (none) -> KiCad/Housings_DIP.pretty:DIP-14_W7.62mm
- U3: renamed from U?; footprint (none) -> KiCad/Housings_DIP.pretty:DIP-16_W7.62mm
- gave numbers to parts that had none: 2
