File: amp/OutputStage.sch (KiCad schematic (older format))
At the start: 36 parts, among them J11 EXT_IN, J12 A_OUT, J13 C_OUT, J14 B_OUT, J15 D_OUT, J16 MAIN_OUT, J17 HP_OUT, SW1 SW_STEREO_SPLIT, U2 LM13700, U3 LM13700, U4 TL072

Commit message: output stage
Parts:
- R1, R2, R3, R4, R5, R6, R7, R8: value 200K -> 560K
- R10, R11, R12, R9: value 200K -> 33K
- R13, R14, R15, R16: value 10K -> 22K
Changed lines of the file:
@@
 AR Path="/5EC4DE09/5EC57D25" Ref="R13"  Part="1"
 F 0 "R13" V 7330 2500 50  0000 C CNN
-F 1 "10K" V 7250 2500 50  0000 C CNN
+F 1 "22K" V 7250 2500 50  0000 C CNN
 F 2 "Resistor_THT:R_Axial_DIN0204_L3.6mm_D1.6mm_P1.90mm_Vertical" V 7180 2500 50  0001 C CNN
 F 3 "" H 7250 2500 50  0001 C CNN
@@
 AR Path="/5EC4DE09/5EC58906" Ref="R14"  Part="1"
 F 0 "R14" V 7330 4600 50  0000 C CNN
-F 1 "10K" V 7250 4600 50  0000 C CNN
+F 1 "22K" V 7250 4600 50  0000 C CNN
 F 2 "Resistor_THT:R_Axial_DIN0204_L3.6mm_D1.6mm_P1.90mm_Vertical" V 7180 4600 50  0001 C CNN
 F 3 "" H 7250 4600 50  0001 C CNN
@@
 AR Path="/5EC4DE09/5EC883DC" Ref="R11"  Part="1"
 F 0 "R11" V 4980 2700 50  0000 C CNN
-F 1 "200K" V 4900 2700 50  0000 C CNN
+F 1 "33K" V 4900 2700 50  0000 C CNN
 F 2 "Resistor_THT:R_Axial_DIN0204_L3.6mm_D1.6mm_P1.90mm_Vertical" V 4830 2700 50  0001 C CNN
 F 3 "" H 4900 2700 50  0001 C CNN
@@
 AR Path="/5EC4DE09/5ED4DDF5" Ref="R12"  Part="1"
 F 0 "R12" V 4980 4100 50  0000 C CNN
-F 1 "200K" V 4900 4100 50  0000 C CNN
+F 1 "33K" V 4900 4100 50  0000 C CNN
 F 2 "Resistor_THT:R_Axial_DIN0204_L3.6mm_D1.6mm_P1.90mm_Vertical" V 4830 4100 50  0001 C CNN
 F 3 "" H 4900 4100 50  0001 C CNN
@@
 AR Path="/5EC4DE09/5ED391E4" Ref="R3"  Part="1"
 F 0 "R3" V 1680 3250 50  0000 C CNN
-F 1 "200K" V 1600 3250 50  0000 C CNN
+F 1 "560K" V 1600 3250 50  0000 C CNN
 F 2 "Resistor_THT:R_Axial_DIN0204_L3.6mm_D1.6mm_P1.90mm_Vertical" V 1530 3250 50  0001 C CNN
 F 3 "" H 1600 3250 50  0001 C CNN
@@
 AR Path="/5EC4DE09/5EC99131" Ref="R1"  Part="1"
 F 0 "R1" V 1680 2600 50  0000 C CNN
-F 1 "200K" V 1600 2600 50  0000 C CNN
+F 1 "560K" V 1600 2600 50  0000 C CNN
 F 2 "Resistor_THT:R_Axial_DIN0204_L3.6mm_D1.6mm_P1.90mm_Vertical" V 1530 2600 50  0001 C CNN
 F 3 "" H 1600 2600 50  0001 C CNN
@@
 AR Path="/5EC4DE09/5EEC4F01" Ref="R2"  Part="1"
 F 0 "R2" V 1680 2950 50  0000 C CNN
-F 1 "200K" V 1600 2950 50  0000 C CNN
+F 1 "560K" V 1600 2950 50  0000 C CNN
 F 2 "Resistor_THT:R_Axial_DIN0204_L3.6mm_D1.6mm_P1.90mm_Vertical" V 1530 2950 50  0001 C CNN
 F 3 "" H 1600 2950 50  0001 C CNN
@@
 AR Path="/5EC4DE09/5EECE800" Ref="R4"  Part="1"
 F 0 "R4" V 1680 3600 50  0000 C CNN
-F 1 "200K" V 1600 3600 50  0000 C CNN
+F 1 "560K" V 1600 3600 50  0000 C CNN
 F 2 "Resistor_THT:R_Axial_DIN0204_L3.6mm_D1.6mm_P1.90mm_Vertical" V 1530 3600 50  0001 C CNN
 F 3 "" H 1600 3600 50  0001 C CNN
@@
 AR Path="/5EC4DE09/5EF0B67F" Ref="R7"  Part="1"
 F 0 "R7" V 1680 4550 50  0000 C CNN
-F 1 "200K" V 1600 4550 50  0000 C CNN
+F 1 "560K" V 1600 4550 50  0000 C CNN
 F 2 "Resistor_THT:R_Axial_DIN0204_L3.6mm_D1.6mm_P1.90mm_Vertical" V 1530 4550 50  0001 C CNN
 F 3 "" H 1600 4550 50  0001 C CNN
@@
 AR Path="/5EC4DE09/5EF0B689" Ref="R5"  Part="1"
 F 0 "R5" V 1680 3900 50  0000 C CNN
-F 1 "200K" V 1600 3900 50  0000 C CNN
+F 1 "560K" V 1600 3900 50  0000 C CNN
 F 2 "Resistor_THT:R_Axial_DIN0204_L3.6mm_D1.6mm_P1.90mm_Vertical" V 1530 3900 50  0001 C CNN
 F 3 "" H 1600 3900 50  0001 C CNN
@@
 AR Path="/5EC4DE09/5EF0B695" Ref="R6"  Part="1"
 F 0 "R6" V 1680 4250 50  0000 C CNN
-F 1 "200K" V 1600 4250 50  0000 C CNN
+F 1 "560K" V 1600 4250 50  0000 C CNN
 F 2 "Resistor_THT:R_Axial_DIN0204_L3.6mm_D1.6mm_P1.90mm_Vertical" V 1530 4250 50  0001 C CNN
 F 3 "" H 1600 4250 50  0001 C CNN
@@
 AR Path="/5EC4DE09/5EF0B6AD" Ref="R8"  Part="1"
 F 0 "R8" V 1680 4900 50  0000 C CNN
-F 1 "200K" V 1600 4900 50  0000 C CNN
+F 1 "560K" V 1600 4900 50  0000 C CNN
 F 2 "Resistor_THT:R_Axial_DIN0204_L3.6mm_D1.6mm_P1.90mm_Vertical" V 1530 4900 50  0001 C CNN
 F 3 "" H 1600 4900 50  0001 C CNN
@@
 AR Path="/5EC4DE09/5EDC9971" Ref="R16"  Part="1"
 F 0 "R16" V 7380 3450 50  0000 C CNN
-F 1 "10K" V 7300 3450 50  0000 C CNN
+F 1 "22K" V 7300 3450 50  0000 C CNN
 F 2 "Resistor_THT:R_Axial_DIN0204_L3.6mm_D1.6mm_P1.90mm_Vertical" V 7230 3450 50  0001 C CNN
 F 3 "" H 7300 3450 50  0001 C CNN
@@
 AR Path="/5EC4DE09/5EDC99A0" Ref="R15"  Part="1"
 F 0 "R15" V 7330 5400 50  0000 C CNN
-F 1 "10K" V 7250 5400 50  0000 C CNN
+F 1 "22K" V 7250 5400 50  0000 C CNN
 F 2 "Resistor_THT:R_Axial_DIN0204_L3.6mm_D1.6mm_P1.90mm_Vertical" V 7180 5400 50  0001 C CNN
 F 3 "" H 7250 5400 50  0001 C CNN
@@
 AR Path="/5EC4DE09/5EF34DA4" Ref="R9"  Part="1"
 F 0 "R9" V 1780 6150 50  0000 C CNN
-F 1 "200K" V 1700 6150 50  0000 C CNN
+F 1 "33K" V 1700 6150 50  0000 C CNN
 F 2 "Resistor_THT:R_Axial_DIN0204_L3.6mm_D1.6mm_P1.90mm_Vertical" V 1630 6150 50  0001 C CNN
 F 3 "" H 1700 6150 50  0001 C CNN
@@
 AR Path="/5EC4DE09/5EF35A70" Ref="R10"  Part="1"
 F 0 "R10" V 1780 6350 50  0000 C CNN
-F 1 "200K" V 1700 6350 50  0000 C CNN
+F 1 "33K" V 1700 6350 50  0000 C CNN
 F 2 "Resistor_THT:R_Axial_DIN0204_L3.6mm_D1.6mm_P1.90mm_Vertical" V 1630 6350 50  0001 C CNN
 F 3 "" H 1700 6350 50  0001 C CNN
