File: utils/utils.sch (KiCad schematic (older format))
At the start: 30 parts

Commit message: fix for eurorack connector
Parts:
- J1, J2, J4, J5, J6, J7, J9: renamed from J?; footprint (none) -> synth:3.5MM_Jack_Breakout_Vertical
- J10: renamed from J?; value 1_OUT -> 2_OUT; footprint (none) -> synth:3.5MM_Jack_Breakout_Vertical
- J11: renamed from J?; footprint KiCad/kicad-footprints/Connector_IDC.pretty:IDC-Header_2x08_P2.54mm_Vertical -> synth:EURORACK_16_IDC
- J3: renamed from J?; value 2_GATE -> 1_GATE; footprint (none) -> synth:3.5MM_Jack_Breakout_Vertical
- J8: renamed from J?; value 1_~OUT -> 2_~OUT; footprint (none) -> synth:3.5MM_Jack_Breakout_Vertical
- Q1, Q2: renamed from Q?; footprint Package_TO_SOT_THT:TO-92_Inline -> KiCad/TO_SOT_Packages_THT.pretty:TO-92_Molded_Narrow
- R1, R10, R2, R3, R4, R5, R6, R7, R8, R9: renamed from R?; footprint (none) -> 4ms/4ms-kicad-lib/4ms-footprints.pretty:Resistor_TH_300
- RV1, RV2: renamed from RV?; footprint (none) -> KiCad/Potentiometers.pretty:Potentiometer_Trimmer_Vishay_T73YP_Horizontal
- U1: renamed from U?; footprint (none) -> 4ms/4ms-kicad-lib/lib-footprints/4ms_Package_DIP.pretty:DIP-14_W7.62mm
Connections:
- wire segments 180 -> 192
Other:
- moved on the sheet: J11

Commit message: use jacks directly for horizontal
Parts:
- J1, J10, J2, J3, J4, J5, J6, J7, J8, J9: footprint synth:3.5MM_Jack_Breakout_Vertical -> synth:Jack_3.5mm_Ledino_KB3SPRS_Horizontal
- Q1, Q2: footprint KiCad/TO_SOT_Packages_THT.pretty:TO-92_Molded_Narrow -> KiCad/TO_SOT_Packages_THT.pretty:TO-92_Inline_Wide
- RV1, RV2: footprint KiCad/Potentiometers.pretty:Potentiometer_Trimmer_Vishay_T73YP_Horizontal -> rdeterre/misc.pretty:Potentiometer_Bourns_PDB182-K_Dual
Changed lines of the file:
@@
 F 0 "RV1" V 3143 2000 50  0000 C CNN
 F 1 "200K" V 3234 2000 50  0000 C CNN
-F 2 "KiCad/Potentiometers.pretty:Potentiometer_Trimmer_Vishay_T73YP_Horizontal" H 3350 2000 50  0001 C CNN
+F 2 "rdeterre/misc.pretty:Potentiometer_Bourns_PDB182-K_Dual" H 3350 2000 50  0001 C CNN
 F 3 "~" H 3350 2000 50  0001 C CNN
 	1    3350 2000
@@
 F 0 "Q1" V 3449 1350 50  0000 C CNN
 F 1 "2N7000" V 3540 1350 50  0000 C CNN
-F 2 "KiCad/TO_SOT_Packages_THT.pretty:TO-92_Molded_Narrow" H 3400 1275 50  0001 L CIN
+F 2 "KiCad/TO_SOT_Packages_THT.pretty:TO-92_Inline_Wide" H 3400 1275 50  0001 L CIN
 F 3 "https://www.fairchildsemi.com/datasheets/2N/2N7000.pdf" H 3200 1350 50  0001 L CNN
 	1    3200 1350
@@
 F 0 "J1" H 832 1425 50  0000 C CNN
 F 1 "1_AIN" H 832 1334 50  0000 C CNN
-F 2 "synth:3.5MM_Jack_Breakout_Vertical" H 800 1200 50  0001 C CNN
+F 2 "synth:Jack_3.5mm_Ledino_KB3SPRS_Horizontal" H 800 1200 50  0001 C CNN
 F 3 "~" H 800 1200 50  0001 C CNN
 	1    800  1000
@@
 F 0 "J2" H 832 2575 50  0000 C CNN
 F 1 "1_BIN" H 832 2484 50  0000 C CNN
-F 2 "synth:3.5MM_Jack_Breakout_Vertical" H 800 2350 50  0001 C CNN
+F 2 "synth:Jack_3.5mm_Ledino_KB3SPRS_Horizontal" H 800 2350 50  0001 C CNN
 F 3 "~" H 800 2350 50  0001 C CNN
 	1    800  2150
@@
 F 0 "J3" H 832 3675 50  0000 C CNN
 F 1 "1_GATE" H 832 3584 50  0000 C CNN
-F 2 "synth:3.5MM_Jack_Breakout_Vertical" H 800 3450 50  0001 C CNN
+F 2 "synth:Jack_3.5mm_Ledino_KB3SPRS_Horizontal" H 800 3450 50  0001 C CNN
 F 3 "~" H 800 3450 50  0001 C CNN
 	1    800  3250
@@
 F 0 "J7" H 6020 1074 50  0000 R CNN
 F 1 "1_~OUT" H 6020 976 50  0000 R CNN
-F 2 "synth:3.5MM_Jack_Breakout_Vertical" H 6200 1250 50  0001 C CNN
+F 2 "synth:Jack_3.5mm_Ledino_KB3SPRS_Horizontal" H 6200 1250 50  0001 C CNN
 F 3 "~" H 6200 1250 50  0001 C CNN
 	1    6200 1050
@@
 F 0 "J9" H 6070 2168 50  0000 R CNN
 F 1 "1_OUT" H 6070 2077 50  0000 R CNN
-F 2 "synth:3.5MM_Jack_Breakout_Vertical" H 6250 2350 50  0001 C CNN
+F 2 "synth:Jack_3.5mm_Ledino_KB3SPRS_Horizontal" H 6250 2350 50  0001 C CNN
 F 3 "~" H 6250 2350 50  0001 C CNN
 	1    6250 2150
@@
 F 0 "RV2" V 3143 5650 50  0000 C CNN
 F 1 "200K" V 3234 5650 50  0000 C CNN
-F 2 "KiCad/Potentiometers.pretty:Potentiometer_Trimmer_Vishay_T73YP_Horizontal" H 3350 5650 50  0001 C CNN
+F 2 "rdeterre/misc.pretty:Potentiometer_Bourns_PDB182-K_Dual" H 3350 5650 50  0001 C CNN
 F 3 "~" H 3350 5650 50  0001 C CNN
 	1    3350 5650
@@
 F 0 "Q2" V 3449 5000 50  0000 C CNN
 F 1 "2N7000" V 3540 5000 50  0000 C CNN
-F 2 "KiCad/TO_SOT_Packages_THT.pretty:TO-92_Molded_Narrow" H 3400 4925 50  0001 L CIN
+F 2 "KiCad/TO_SOT_Packages_THT.pretty:TO-92_Inline_Wide" H 3400 4925 50  0001 L CIN
 F 3 "https://www.fairchildsemi.com/datasheets/2N/2N7000.pdf" H 3200 5000 50  0001 L CNN
 	1    3200 5000
@@
 F 0 "J4" H 832 5075 50  0000 C CNN
 F 1 "2_AIN" H 832 4984 50  0000 C CNN
-F 2 "synth:3.5MM_Jack_Breakout_Vertical" H 800 4850 50  0001 C CNN
+F 2 "synth:Jack_3.5mm_Ledino_KB3SPRS_Horizontal" H 800 4850 50  0001 C CNN
 F 3 "~" H 800 4850 50  0001 C CNN
 	1    800  4650
@@
 F 0 "J5" H 832 6225 50  0000 C CNN
 F 1 "2_BIN" H 832 6134 50  0000 C CNN
-F 2 "synth:3.5MM_Jack_Breakout_Vertical" H 800 6000 50  0001 C CNN
+F 2 "synth:Jack_3.5mm_Ledino_KB3SPRS_Horizontal" H 800 6000 50  0001 C CNN
 F 3 "~" H 800 6000 50  0001 C CNN
 	1    800  5800
@@
 F 0 "J6" H 832 7325 50  0000 C CNN
 F 1 "2_GATE" H 832 7234 50  0000 C CNN
-F 2 "synth:3.5MM_Jack_Breakout_Vertical" H 800 7100 50  0001 C CNN
+F 2 "synth:Jack_3.5mm_Ledino_KB3SPRS_Horizontal" H 800 7100 50  0001 C CNN
 F 3 "~" H 800 7100 50  0001 C CNN
 	1    800  6900
@@
 F 0 "J8" H 6020 4724 50  0000 R CNN
 F 1 "2_~OUT" H 6020 4626 50  0000 R CNN
-F 2 "synth:3.5MM_Jack_Breakout_Vertical" H 6200 4900 50  0001 C CNN
+F 2 "synth:Jack_3.5mm_Ledino_KB3SPRS_Horizontal" H 6200 4900 50  0001 C CNN
 F 3 "~" H 6200 4900 50  0001 C CNN
 	1    6200 4700
@@
 F 0 "J10" H 6070 5818 50  0000 R CNN
 F 1 "2_OUT" H 6070 5727 50  0000 R CNN
-F 2 "synth:3.5MM_Jack_Breakout_Vertical" H 6250 6000 50  0001 C CNN
+F 2 "synth:Jack_3.5mm_Ledino_KB3SPRS_Horizontal" H 6250 6000 50  0001 C CNN
 F 3 "~" H 6250 6000 50  0001 C CNN
 	1    6250 5800

Commit message: switched fet with cd4066
Parts:
- removed J10: 2_OUT, synth:Jack_3.5mm_Ledino_KB3SPRS_Horizontal, symbol Connector:AudioJack2_Ground_Switch
- removed J4: 2_AIN, synth:Jack_3.5mm_Ledino_KB3SPRS_Horizontal, symbol Connector:AudioJack2_Ground_Switch
- removed J5: 2_BIN, synth:Jack_3.5mm_Ledino_KB3SPRS_Horizontal, symbol Connector:AudioJack2_Ground_Switch
- removed J6: 2_GATE, synth:Jack_3.5mm_Ledino_KB3SPRS_Horizontal, symbol Connector:AudioJack2_Ground_Switch
- removed J8: 2_~OUT, synth:Jack_3.5mm_Ledino_KB3SPRS_Horizontal, symbol Connector:AudioJack2_Ground_Switch
- removed Q1, Q2: 2N7000, KiCad/TO_SOT_Packages_THT.pretty:TO-92_Inline_Wide, symbol Transistor_FET:2N7000
- removed R1, R10, R2, R4: 100K, 4ms/4ms-kicad-lib/4ms-footprints.pretty:Resistor_TH_300, symbol Device:R
- removed RV1, RV2: 200K, rdeterre/misc.pretty:Potentiometer_Bourns_PDB182-K_Dual, symbol Device:R_POT
- removed U1: TL074, 4ms/4ms-kicad-lib/lib-footprints/4ms_Package_DIP.pretty:DIP-14_W7.62mm, symbol Amplifier_Operational:TL074
- added R3: 100K, 4ms/4ms-kicad-lib/4ms-footprints.pretty:Resistor_TH_300, symbol Device:R
- added R7: 1K5, 4ms/4ms-kicad-lib/4ms-footprints.pretty:Resistor_TH_300, symbol Device:R
- added R9: 220, 4ms/4ms-kicad-lib/4ms-footprints.pretty:Resistor_TH_300, symbol Device:R
- added RV1: 100K, rdeterre/misc.pretty:Potentiometer_Bourns_PDB182-K_Dual, symbol Device:R_POT_Dual
- added U1: TL072, KiCad/kicad-footprints/Package_DIP.pretty:DIP-8_W7.62mm, symbol Amplifier_Operational:TL072
- added U2: 4066, KiCad/kicad-footprints/Package_DIP.pretty:DIP-14_W7.62mm, symbol 4xxx:4066
- added U3: LM317L_TO92, KiCad/TO_SOT_Packages_THT.pretty:TO-220-3_Vertical, symbol Regulator_Linear:LM317L_TO92
- added U4: LM337L_TO92, KiCad/TO_SOT_Packages_THT.pretty:TO-220-3_Vertical, symbol Regulator_Linear:LM337L_TO92
- J1: value 1_AIN -> AIN; symbol Connector:AudioJack2_Ground_Switch -> synth:AudioJack2_Ground_Switch
- J2: value 1_BIN -> BIN; symbol Connector:AudioJack2_Ground_Switch -> synth:AudioJack2_Ground_Switch
- J3: value 1_GATE -> GATE; symbol Connector:AudioJack2_Ground_Switch -> synth:AudioJack2_Ground_Switch
- J5: renamed from J7; value 1_~OUT -> ~OUT; symbol Connector:AudioJack2_Ground_Switch -> synth:AudioJack2_Ground_Switch
- J6: renamed from J9; value 1_OUT -> OUT; symbol Connector:AudioJack2_Ground_Switch -> synth:AudioJack2_Ground_Switch
- R6: value 100K -> 220
- R8: value 100K -> 1K5
- renumbered J11 to J4, R3 to R1, R5 to R2, R7 to R4, R9 to R5
Connections:
- net labels added: AIN, BIN, GATE, OUT, ~OUT
- net labels removed: 1_AIN, 1_BIN, 1_GATE, 1_OUT, 1_~OUT, 2_AIN, 2_BIN, 2_GATE, 2_OUT, 2_~OUT
- wire segments 192 -> 123
Other:
- note added: "Considered an LED here, but most require 20mA\nwhich is a serious bite out of the power supply"
- note added: "I was originally targeting a 200K pot. However,\nThe only 1 Detent PDB18X available was a 100K\n2 gang pot, so instead we use both gangs in series\nand can keep the input impedance at 100K and still\nget a gain of 0-2"
- note added: "In order to share the switches of a single CD4066\nacross multiple boards, there are some hacks in the\nPCB design. The CD4066 and the LM*37s are only\nrequired on one board"
- note added: "The CD4066 has a max power supply voltage of 20V,\nso we step the 24V down to about 19.5 via regulators.\nIn theory we could hacky do this with 6 diodes instead"
- note removed: "FET on shorts Rf for a gain of 0"
- note removed: "gain 0-2"
- moved on the sheet: J4, R1, R2, R4, R5

Commit message: pcb mostly laid out
Parts:
- added J7: Conn_01x04, imciner2/KiCad-Libraries/modules/Connectors.pretty:CONN_2.54mm_1x04, symbol Connector_Generic:Conn_01x04
- added J8: Conn_01x05, imciner2/KiCad-Libraries/modules/Connectors.pretty:CONN_2.54mm_1x05, symbol Connector_Generic:Conn_01x05
- added unit 2 of U2
- added unit 3 of U2
- added unit 4 of U2
Connections:
- net labels added: 4066_10, 4066_11, 4066_12, 4066_3, 4066_4, 4066_5, 4066_6, 4066_8, 4066_9
- wire segments 123 -> 147
Changed lines of the file:
@@
 Text Notes 9050 3200 0    50   ~ 0
 The CD4066 has a max power supply voltage of 20V,\nso we step the 24V down to about 19.5 via regulators.\nIn theory we could hacky do this with 6 diodes instead
-Text Notes 4450 7450 0    50   ~ 0
+Text Notes 1150 7500 0    50   ~ 0
 In order to share the switches of a single CD4066\nacross multiple boards, there are some hacks in the\nPCB design. The CD4066 and the LM*37s are only\nrequired on one board
+$Comp
+L 4xxx:4066 U2
+U 2 1 5EF33DA8
+P 1050 5900
+F 0 "U2" H 1050 5727 50  0000 C CNN
+F 1 "4066" H 1050 5636 50  0000 C CNN
+F 2 "KiCad/kicad-footprints/Package_DIP.pretty:DIP-14_W7.62mm" H 1050 5900 50  0001 C CNN
+F 3 "http://www.ti.com/lit/ds/symlink/cd4066b.pdf" H 1050 5900 50  0001 C CNN
+	2    1050 5900
+	1    0    0    -1
+$EndComp
+$Comp
+L 4xxx:4066 U2
+U 3 1 5EF34E81
+P 1900 5900
+F 0 "U2" H 1900 5727 50  0000 C CNN
+F 1 "4066" H 1900 5636 50  0000 C CNN
+F 2 "KiCad/kicad-footprints/Package_DIP.pretty:DIP-14_W7.62mm" H 1900 5900 50  0001 C CNN
+F 3 "http://www.ti.com/lit/ds/symlink/cd4066b.pdf" H 1900 5900 50  0001 C CNN
+	3    1900 5900
+	1    0    0    -1
+$EndComp
+$Comp
+L 4xxx:4066 U2
+U 4 1 5EF35DAB
+P 2700 5900
+F 0 "U2" H 2700 5727 50  0000 C CNN
+F 1 "4066" H 2700 5636 50  0000 C CNN
+F 2 "KiCad/kicad-footprints/Package_DIP.pretty:DIP-14_W7.62mm" H 2700 5900 50  0001 C CNN
+F 3 "http://www.ti.com/lit/ds/symlink/cd4066b.pdf" H 2700 5900 50  0001 C CNN
+	4    2700 5900
+	1    0    0    -1
+$EndComp
+Text GLabel 1500 6500 2    50   Input ~ 0
+4066_3
+Text GLabel 1500 6600 2    50   Input ~ 0
+4066_4
+Text GLabel 1500 6700 2    50   Input ~ 0
+4066_5
+Text GLabel 1500 6800 2    50   Input ~ 0
+4066_6
+Text GLabel 2250 6500 0    50   Input ~ 0
+4066_12
+Text GLabel 2250 6600 0    50   Input ~ 0
+4066_11
+Text GLabel 2250 6700 0    50   Input ~ 0
+4066_10
+Text GLabel 2250 6800 0    50   Input ~ 0
+4066_9
+Text GLabel 2250 6900 0    50   Input ~ 0
+4066_8
+Wire Wire Line
+	2400 6900 2250 6900
+Wire Wire Line
+	2250 6800 2400 6800
+Wire Wire Line
+	2400 6700 2250 6700
+Wire Wire Line
+	2250 6600 2400 6600
+Wire Wire Line
+	2400 6500 2250 6500
+Wire Wire Line
+	1350 6800 1500 6800
+Wire Wire Line
+	1350 6700 1500 6700
+Wire Wire Line
+	1500 6600 1350 6600
+Wire Wire Line
+	1350 6500 1500 6500
+$Comp
+L Connector_Generic:Conn_01x05 J8
+U 1 1 5EFFDABB
+P 2600 6700
+F 0 "J8" H 2680 6742 50  0000 L CNN
+F 1 "Conn_01x05" H 2680 6651 50  0000 L CNN
+F 2 "imciner2/KiCad-Libraries/modules/Connectors.pretty:CONN_2.54mm_1x05" H 2600 6700 50  0001 C CNN
+F 3 "~" H 2600 6700 50  0001 C CNN
+	1    2600 6700
+	1    0    0    -1
+$EndComp
+$Comp
+L Connector_Generic:Conn_01x04 J7
+U 1 1 5EFFF3AA
+P 1150 6600
+F 0 "J7" H 1068 6917 50  0000 C CNN
+F 1 "Conn_01x04" H 1068 6826 50  0000 C CNN
+F 2 "imciner2/KiCad-Libraries/modules/Connectors.pretty:CONN_2.54mm_1x04" H 1150 6600 50  0001 C CNN
+F 3 "~" H 1150 6600 50  0001 C CNN
+	1    1150 6600
+	-1   0    0    -1
+$EndComp
+Text GLabel 1400 5850 1    50   Input ~ 0
+4066_3
+Text GLabel 700  5850 1    50   Input ~ 0
+4066_4
+Text GLabel 1050 5500 1    50   Input ~ 0
+4066_5
+Text GLabel 1900 5500 1    50   Input ~ 0
+4066_6
+Text GLabel 1550 5850 1    50   Input ~ 0
+4066_8
+Text GLabel 2250 5850 1    50   Input ~ 0
+4066_9
+Text GLabel 3050 5850 1    50   Input ~ 0
+4066_10
+Text GLabel 2350 5850 1    50   Input ~ 0
+4066_11
+Text GLabel 2700 5500 1    50   Input ~ 0
+4066_12
+Wire Wire Line
+	2700 5500 2700 5600
+Wire Wire Line
+	3050 5850 3050 5900
+Wire Wire Line
+	3050 5900 3000 5900
+Wire Wire Line
+	2400 5900 2350 5900
+Wire Wire Line
+	2350 5900 2350 5850
+Wire Wire Line
+	2200 5900 2250 5900
+Wire Wire Line
+	2250 5900 2250 5850
+Wire Wire Line
+	1900 5600 1900 5500
+Wire Wire Line
+	1600 5900 1550 5900
+Wire Wire Line
+	1550 5900 1550 5850
+Wire Wire Line
+	1400 5850 1400 5900
+Wire Wire Line
+	1400 5900 1350 5900
+Wire Wire Line
+	1050 5600 1050 5500
+Wire Wire Line
+	750  5900 700  5900
+Wire Wire Line
+	700  5900 700  5850
 $EndSCHEMATC

Commit message: move the quirks of the pcb out of the schematic
Parts:
- removed J7: Conn_01x04, imciner2/KiCad-Libraries/modules/Connectors.pretty:CONN_2.54mm_1x04, symbol Connector_Generic:Conn_01x04
- removed J8: Conn_01x05, imciner2/KiCad-Libraries/modules/Connectors.pretty:CONN_2.54mm_1x05, symbol Connector_Generic:Conn_01x05
- removed RV1: 100K, rdeterre/misc.pretty:Potentiometer_Bourns_PDB182-K_Dual, symbol Device:R_POT_Dual
- removed unit 2 of U2
- removed unit 3 of U2
- removed unit 4 of U2
- added RV1: 200K, rdeterre/misc.pretty:Potentiometer_Bourns_PDB182-K_Dual, symbol Device:R_POT
Connections:
- net labels removed: 4066_10, 4066_11, 4066_12, 4066_3, 4066_4, 4066_5, 4066_6, 4066_8, 4066_9
- wire segments 147 -> 121
Other:
- note added: "gain 0-2\nideally 1 detent pot so it sits at g=1"
- note removed: "I was originally targeting a 200K pot. However,\nThe only 1 Detent PDB18X available was a 100K\n2 gang pot, so instead we use both gangs in series\nand can keep the input impedance at 100K and still\nget a gain of 0-2"
- note removed: "In order to share the switches of a single CD4066\nacross multiple boards, there are some hacks in the\nPCB design. The CD4066 and the LM*37s are only\nrequired on one board"
Changed lines of the file:
@@
 	1    0    0    -1
 $EndComp
-$Comp
-L Device:R_POT_Dual RV1
-U 1 1 5ECF889E
-P 4550 3800
-F 0 "RV1" H 4450 3900 50  0000 C CNN
-F 1 "100K" H 4550 3600 50  0000 C CNN
-F 2 "rdeterre/misc.pretty:Potentiometer_Bourns_PDB182-K_Dual" H 4800 3725 50  0001 C CNN
-F 3 "~" H 4800 3725 50  0001 C CNN
-	1    4550 3800
-	1    0    0    1
-$EndComp
-Text Notes 5000 3550 2    50   ~ 0
-I was originally targeting a 200K pot. However,\nThe only 1 Detent PDB18X available was a 100K\n2 gang pot, so instead we use both gangs in series\nand can keep the input impedance at 100K and still\nget a gain of 0-2
-Wire Wire Line
-	4050 3700 4050 3900
-Wire Wire Line
-	4650 3700 4550 3700
-Wire Wire Line
-	4800 3900 4550 3900
-Wire Wire Line
-	4550 3900 4550 3700
-Connection ~ 4550 3700
-Wire Wire Line
-	4550 3700 4450 3700
-Wire Wire Line
-	4950 3700 5050 3700
+Text Notes 4850 3350 2    50   ~ 0
+gain 0-2\nideally 1 detent pot so it sits at g=1
 Text Notes 7900 3450 2    50   ~ 0
 Considered an LED here, but most require 20mA\nwhich is a serious bite out of the power supply
-Wire Wire Line
-	4050 3700 4150 3700
-Wire Wire Line
-	4050 3900 4300 3900
-Connection ~ 4050 3900
-Wire Wire Line
-	4050 3900 4050 4150
 $Comp
 L 4xxx:4066 U2
@@
 	1    0    0    -1
 $EndComp
-Wire Wire Line
-	5050 3700 5050 4250
-Wire Wire Line
-	4700 4250 5050 4250
-Connection ~ 5050 4250
-Wire Wire Line
-	5050 4250 5150 4250
 Wire Wire Line
 	5750 4250 5800 4250
@@
 Text Notes 9050 3200 0    50   ~ 0
 The CD4066 has a max power supply voltage of 20V,\nso we step the 24V down to about 19.5 via regulators.\nIn theory we could hacky do this with 6 diodes instead
-Text Notes 1150 7500 0    50   ~ 0
-In order to share the switches of a single CD4066\nacross multiple boards, there are some hacks in the\nPCB design. The CD4066 and the LM*37s are only\nrequired on one board
-$Comp
-L 4xxx:4066 U2
-U 2 1 5EF33DA8
-P 1050 5900
-F 0 "U2" H 1050 5727 50  0000 C CNN
-F 1 "4066" H 1050 5636 50  0000 C CNN
-F 2 "KiCad/kicad-footprints/Package_DIP.pretty:DIP-14_W7.62mm" H 1050 5900 50  0001 C CNN
-F 3 "http://www.ti.com/lit/ds/symlink/cd4066b.pdf" H 1050 5900 50  0001 C CNN
-	2    1050 5900
-	1    0    0    -1
-$EndComp
-$Comp
-L 4xxx:4066 U2
-U 3 1 5EF34E81
-P 1900 5900
-F 0 "U2" H 1900 5727 50  0000 C CNN
-F 1 "4066" H 1900 5636 50  0000 C CNN
-F 2 "KiCad/kicad-footprints/Package_DIP.pretty:DIP-14_W7.62mm" H 1900 5900 50  0001 C CNN
-F 3 "http://www.ti.com/lit/ds/symlink/cd4066b.pdf" H 1900 5900 50  0001 C CNN
-	3    1900 5900
-	1    0    0    -1
-$EndComp
-$Comp
-L 4xxx:4066 U2
-U 4 1 5EF35DAB
-P 2700 5900
-F 0 "U2" H 2700 5727 50  0000 C CNN
-F 1 "4066" H 2700 5636 50  0000 C CNN
-F 2 "KiCad/kicad-footprints/Package_DIP.pretty:DIP-14_W7.62mm" H 2700 5900 50  0001 C CNN
-F 3 "http://www.ti.com/lit/ds/symlink/cd4066b.pdf" H 2700 5900 50  0001 C CNN
-	4    2700 5900
-	1    0    0    -1
-$EndComp
-Text GLabel 1500 6500 2    50   Input ~ 0
-4066_3
-Text GLabel 1500 6600 2    50   Input ~ 0
-4066_4
-Text GLabel 1500 6700 2    50   Input ~ 0
-4066_5
-Text GLabel 1500 6800 2    50   Input ~ 0
-4066_6
-Text GLabel 2250 6500 0    50   Input ~ 0
-4066_12
-Text GLabel 2250 6600 0    50   Input ~ 0
-4066_11
-Text GLabel 2250 6700 0    50   Input ~ 0
-4066_10
-Text GLabel 2250 6800 0    50   Input ~ 0
-4066_9
-Text GLabel 2250 6900 0    50   Input ~ 0
-4066_8
-Wire Wire Line
-	2400 6900 2250 6900
-Wire Wire Line
-	2250 6800 2400 6800
-Wire Wire Line
-	2400 6700 2250 6700
-Wire Wire Line
-	2250 6600 2400 6600
-Wire Wire Line
-	2400 6500 2250 6500
-Wire Wire Line
-	1350 6800 1500 6800
-Wire Wire Line
-	1350 6700 1500 6700
-Wire Wire Line
-	1500 6600 1350 6600
-Wire Wire Line
-	1350 6500 1500 6500
-$Comp
-L Connector_Generic:Conn_01x05 J8
-U 1 1 5EFFDABB
-P 2600 6700
-F 0 "J8" H 2680 6742 50  0000 L CNN
-F 1 "Conn_01x05" H 2680 6651 50  0000 L CNN
-F 2 "imciner2/KiCad-Libraries/modules/Connectors.pretty:CONN_2.54mm_1x05" H 2600 6700 50  0001 C CNN
-F 3 "~" H 2600 6700 50  0001 C CNN
-	1    2600 6700
-	1    0    0    -1
-$EndComp
-$Comp
-L Connector_Generic:Conn_01x04 J7
-U 1 1 5EFFF3AA
-P 1150 6600
-F 0 "J7" H 1068 6917 50  0000 C CNN
-F 1 "Conn_01x04" H 1068 6826 50  0000 C CNN
-F 2 "imciner2/KiCad-Libraries/modules/Connectors.pretty:CONN_2.54mm_1x04" H 1150 6600 50  0001 C CNN
-F 3 "~" H 1150 6600 50  0001 C CNN
-	1    1150 6600
-	-1   0    0    -1
-$EndComp
-Text GLabel 1400 5850 1    50   Input ~ 0
-4066_3
-Text GLabel 700  5850 1    50   Input ~ 0
-4066_4
-Text GLabel 1050 5500 1    50   Input ~ 0
-4066_5
-Text GLabel 1900 5500 1    50   Input ~ 0
-4066_6
-Text GLabel 1550 5850 1    50   Input ~ 0
-4066_8
-Text GLabel 2250 5850 1    50   Input ~ 0
-4066_9
-Text GLabel 3050 5850 1    50   Input ~ 0
-4066_10
-Text GLabel 2350 5850 1    50   Input ~ 0
-4066_11
-Text GLabel 2700 5500 1    50   Input ~ 0
-4066_12
-Wire Wire Line
-	2700 5500 2700 5600
-Wire Wire Line
-	3050 5850 3050 5900
-Wire Wire Line
-	3050 5900 3000 5900
-Wire Wire Line
-	2400 5900 2350 5900
-Wire Wire Line
-	2350 5900 2350 5850
-Wire Wire Line
-	2200 5900 2250 5900
-Wire Wire Line
-	2250 5900 2250 5850
-Wire Wire Line
-	1900 5600 1900 5500
-Wire Wire Line
-	1600 5900 1550 5900
-Wire Wire Line
-	1550 5900 1550 5850
-Wire Wire Line
-	1400 5850 1400 5900
-Wire Wire Line
-	1400 5900 1350 5900
-Wire Wire Line
-	1050 5600 1050 5500
-Wire Wire Line
-	750  5900 700  5900
-Wire Wire Line
-	700  5900 700  5850
+$Comp
+L Device:R_POT RV1
+U 1 1 5ECB664B
+P 4500 3700
+F 0 "RV1" V 4293 3700 50  0000 C CNN
+F 1 "200K" V 4384 3700 50  0000 C CNN
+F 2 "rdeterre/misc.pretty:Potentiometer_Bourns_PDB182-K_Dual" H 4500 3700 50  0001 C CNN
+F 3 "~" H 4500 3700 50  0001 C CNN
+	1    4500 3700
+	0    1    1    0
+$EndComp
+Wire Wire Line
+	4050 3700 4050 4150
+Wire Wire Line
+	4050 3700 4250 3700
+Wire Wire Line
+	4500 3850 4500 3900
+Wire Wire Line
+	4500 3900 4250 3900
+Wire Wire Line
+	4250 3900 4250 3700
+Connection ~ 4250 3700
+Wire Wire Line
+	4250 3700 4350 3700
+Wire Wire Line
+	4700 4250 4800 4250
+Wire Wire Line
+	4650 3700 4800 3700
+Wire Wire Line
+	4800 3700 4800 4250
+Connection ~ 4800 4250
+Wire Wire Line
+	4800 4250 5150 4250
 $EndSCHEMATC
