File: vco/vco.sch (KiCad schematic (older format))
At the start: 56 parts

Commit message: write code for shape selector, design CV input stage of vco
Parts:
- added D? (x4): LED, symbol Device:LED
- added R? (x2): 10K, symbol Device:R
- added R? (x4): 100K, symbol Device:R
- added R? (x2): 110K, symbol Device:R
- added R? (x4): 220, symbol Device:R
- added RV?: 100K, symbol Device:R_POT
- added RV?: 10K, symbol Device:R_POT
- added U?: DG403, Package_SO:SOIC-16_3.9x9.9mm_P1.27mm, symbol synth:DG403
- added U? (x2): TL072, symbol Amplifier_Operational:TL072
- RV?: value R_POT -> 100K
Connections:
- net +12V: now also R?.2, R?.2
- net GND: now also R?.1, R?.1, R?.2, R?.2, R?.2, R?.2, R?.2, U?.1 (D1)
- net SINE: now also U?.3 (D3)
- net SINE_EN: now also U?.5 (AREF/PB0), D?.2 (A); no longer U?.7 (PB2)
- net SQUARE: no longer U?.3 (D3), U?.6 (D4)
- net SQUARE_EN: now also U?.3 (XTAL2/PB4); no longer U?.5 (AREF/PB0)
- net TRIANGLE: now also U?.6 (D4)
- net TRIANGLE_EN: no longer R?.1, U?.10 (IN2)
- net at R?.1, R?.2, R?.2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: now also R?.2, R?.2
- net OCT_EN: now reaches U?.2 (XTAL1/PB3)
- net OCT_EN: now also D?.2 (A), R?.1, U?.15 (IN1)
- net at RV?.2: now also U?.7 (PB2); no longer U?.3 (XTAL2/PB4)
- net at R?.2, R?.2, R?.2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: now also R?.2
- new net: D?.2 (A), R?.1, U?.10 (IN2)
- new net: R?.1, U?.16 (S1), U?.4 (S3)
- new net: RV?.2, U?.5 (+) (x2)
- new net: R?.1, RV?.1 (x2)
- new net: R?.2, RV?.3 (x2)
- new net: D?.1 (K), R?.1 (x4)
- new net COARSE_CV: R?.1, U?.6 (-), U?.7
- new net FINE_CV: R?.1, U?.6 (-), U?.7
- new net OCT: U?.3 (D3)
- no-connect marks 0 -> 1
Other:
- note added: "0-10V, 1V/octave"
- note added: "COARSE knob\n-4V to 4V"
- note added: "FINE knob\n-0.52V to 0.52V\nTODO might need to be even finer"
- note added: "PWM control\nvia adjusting reference voltage of comparator\nTODO this is a pretty janky way to do this"
- note added: "TODO does this value need to be tunable?"
- note added: "system of equations:\n24(b/(a+b+100))=11\n24((b+100)/(a+b+100))=21"
- note added: "tempco\nthermally connected to bjts"
- note removed: "PWM control\nvia adjusting reference voltage of comparator"
- note removed: "TODO: one more output available if we can find a shape"
- note removed: "tempco"
- moved on the sheet: R?, RV?, U?, U?A, U?B

Commit message: notes
Parts:
- added R?: 150k, symbol Device:R
- added R?: 100k, symbol Device:R
- added R? (x3): 10K, symbol Device:R
- added RV?: 1K, symbol Device:R_POT
- added U?: LM311, symbol Comparator:LM311
Connections:
- net +12V: now also R?.1, R?.1, U?.8 (V+)
- net -12V: now also R?.2, U?.1 (GND), U?.4 (V-)
- new net: R?.1, R?.2, U?.2 (+)
- new net: R?.1, R?.2, U?.7
- new net: R?.2, RV?.2
- new net: R?.2, RV?.3
- new net: R?.1, RV?.1
- no-connect marks 1 -> 3
Other:
- note added: "Compensate for VBE"
- note added: "TODO If it helps performance, a real comparator can be used here instead:"
- note added: "TODO: these can be combined to one"
Changed lines of the file:
@@
 Text Notes 1650 4150 0    50   ~ 0
 TODO does this value need to be tunable?
+Text Notes -1200 3650 0    50   ~ 0
+TODO: these can be combined to one
+Text Notes 4000 750  0    50   ~ 0
+TODO If it helps performance, a real comparator can be used here instead:
+$Comp
+L Comparator:LM311 U?
+U 1 1 6043D86B
+P 5050 1450
+F 0 "U?" H 5394 1496 50  0000 L CNN
+F 1 "LM311" H 5394 1405 50  0000 L CNN
+F 2 "" H 5050 1450 50  0001 C CNN
+F 3 "https://www.st.com/resource/en/datasheet/lm311.pdf" H 5050 1450 50  0001 C CNN
+	1    5050 1450
+	1    0    0    -1
+$EndComp
+$Comp
+L power:+12V #PWR?
+U 1 1 6043FDAB
+P 4950 1050
+F 0 "#PWR?" H 4950 900 50  0001 C CNN
+F 1 "+12V" H 4965 1223 50  0000 C CNN
+F 2 "" H 4950 1050 50  0001 C CNN
+F 3 "" H 4950 1050 50  0001 C CNN
+	1    4950 1050
+	1    0    0    -1
+$EndComp
+$Comp
+L power:-12V #PWR?
+U 1 1 6044046B
+P 4950 1850
+F 0 "#PWR?" H 4950 1950 50  0001 C CNN
+F 1 "-12V" H 4965 2023 50  0000 C CNN
+F 2 "" H 4950 1850 50  0001 C CNN
+F 3 "" H 4950 1850 50  0001 C CNN
+	1    4950 1850
+	-1   0    0    1
+$EndComp
+$Comp
+L Device:R R?
+U 1 1 60440D89
+P 5500 1850
+F 0 "R?" H 5600 1950 50  0000 L CNN
+F 1 "150k" H 5600 1800 50  0000 L CNN
+F 2 "" V 5430 1850 50  0001 C CNN
+F 3 "~" H 5500 1850 50  0001 C CNN
+	1    5500 1850
+	1    0    0    -1
+$EndComp
+$Comp
+L Device:R R?
+U 1 1 60440D93
+P 5500 2300
+F 0 "R?" H 5600 2350 50  0000 L CNN
+F 1 "100k" H 5600 2250 50  0000 L CNN
+F 2 "" V 5430 2300 50  0001 C CNN
+F 3 "~" H 5500 2300 50  0001 C CNN
+	1    5500 2300
+	1    0    0    -1
+$EndComp
+Wire Wire Line
+	5500 2150 5500 2100
+Wire Wire Line
+	5500 2100 4600 2100
+Connection ~ 5500 2100
+Wire Wire Line
+	5500 2100 5500 2000
+Wire Wire Line
+	4750 1350 4600 1350
+Wire Wire Line
+	4600 1350 4600 2100
+Wire Wire Line
+	5500 1700 5500 1450
+Wire Wire Line
+	5500 1450 5350 1450
+$Comp
+L Device:R R?
+U 1 1 6047CFEB
+P 5950 2200
+F 0 "R?" V 6050 2150 50  0000 L CNN
+F 1 "10K" V 5950 2100 50  0000 L CNN
+F 2 "" V 5880 2200 50  0001 C CNN
+F 3 "~" H 5950 2200 50  0001 C CNN
+	1    5950 2200
+	1    0    0    -1
+$EndComp
+$Comp
+L Device:R R?
+U 1 1 6047CFF5
+P 5950 2900
+F 0 "R?" V 6050 2850 50  0000 L CNN
+F 1 "10K" V 5950 2800 50  0000 L CNN
+F 2 "" V 5880 2900 50  0001 C CNN
+F 3 "~" H 5950 2900 50  0001 C CNN
+	1    5950 2900
+	1    0    0    -1
+$EndComp
+$Comp
+L Device:R_POT RV?
+U 1 1 6047CFFF
+P 5950 2550
+F 0 "RV?" H 5880 2596 50  0000 R CNN
+F 1 "1K" H 5880 2505 50  0000 R CNN
+F 2 "" H 5950 2550 50  0001 C CNN
+F 3 "~" H 5950 2550 50  0001 C CNN
+	1    5950 2550
+	-1   0    0    1
+$EndComp
+$Comp
+L power:+12V #PWR?
+U 1 1 6047D009
+P 5950 2000
+F 0 "#PWR?" H 5950 1850 50  0001 C CNN
+F 1 "+12V" H 5965 2173 50  0000 C CNN
+F 2 "" H 5950 2000 50  0001 C CNN
+F 3 "" H 5950 2000 50  0001 C CNN
+	1    5950 2000
+	1    0    0    -1
+$EndComp
+$Comp
+L power:-12V #PWR?
+U 1 1 6047D013
+P 5950 3100
+F 0 "#PWR?" H 5950 3200 50  0001 C CNN
+F 1 "-12V" H 5965 3273 50  0000 C CNN
+F 2 "" H 5950 3100 50  0001 C CNN
+F 3 "" H 5950 3100 50  0001 C CNN
+	1    5950 3100
+	-1   0    0    1
+$EndComp
+Wire Wire Line
+	5950 3100 5950 3050
+Wire Wire Line
+	5950 2750 5950 2700
+Wire Wire Line
+	5950 2400 5950 2350
+Wire Wire Line
+	5950 2000 5950 2050
+Wire Wire Line
+	5800 2550 5500 2550
+Wire Wire Line
+	5500 2550 5500 2450
+Text Notes 6300 2900 1    50   ~ 0
+Compensate for VBE
+Wire Wire Line
+	4950 1850 4950 1800
+Wire Wire Line
+	4950 1150 4950 1050
+NoConn ~ 5050 1150
+NoConn ~ 5150 1150
+Wire Wire Line
+	5050 1750 5050 1800
+Wire Wire Line
+	5050 1800 4950 1800
+Connection ~ 4950 1800
+Wire Wire Line
+	4950 1800 4950 1750
+$Comp
+L Device:R R?
+U 1 1 60534A48
+P 5500 1150
+F 0 "R?" H 5600 1250 50  0000 L CNN
+F 1 "10K" H 5600 1100 50  0000 L CNN
+F 2 "" V 5430 1150 50  0001 C CNN
+F 3 "~" H 5500 1150 50  0001 C CNN
+	1    5500 1150
+	1    0    0    -1
+$EndComp
+Wire Wire Line
+	5500 1300 5500 1450
+Connection ~ 5500 1450
+$Comp
+L power:+12V #PWR?
+U 1 1 6054A16D
+P 5500 900
+F 0 "#PWR?" H 5500 750 50  0001 C CNN
+F 1 "+12V" H 5515 1073 50  0000 C CNN
+F 2 "" H 5500 900 50  0001 C CNN
+F 3 "" H 5500 900 50  0001 C CNN
+	1    5500 900
+	1    0    0    -1
+$EndComp
+Wire Wire Line
+	5500 900  5500 1000
 $EndSCHEMATC
