File: clock/clock/clock.sch (KiCad schematic (older format))
At the start: 46 parts, among them J1 AVR-ISP-6, J10 Conn_01x05_Male, J11 CV_IN, J12 CLOCK_OUT, J13 SUBDIV_OUT, J2 EURORACK_CONN_10, J3 Conn_01x05_Female, J4 Conn_01x05_Male, J5 Conn_01x05_Female, J6 Conn_01x05_Male, J7 Conn_01x05_Female, J8 Conn_01x05_Male, J9 Conn_01x05_Female, SW1 SW_Push, SW2 SW_Push, SW3 SW_Rotary8, U1 ATmega328P-PU, U2 L7805, U3 SM460281N, U4 SM460281N, U5 SM460281N, Y1 16MHz

Commit message: refactor
Parts:
- added R?: 120K, symbol Device:R
- added R?: 680k, symbol Device:R
- added R?: 220K, symbol Device:R
- added R?: 470K, symbol Device:R
- added R?: 1M, symbol Device:R
- added SW?: SW_Coded_SH-7050, symbol Switch:SW_Coded_SH-7050
Connections:
- net +5V: now also R?.1, R?.1, R?.1, R?.1
- net GND: now also R?.1
- net KNOB: now also R?.2, SW?.C
- new net: R?.2, SW?.1
- new net: R?.2, SW?.2
- new net: R?.2, SW?.4
- new net: R?.2, SW?.8
Changed lines of the file:
@@
 Text Notes 7800 5150 0    50   ~ 0
 bound input CV to 0-5V
+$Comp
+L Switch:SW_Coded_SH-7050 SW?
+U 1 1 6348F991
+P 4150 10300
+F 0 "SW?" H 4207 10767 50  0000 C CNN
+F 1 "SW_Coded_SH-7050" H 4207 10676 50  0000 C CNN
+F 2 "" H 3850 9850 50  0001 L CNN
+F 3 "https://www.nidec-copal-electronics.com/e/catalog/switch/sh-7000.pdf" H 4150 10300 50  0001 C CNN
+	1    4150 10300
+	1    0    0    -1
+$EndComp
+$Comp
+L Device:R R?
+U 1 1 634912AF
+P 4900 10200
+F 0 "R?" V 4900 10500 50  0000 C CNN
+F 1 "120K" V 4900 10200 50  0000 C CNN
+F 2 "" V 4830 10200 50  0001 C CNN
+F 3 "~" H 4900 10200 50  0001 C CNN
+	1    4900 10200
+	0    1    1    0
+$EndComp
+$Comp
+L Device:R R?
+U 1 1 63491618
+P 5500 10250
+F 0 "R?" H 5430 10204 50  0000 R CNN
+F 1 "680k" H 5430 10295 50  0000 R CNN
+F 2 "" V 5430 10250 50  0001 C CNN
+F 3 "~" H 5500 10250 50  0001 C CNN
+	1    5500 10250
+	-1   0    0    1
+$EndComp
+$Comp
+L power:+5V #PWR?
+U 1 1 63492617
+P 5100 9900
+F 0 "#PWR?" H 5100 9750 50  0001 C CNN
+F 1 "+5V" H 5115 10073 50  0000 C CNN
+F 2 "" H 5100 9900 50  0001 C CNN
+F 3 "" H 5100 9900 50  0001 C CNN
+	1    5100 9900
+	1    0    0    -1
+$EndComp
+$Comp
+L power:GND #PWR?
+U 1 1 6349300A
+P 5500 10600
+F 0 "#PWR?" H 5500 10350 50  0001 C CNN
+F 1 "GND" H 5505 10427 50  0000 C CNN
+F 2 "" H 5500 10600 50  0001 C CNN
+F 3 "" H 5500 10600 50  0001 C CNN
+	1    5500 10600
+	1    0    0    -1
+$EndComp
+Wire Wire Line
+	5500 10600 5500 10400
+Wire Wire Line
+	5500 10100 4550 10100
+Wire Wire Line
+	5100 9900 5100 10200
+Wire Wire Line
+	5100 10500 5050 10500
+Wire Wire Line
+	5050 10400 5100 10400
+Connection ~ 5100 10400
+Wire Wire Line
+	5100 10400 5100 10500
+Wire Wire Line
+	5050 10300 5100 10300
+Connection ~ 5100 10300
+Wire Wire Line
+	5100 10300 5100 10400
+Wire Wire Line
+	5100 10200 5050 10200
+Connection ~ 5100 10200
+Wire Wire Line
+	5100 10200 5100 10300
+Wire Wire Line
+	4750 10200 4550 10200
+Wire Wire Line
+	4550 10300 4750 10300
+Wire Wire Line
+	4750 10400 4550 10400
+Wire Wire Line
+	4550 10500 4750 10500
+Text Label 5850 10100 0    50   ~ 0
+KNOB
+Wire Wire Line
+	5850 10100 5500 10100
+Connection ~ 5500 10100
+$Comp
+L Device:R R?
+U 1 1 635B6095
+P 4900 10300
+F 0 "R?" V 4900 10600 50  0000 C CNN
+F 1 "220K" V 4900 10300 50  0000 C CNN
+F 2 "" V 4830 10300 50  0001 C CNN
+F 3 "~" H 4900 10300 50  0001 C CNN
+	1    4900 10300
+	0    1    1    0
+$EndComp
+$Comp
+L Device:R R?
+U 1 1 635B63E3
+P 4900 10400
+F 0 "R?" V 4900 10700 50  0000 C CNN
+F 1 "470K" V 4900 10400 50  0000 C CNN
+F 2 "" V 4830 10400 50  0001 C CNN
+F 3 "~" H 4900 10400 50  0001 C CNN
+	1    4900 10400
+	0    1    1    0
+$EndComp
+$Comp
+L Device:R R?
+U 1 1 635B6785
+P 4900 10500
+F 0 "R?" V 4900 10800 50  0000 C CNN
+F 1 "1M" V 4900 10500 50  0000 C CNN
+F 2 "" V 4830 10500 50  0001 C CNN
+F 3 "~" H 4900 10500 50  0001 C CNN
+	1    4900 10500
+	0    1    1    0
+$EndComp
 $EndSCHEMATC

Commit message: tuned
Parts:
- removed R10, R11, R12, R6, R7, R8, R9: 10K, Resistor_THT:R_Axial_DIN0207_L6.3mm_D2.5mm_P2.54mm_Vertical, symbol Device:R
- removed SW3: SW_Rotary8, synth:RM100772BCB, symbol Switch:SW_Rotary8
- R?: value 680k -> 68k
Other:
- moved on the sheet: R?, SW?
