File: adsr/adsr.kicad_pcb (KiCad board)
At the start: 2 copper layers, 80.3 x 112.3 mm, 41 parts, among them J10 Conn_01x08_Male, J11 Conn_01x08_Female, J12 Conn_01x08_Male, J3 B_IN, J4 A_IN, J5 B_OUT, J6 A_OUT, J7 EURORACK_CONN_16, J8 Conn_01x04_Male, J9 Conn_01x08_Female, Q1 2N3904, Q2 2N3904, Q5 DMMT5401, U1 LM13700, U2 TL074, U3 DG403, U4 DG403

Commit message: adsr improvements
Parts:
- added C11: 4.7u, Capacitor_SMD:C_1206_3216Metric_Pad1.42x1.75mm_HandSolder, F.Cu at (115.1, 48.0)
- added C12: 4.7u, Capacitor_SMD:C_1206_3216Metric_Pad1.42x1.75mm_HandSolder, F.Cu at (135.4, 56.4)
- added C3: 0.1u, Capacitor_SMD:C_1206_3216Metric_Pad1.42x1.75mm_HandSolder, F.Cu at (127.1, 60.5)
- added C4: 100n, Capacitor_SMD:C_1206_3216Metric_Pad1.42x1.75mm_HandSolder, F.Cu at (135.3, 102.7)
- added C5: 0.1u, Capacitor_SMD:C_1206_3216Metric_Pad1.42x1.75mm_HandSolder, F.Cu at (122.7, 32.0)
- added C6: 0.1u, Capacitor_SMD:C_1206_3216Metric_Pad1.42x1.75mm_HandSolder, F.Cu at (126.6, 32.0)
- added D2: D, Diode_THT:D_A-405_P2.54mm_Vertical_AnodeUp, F.Cu at (129.6, 105.1)
- added J1: Conn_01x04_Female, Connector_PinHeader_2.54mm:PinHeader_1x04_P2.54mm_Vertical, F.Cu at (114.0, 29.7)
- added J13: Conn_01x04_Male, Connector_PinHeader_2.54mm:PinHeader_1x04_P2.54mm_Vertical, B.Cu at (135.6, 41.9)
- added J14: Conn_01x04_Male, Connector_PinHeader_2.54mm:PinHeader_1x04_P2.54mm_Vertical, F.Cu at (69.3, 29.5)
- added J2: Conn_01x04_Male, Connector_PinHeader_2.54mm:PinHeader_1x04_P2.54mm_Vertical, B.Cu at (90.9, 41.7)
- added Q3: 2N3904, Package_TO_SOT_THT:TO-92_Inline, F.Cu at (134.7, 108.5)
- added Q4: 2N3904, Package_TO_SOT_THT:TO-92_Inline, F.Cu at (129.2, 108.5)
- added Q6: DMMT5401, Package_TO_SOT_SMD:SOT-23-6_Handsoldering, F.Cu at (146.3, 138.4)
- added R10: 100K, Resistor_SMD:R_1206_3216Metric_Pad1.42x1.75mm_HandSolder, F.Cu at (129.3, 114.2)
- added R11: 100K, Resistor_SMD:R_1206_3216Metric_Pad1.42x1.75mm_HandSolder, F.Cu at (135.3, 114.2)
- added R12: 1K, Resistor_SMD:R_1206_3216Metric_Pad1.42x1.75mm_HandSolder, F.Cu at (135.3, 105.3)
- added R17: 10K, Resistor_SMD:R_1206_3216Metric_Pad1.42x1.75mm_HandSolder, F.Cu at (74.2, 123.8)
- added R18: 10K, Resistor_SMD:R_1206_3216Metric_Pad1.42x1.75mm_HandSolder, F.Cu at (81.4, 124.5)
- added R20: 6.8k, Resistor_SMD:R_1206_3216Metric_Pad1.42x1.75mm_HandSolder, F.Cu at (138.9, 137.4)
- added R21: 1K, Resistor_SMD:R_1206_3216Metric_Pad1.42x1.75mm_HandSolder, F.Cu at (90.7, 98.3)
- added R22: 100K, Resistor_SMD:R_1206_3216Metric_Pad1.42x1.75mm_HandSolder, F.Cu at (86.5, 104.6)
- added R23: 1K, Resistor_SMD:R_1206_3216Metric_Pad1.42x1.75mm_HandSolder, F.Cu at (86.4, 92.9)
- added R24: 100K, Resistor_SMD:R_1206_3216Metric_Pad1.42x1.75mm_HandSolder, F.Cu at (92.4, 89.6)
- added R7: 6.8k, Resistor_SMD:R_1206_3216Metric_Pad1.42x1.75mm_HandSolder, F.Cu at (147.0, 146.0)
- added R8: 1K, Resistor_SMD:R_1206_3216Metric_Pad1.42x1.75mm_HandSolder, F.Cu at (113.2, 66.0)
- added R9: 100K, Resistor_SMD:R_1206_3216Metric_Pad1.42x1.75mm_HandSolder, F.Cu at (116.5, 66.0)
- added U5: DG403, Package_SO:SOIC-16_3.9x9.9mm_P1.27mm, F.Cu at (119.4, 98.8)
- added U6: DG403, Package_SO:SOIC-16_3.9x9.9mm_P1.27mm, F.Cu at (85.3, 74.2)
- added U7: TL074, Package_DIP:DIP-14_W7.62mm, F.Cu at (72.9, 95.2)
- added U8: TL072, Package_DIP:DIP-8_W7.62mm, F.Cu at (128.4, 72.6)
- C1: value 4.7u -> 0.1u
- J10, J12: moved to B.Cu
- J8: footprint Connector_PinHeader_2.54mm:PinHeader_2x02_P2.54mm_Vertical -> Connector_PinHeader_2.54mm:PinHeader_1x04_P2.54mm_Vertical; moved to B.Cu
- moved R19 97.0 mm to (124.9, 138.9)
- moved U3 89.6 mm to (119.4, 110.9), turned to 0 degrees
- moved Q5 89.3 mm to (118.1, 139.1)
- moved R15 73.9 mm to (59.9, 121.8)
- moved R16 73.9 mm to (59.9, 124.8)
- moved C8 69.2 mm to (61.1, 115.3)
- moved C7 69.2 mm to (55.3, 115.3)
- moved R4 65.2 mm to (129.8, 83.5), turned to 0 degrees
- moved R3 65.0 mm to (135.9, 68.7), turned to 90 degrees
- moved C2 64.5 mm to (135.4, 95.9), turned to 0 degrees
- moved Q1 64.1 mm to (134.9, 86.8)
- moved R2 62.2 mm to (132.6, 68.7), turned to 270 degrees
- moved R6 61.5 mm to (135.4, 92.8), turned to 0 degrees
- moved U1 60.8 mm to (128.4, 54.1)
- moved R5 60.4 mm to (135.3, 83.7), turned to 180 degrees
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Connections:
- net Net-(C3-Pad1) renamed /sheet5F5D80AF/VC
- C1 pad 1: Net-(C1-Pad1) -> +12V
- D3 pad 1: Net-(D3-Pad1) -> /envelope/IN_RAW
- D4 pad 1: Net-(D4-Pad1) -> /sheet5F5D80AF/IN_RAW
- J10 pad 1: A_OUT -> /envelope/IN_RAW
- J10 pad 2: /envelope/ATTACK -> A_OUT
- J10 pad 3: /envelope/DECAY -> /envelope/ATTACK
- J10 pad 4: /envelope/REF_RAW -> /envelope/DECAY
- J10 pad 5: /envelope/SUS_RAW -> /envelope/REF_RAW
- J10 pad 6: /envelope/RELEASE -> /envelope/SUS_RAW
- J10 pad 7: GND -> /envelope/RELEASE
- J11 pad 1: B_OUT -> /sheet5F5D80AF/IN_RAW
- J11 pad 2: /sheet5F5D80AF/ATTACK -> B_OUT
- J11 pad 3: /sheet5F5D80AF/DECAY -> /sheet5F5D80AF/ATTACK
- J11 pad 4: /sheet5F5D80AF/REF_RAW -> /sheet5F5D80AF/DECAY
- J11 pad 5: /sheet5F5D80AF/SUS_RAW -> /sheet5F5D80AF/REF_RAW
- J11 pad 6: /sheet5F5D80AF/RELEASE -> /sheet5F5D80AF/SUS_RAW
- J11 pad 7: GND -> /sheet5F5D80AF/RELEASE
- J12 pad 1: B_OUT -> /sheet5F5D80AF/IN_RAW
- J12 pad 2: /sheet5F5D80AF/ATTACK -> B_OUT
- J12 pad 3: /sheet5F5D80AF/DECAY -> /sheet5F5D80AF/ATTACK
- J12 pad 4: /sheet5F5D80AF/REF_RAW -> /sheet5F5D80AF/DECAY
- J12 pad 5: /sheet5F5D80AF/SUS_RAW -> /sheet5F5D80AF/REF_RAW
- J12 pad 6: /sheet5F5D80AF/RELEASE -> /sheet5F5D80AF/SUS_RAW
- J12 pad 7: GND -> /sheet5F5D80AF/RELEASE
- J8 pad 1: A_IN_DEFAULT -> B_OUT_DEFAULT
- J8 pad 3: A_OUT_DEFAULT -> A_IN_DEFAULT
- J8 pad 4: B_OUT_DEFAULT -> A_OUT_DEFAULT
- J9 pad 1: A_OUT -> /envelope/IN_RAW
- J9 pad 2: /envelope/ATTACK -> A_OUT
- J9 pad 3: /envelope/DECAY -> /envelope/ATTACK
- J9 pad 4: /envelope/REF_RAW -> /envelope/DECAY
- J9 pad 5: /envelope/SUS_RAW -> /envelope/REF_RAW
- J9 pad 6: /envelope/RELEASE -> /envelope/SUS_RAW
- J9 pad 7: GND -> /envelope/RELEASE
- R13 pad 1: Net-(D3-Pad1) -> /envelope/IN_RAW
- R14 pad 1: Net-(D4-Pad1) -> /sheet5F5D80AF/IN_RAW
- R4 pad 1: /envelope/REF -> /envelope/VINS
- U1 pad 12: Net-(C1-Pad1) -> /envelope/VC
- U1 pad 13: Net-(C1-Pad1) -> /envelope/VC
- U2 pad 10: Net-(R2-Pad2) -> /envelope/VC
- U2 pad 12: Net-(C1-Pad1) -> /envelope/IN_RAW
- U2 pad 13: Net-(R15-Pad2) -> Net-(R21-Pad1)
- U2 pad 14: A_OUT -> /envelope/VINS
- U2 pad 8: Net-(U1-Pad10) -> A_OUT
- U2 pad 9: Net-(C1-Pad1) -> Net-(R15-Pad2)
- U3 pad 15: /envelope/REF -> /envelope/VINS
- U4 pad 15: /envelope/REF -> /envelope/VINS
Routing:
- net +12V: track 205.6 -> 71.3 mm, vias 7 -> 1
- net -12V: track 156.8 -> 75.2 mm, vias 3 -> 0
- net /envelope/STATE: track 85.6 -> 4.41 mm, vias 3 -> 0
- net Net-(U1-Pad14): track 74.1 -> 0.00 mm, vias 1 -> 0
- net Net-(R2-Pad2): track 53.4 -> 0.00 mm, vias 1 -> 0
- net /envelope/REF: track 49.9 -> 0.00 mm, vias 1 -> 0
- net Net-(Q5-Pad4): track 48.9 -> 0.00 mm, vias 2 -> 0
- net Net-(C1-Pad1): track 43.3 -> 0.00 mm, vias 1 -> 0
- net /envelope/ATTACK: track 82.4 -> 40.7 mm
- net /envelope/DECAY: track 68.4 -> 30.3 mm
- net A_OUT: track 74.0 -> 38.7 mm, vias 3 -> 1
- net /envelope/SUS: track 34.0 -> 0.00 mm, vias 1 -> 0
- net Net-(R15-Pad2): track 31.2 -> 0.00 mm, vias 1 -> 0
- net Net-(Q1-Pad2): track 33.1 -> 6.80 mm, vias 2 -> 0
- net /envelope/RELEASE: track 103.3 -> 78.2 mm, vias 1 -> 0
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Other:
- board size 80.3 x 112.3 mm -> 125 x 112.5 mm

Commit message: update adsr to kicad 6
Connections:
- J7 pad 13: Net-(J7-Pad13) -> unconnected-(J7-Pad13)
- J7 pad 15: Net-(J7-Pad15) -> unconnected-(J7-Pad15)
- U1 pad 15: Net-(U1-Pad15) -> unconnected-(U1-Pad15)
- U1 pad 2: Net-(U1-Pad2) -> unconnected-(U1-Pad2)
- U3 pad 2: Net-(U3-Pad2) -> unconnected-(U3-Pad2)
- U3 pad 7: Net-(U3-Pad7) -> unconnected-(U3-Pad7)
- U4 pad 2: Net-(U4-Pad2) -> unconnected-(U4-Pad2)
- U4 pad 7: Net-(U4-Pad7) -> unconnected-(U4-Pad7)
- U5 pad 2: Net-(U5-Pad2) -> unconnected-(U5-Pad2)
- U5 pad 7: Net-(U5-Pad7) -> unconnected-(U5-Pad7)
- U6 pad 2: Net-(U6-Pad2) -> unconnected-(U6-Pad2)
- U6 pad 7: Net-(U6-Pad7) -> unconnected-(U6-Pad7)
Routing:
- net unconnected-(J7-Pad15): track 0.00 -> 2.54 mm
- net unconnected-(J7-Pad13): track 0.00 -> 2.54 mm
- net Net-(J7-Pad15): track 2.54 -> 0.00 mm
- net Net-(J7-Pad13): track 2.54 -> 0.00 mm
Other:
- net class Default removed
