File: mixer/channel.kicad_sch (KiCad schematic)
At the start: 36 parts, among them J7 CHANNEL_IN, J8 AVR-ISP-6, Q1 NMOS, SW1 AUX_PRE_POST_FADER_SLIDESW, SW2 MONO_PBSW, SW3 SOLO_PBSW, U2 TL074, U3 DG403, U4 TL074, U5 TL074, U6 TL074, U7 TL074, U8 TL074, U9 ATtiny85-20S

Commit message: working out some parts
Parts:
- added RV1: A1M_AUX_SEND, synth:Potentiometer_Alpha_RD901F-40-00D_Single_Vertical, symbol Device:R_Potentiometer
- added U10: TL074, symbol Amplifier_Operational:TL074
- RV5: value A1M_GAIN -> B1M_GAIN; footprint Potentiometer_THT:Potentiometer_Alpha_RD901F-40-00D_Single_Vertical -> _project:3352W
- RV6: footprint Potentiometer_THT:Potentiometer_Alpha_RD902F-40-00D_Dual_Vertical_CircularHoles -> synth:Potentiometer_Alpha_RD902F-40-00D_Dual_Vertical_CircularHoles
- SW1: footprint (none) -> synth:Dailywell SPDT Sub-Mini Slide SW
- SW2, SW3: footprint (none) -> Button_Switch_THT:SW_PUSH_6mm; symbol Switch:SW_Push_Dual -> Switch:SW_Push
Connections:
- net +5V: no longer SW2.3, SW3.3
- net C_AUX: now also RV1.1; no longer R11.1
- net GND: now also RV1.3
- net at J8.4 (MOSI), R17.1, SW2.2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: no longer SW2.4
- net at J8.1 (MISO), R19.1, SW3.2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: no longer SW3.4
- new net: RV1.2, U10.10 (+)
- new net: R11.1, U10.8, U10.9 (-)
Other:
- note added: "3352W-105LF-ND This little thumbwheel allows us to squeeze one more pot in so that the fader can be entirely negative gain"
- note added: "https://www.thonk.co.uk/shop/dailywell-sl1/"

Commit message: 2 channel chain
Parts:
- removed C5: 100n, symbol Device:C
- removed J8: AVR-ISP-6, symbol Connector:AVR-ISP-6
- removed Q1: NMOS, symbol Simulation_SPICE:NMOS
- removed R10, R11, R12, R13, R14, R15, R7, R8, R9: 100k, symbol Device:R
- removed U10, U4, U8: TL074, symbol Amplifier_Operational:TL074
- removed unit 3 of U2
- removed U9: ATtiny85-20S, Package_SO:SOIC-8_5.3x5.3mm_P1.27mm, symbol MCU_Microchip_ATtiny:ATtiny85-20S
- added U5: TL072, symbol Amplifier_Operational:TL072
- R12: renamed from R21; value 1k -> 10k
- SW1: renamed from SW2; value MONO_PBSW -> MUTE_PBSW
- renumbered D2 to D1, D1 to D2, R6 to R10, R5 to R11, R17 to R6, R19 to R7, R18 to R8, R20 to R9, RV5 to RV3, RV1 to RV5, SW3 to SW2, SW1 to SW3, U5 to U2, U6 to U4, U7 to U4
Connections:
- net C_AUX_OUT: now also U5.1, U5.2 (-)
- net C_PAN_L: now also U4.6 (-), U4.7; no longer U4.8, U4.9 (-)
- net C_PAN_R: now also U4.1, U4.2 (-); no longer U4.8, U4.9 (-)
- net at R8.1: now also D1.1 (K); no longer D2.1 (K)
- net C_SOLO_LED: now reaches D2.2 (A)
- net C_MUTE_LED: now reaches D1.2 (A)
- net C_MUTE: now reaches R6.1, SW1.2
- net C_SOLO: now reaches R7.1, SW2.2
- net at R9.1: now also D2.1 (K); no longer D1.1 (K)
- net at RV6.2: now also U4.5 (+); no longer U4.10 (+)
- net at RV4.2: now also U2.5 (+); no longer U2.10 (+)
- net at RV5.2: now also U5.3 (+)
- net at RV6.5: now also U4.3 (+); no longer U4.10 (+)
- net C_AUX: no longer names the net of RV5.1, SW3.2 (B)
- net C_FADER: no longer names the net of RV6.3, RV6.4, SW3.3 (C)
- net C_FADER: now also U2.6 (-), U2.7; no longer U2.8, U2.9 (-)
- net C_IN: no longer names the net of J7.T, R10.1
- net MUTED renamed C_MUTED
Other:
- note added: "MUTE/SOLO"
- note removed: "Considered using discrete digital logic. However, with debounce, latch, and gates, MCU much more space efficenct (even with programming headers)"
- note removed: "pullup on master"
- moved on the sheet: D1, D2, J7, R10, R11, R12, R6, R7, R8, R9, RV3, RV4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

Commit message: making progress on the outline
Parts:
- D1, D2: footprint (none) -> LED_THT:LED_D2.0mm_W4.8mm_H2.5mm_FlatTop
- R10, R11, R12, R6, R7, R8, R9: footprint (none) -> Resistor_SMD:R_0603_1608Metric
- U2, U4: footprint (none) -> Package_SO:SOIC-14_3.9x8.7mm_P1.27mm
- U5: footprint (none) -> Package_SO:SOIC-8_3.9x4.9mm_P1.27mm
Connections:
- net GND: now also RV4.1; no longer RV4.3
- net at RV3.2, RV3.3, U2.1: now also U3.3 (D3); no longer U3.1 (D1)
- net at U3.4 (S3): now also RV4.3, SW3.1 (A)
- now unconnected: U3.16 (S1)
Other:
- note added: "AUX"
- note added: "FADER"
- note added: "PAN"
- moved on the sheet: D1, D2, R12, R6, R7, R8, R9, SW1, SW2, U3A

Commit message: layed out parts
Parts:
- removed U5: TL072, Package_SO:SOIC-8_3.9x4.9mm_P1.27mm, symbol Amplifier_Operational:TL072
- RV5: value A1M_AUX_SEND -> B1M_AUX_SEND
- RV6: value B100K_PAN -> A100K_PAN
Connections:
- net C_AUX_OUT: now also RV5.2
Changed lines of the file:
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@@
-	)
-	(junction
-		(at 228.6 134.62)
-		(diameter 0)
-		(color 0 0 0 0)
 	)
 	(junction
@@
 	(wire
 		(pts
-			(xy 228.6 140.97) (xy 228.6 134.62)
-		)
-		(stroke
-			(width 0)
-			(type default)
-		)
-	)
-	(wire
-		(pts
 			(xy 209.55 87.63) (xy 228.6 87.63)
 		)
@@
 	(wire
 		(pts
+			(xy 193.04 132.08) (xy 208.28 132.08)
+		)
+		(stroke
+			(width 0)
+			(type default)
+		)
+	)
+	(wire
+		(pts
 			(xy 72.39 72.39) (xy 76.2 72.39)
 		)
@@
 	(wire
 		(pts
-			(xy 193.04 132.08) (xy 210.82 132.08)
-		)
-		(stroke
-			(width 0)
-			(type default)
-		)
-	)
-	(wire
-		(pts
 			(xy 209.55 116.84) (xy 209.55 120.65)
 		)
@@
 	(wire
 		(pts
-			(xy 226.06 134.62) (xy 228.6 134.62)
-		)
-		(stroke
-			(width 0)
-			(type default)
-		)
-	)
-	(wire
-		(pts
 			(xy 106.68 69.85) (xy 109.22 69.85)
 		)
@@
 	(wire
 		(pts
-			(xy 210.82 137.16) (xy 209.55 137.16)
-		)
-		(stroke
-			(width 0)
-			(type default)
-		)
-	)
-	(wire
-		(pts
 			(xy 96.52 76.2) (xy 96.52 69.85)
 		)
@@
 	(wire
 		(pts
-			(xy 228.6 134.62) (xy 232.41 134.62)
-		)
-		(stroke
-			(width 0)
-			(type default)
-		)
-	)
-	(wire
-		(pts
 			(xy 228.6 114.3) (xy 226.06 114.3)
 		)
@@
 	(wire
 		(pts
-			(xy 209.55 137.16) (xy 209.55 140.97)
-		)
-		(stroke
-			(width 0)
-			(type default)
-		)
-	)
-	(wire
-		(pts
 			(xy 142.24 81.28) (xy 172.72 81.28)
 		)
@@
 		(pts
 			(xy 172.72 86.36) (xy 170.18 86.36)
-		)
-		(stroke
-			(width 0)
-			(type default)
-		)
-	)
-	(wire
-		(pts
-			(xy 209.55 140.97) (xy 228.6 140.97)
 		)
 		(stroke
@@
 	(hierarchical_label "C_AUX_OUT"
 		(shape input)
-		(at 232.41 134.62 0)
+		(at 208.28 132.08 0)
 		(effects
 			(font
@@
 	)
 	(symbol
-		(lib_id "Amplifier_Operational:TL072")
-		(at 218.44 134.62 0)
-		(unit 1)
-		(exclude_from_sim no)
-		(in_bom yes)
-		(on_board yes)
-		(dnp no)
-		(property "Reference" "U5"
-			(at 221.234 128.778 0)
-			(effects
-				(font
-					(size 1.27 1.27)
-				)
-			)
-		)
-		(property "Value" "TL072"
-			(at 221.234 131.318 0)
-			(effects
-				(font
-					(size 1.27 1.27)
-				)
-			)
-		)
-		(property "Footprint" "Package_SO:SOIC-8_3.9x4.9mm_P1.27mm"
-			(at 218.44 134.62 0)
-			(effects
-				(font
-					(size 1.27 1.27)
-				)
-				(hide yes)
-			)
-		)
-		(property "Datasheet" "http://www.ti.com/lit/ds/symlink/tl071.pdf"
-			(at 218.44 134.62 0)
-			(effects
-				(font
-					(size 1.27 1.27)
-				)
-				(hide yes)
-			)
-		)
-		(property "Description" "Dual Low-Noise JFET-Input Operational Amplifiers, DIP-8/SOIC-8"
-			(at 218.44 134.62 0)
-			(effects
-				(font
-					(size 1.27 1.27)
-				)
-				(hide yes)
-			)
-		)
-		(pin "4"
-		)
-		(pin "2"
-		)
-		(pin "3"
-		)
-		(pin "5"
-		)
-		(pin "6"
-		)
-		(pin "1"
-		)
-		(pin "7"
-		)
-		(pin "8"
-		)
-		(instances
-			(project "mixer"
-				(path "/7887173d-29cc-4936-b1a7-ffeb730ae153/45f99337-f06b-4142-99e3-547e8fb47392/206f6037-7ae6-4b64-94eb-9a85666ebdcd"
-					(reference "U5")
-					(unit 1)
-				)
-				(path "/7887173d-29cc-4936-b1a7-ffeb730ae153/45f99337-f06b-4142-99e3-547e8fb47392/5c9695de-fd6a-48f6-b871-1584ea81abcb"
-					(reference "U5")
-					(unit 2)
-				)
-			)
-		)
-	)
-	(symbol
 		(lib_id "Device:R_Potentiometer_Dual_Separate")
 		(at 207.01 105.41 270)
@@
 			)
 		)
-		(property "Value" "B100K_PAN"
+		(property "Value" "A100K_PAN"
 			(at 212.852 100.33 90)
 			(effects
@@
 			)
 		)
-		(property "Value" "A1M_AUX_SEND"
+		(property "Value" "B1M_AUX_SEND"
 			(at 186.69 133.3499 0)
 			(effects
@@
 			)
 		)
-		(property "Value" "B100K_PAN"
+		(property "Value" "A100K_PAN"
 			(at 201.93 98.044 90)
 			(effects

Commit message: layout master board
Parts:
- RV4: footprint Potentiometer_THT:Potentiometer_Bourns_PTA3043_Single_Slide -> _project:Potentiometer_Bourns_PTA3043_Single_Slide
Changed lines of the file:
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@@
 			)
 		)
-		(property "Footprint" "Potentiometer_THT:Potentiometer_Bourns_PTA3043_Single_Slide"
+		(property "Footprint" "_project:Potentiometer_Bourns_PTA3043_Single_Slide"
 			(at 142.24 96.52 0)
 			(effects

Commit message: first pass route
Parts:
- renumbered U4 to U2, U2 to U4
Connections:
- net C_PAN_L: now also U2.13 (-), U2.14; no longer U2.6 (-), U2.7
- net C_PAN_R: now also U2.8, U2.9 (-); no longer U2.1, U2.2 (-)
- net GND: now also U4.12 (+); no longer U4.3 (+)
- net at RV6.2: now also U2.12 (+); no longer U2.5 (+)
- net at RV6.3, RV6.4, SW3.3 (C): now also U4.8, U4.9 (-); no longer U4.6 (-), U4.7
- net at R10.2, R11.1: now also U4.13 (-); no longer U4.2 (-)
- net at RV4.2: now also U4.10 (+); no longer U4.5 (+)
- net at RV3.2, RV3.3, U3.3 (D3): now also U4.14; no longer U4.1
- net at RV6.5: now also U2.10 (+); no longer U2.3 (+)
Changed lines of the file:
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@@
 		(lib_id "Amplifier_Operational:TL074")
 		(at 158.75 99.06 0)
-		(unit 2)
-		(exclude_from_sim no)
-		(in_bom yes)
-		(on_board yes)
-		(dnp no)
-		(property "Reference" "U2"
+		(unit 3)
+		(exclude_from_sim no)
+		(in_bom yes)
+		(on_board yes)
+		(dnp no)
+		(property "Reference" "U4"
 			(at 160.528 92.456 0)
 			(effects
@@
 			(project "mixer"
 				(path "/7887173d-29cc-4936-b1a7-ffeb730ae153/45f99337-f06b-4142-99e3-547e8fb47392/206f6037-7ae6-4b64-94eb-9a85666ebdcd"
-					(reference "U2")
+					(reference "U4")
+					(unit 3)
+				)
+				(path "/7887173d-29cc-4936-b1a7-ffeb730ae153/45f99337-f06b-4142-99e3-547e8fb47392/5c9695de-fd6a-48f6-b871-1584ea81abcb"
+					(reference "U4")
 					(unit 2)
-				)
-				(path "/7887173d-29cc-4936-b1a7-ffeb730ae153/45f99337-f06b-4142-99e3-547e8fb47392/5c9695de-fd6a-48f6-b871-1584ea81abcb"
-					(reference "U2")
-					(unit 4)
 				)
 			)
@@
 		(lib_id "Amplifier_Operational:TL074")
 		(at 218.44 81.28 0)
-		(unit 1)
-		(exclude_from_sim no)
-		(in_bom yes)
-		(on_board yes)
-		(dnp no)
-		(property "Reference" "U4"
+		(unit 3)
+		(exclude_from_sim no)
+		(in_bom yes)
+		(on_board yes)
+		(dnp no)
+		(property "Reference" "U2"
 			(at 220.218 74.676 0)
 			(effects
@@
 			(project "mixer"
 				(path "/7887173d-29cc-4936-b1a7-ffeb730ae153/45f99337-f06b-4142-99e3-547e8fb47392/206f6037-7ae6-4b64-94eb-9a85666ebdcd"
-					(reference "U4")
-					(unit 1)
-				)
-				(path "/7887173d-29cc-4936-b1a7-ffeb730ae153/45f99337-f06b-4142-99e3-547e8fb47392/5c9695de-fd6a-48f6-b871-1584ea81abcb"
-					(reference "U4")
+					(reference "U2")
 					(unit 3)
+				)
+				(path "/7887173d-29cc-4936-b1a7-ffeb730ae153/45f99337-f06b-4142-99e3-547e8fb47392/5c9695de-fd6a-48f6-b871-1584ea81abcb"
+					(reference "U2")
+					(unit 2)
 				)
 			)
@@
 		(lib_id "Amplifier_Operational:TL074")
 		(at 218.44 114.3 0)
-		(unit 2)
-		(exclude_from_sim no)
-		(in_bom yes)
-		(on_board yes)
-		(dnp no)
-		(property "Reference" "U4"
+		(unit 4)
+		(exclude_from_sim no)
+		(in_bom yes)
+		(on_board yes)
+		(dnp no)
+		(property "Reference" "U2"
 			(at 220.218 107.696 0)
 			(effects
@@
 			(project "mixer"
 				(path "/7887173d-29cc-4936-b1a7-ffeb730ae153/45f99337-f06b-4142-99e3-547e8fb47392/206f6037-7ae6-4b64-94eb-9a85666ebdcd"
-					(reference "U4")
-					(unit 2)
-				)
-				(path "/7887173d-29cc-4936-b1a7-ffeb730ae153/45f99337-f06b-4142-99e3-547e8fb47392/5c9695de-fd6a-48f6-b871-1584ea81abcb"
-					(reference "U4")
+					(reference "U2")
 					(unit 4)
+				)
+				(path "/7887173d-29cc-4936-b1a7-ffeb730ae153/45f99337-f06b-4142-99e3-547e8fb47392/5c9695de-fd6a-48f6-b871-1584ea81abcb"
+					(reference "U2")
+					(unit 1)
 				)
 			)
@@
 		(at 109.22 78.74 0)
 		(mirror x)
-		(unit 1)
-		(exclude_from_sim no)
-		(in_bom yes)
-		(on_board yes)
-		(dnp no)
-		(property "Reference" "U2"
+		(unit 4)
+		(exclude_from_sim no)
+		(in_bom yes)
+		(on_board yes)
+		(dnp no)
+		(property "Reference" "U4"
 			(at 111.252 86.106 0)
 			(effects
@@
 			(project "mixer"
 				(path "/7887173d-29cc-4936-b1a7-ffeb730ae153/45f99337-f06b-4142-99e3-547e8fb47392/206f6037-7ae6-4b64-94eb-9a85666ebdcd"
-					(reference "U2")
-					(unit 1)
-				)
-				(path "/7887173d-29cc-4936-b1a7-ffeb730ae153/45f99337-f06b-4142-99e3-547e8fb47392/5c9695de-fd6a-48f6-b871-1584ea81abcb"
-					(reference "U2")
-					(unit 3)
-				)
-			)
+					(reference "U4")
+					(unit 4)
+				)
+				(path "/7887173d-29cc-4936-b1a7-ffeb730ae153/45f99337-f06b-4142-99e3-547e8fb47392/5c9695de-fd6a-48f6-b871-1584ea81abcb"
+					(reference "U4")
+					(unit 1)
+				)
+			)
