File: mixer/channels.kicad_sch (KiCad schematic)
At the start: 21 parts, among them J8 AVR-ISP-6, Q1 NMOS, U2 TL074, U3 DG403, U4 TL074, U5 TL072, U6 ATtiny24-20SS, U7 TL074

Commit message: making progress on the outline
Parts:
- added C6, C7, C8, C9: 100n, Capacitor_SMD:C_0603_1608Metric, symbol Device:C
- C5: footprint (none) -> Capacitor_SMD:C_0603_1608Metric
- J8: footprint (none) -> _project:IVR_PADS
- R13, R14, R15, R16, R17, R18, R19, R20, R21, R22, R23, R24: footprint (none) -> Resistor_SMD:R_0603_1608Metric
- U2, U4, U7: footprint (none) -> Package_SO:SOIC-14_3.9x8.7mm_P1.27mm
- U5: footprint (none) -> Package_SO:SOIC-8_3.9x4.9mm_P1.27mm
Connections:
- net +12V: now also U2.4 (V+), U3.11 (V+), U4.4 (V+), U5.8 (V+), U7.4 (V+), C6.1, C7.1, C8.1, C9.1
- net +5V: now also U3.12 (VL)
- net -12V: now also U2.11 (V-), U3.14 (V-), U4.11 (V-), U5.4 (V-), U7.11 (V-), C6.2, C7.2, C8.2, C9.2
- net GND: now also U3.13 (GND)
Other:
- moved on the sheet: U2E, U3C, U4E, U5C, U7E

Commit message: layed out parts
Parts:
- removed C8, C9: 100n, Capacitor_SMD:C_0603_1608Metric, symbol Device:C
- removed R13, R16, R19, R22, R23, R24: 100k, Resistor_SMD:R_0603_1608Metric, symbol Device:R
- removed U5: TL072, Package_SO:SOIC-8_3.9x4.9mm_P1.27mm, symbol Amplifier_Operational:TL072
- removed U7: TL074, Package_SO:SOIC-14_3.9x8.7mm_P1.27mm, symbol Amplifier_Operational:TL074
- R17, R18, R20, R21: value 100k -> 33k
Connections:
- net C_BUS_L: now reaches R20.2, R21.2
- net C_BUS_AUX: now reaches R14.2, R15.2
- net C_BUS_R: now reaches R17.2, R18.2
Other:
- note added: "These resistors matched to summing amp in master"
- note removed: "summing"
- note removed: "unused"

Commit message: first pass route
Parts:
- removed Q1: NMOS, symbol Simulation_SPICE:NMOS
- added C10, C8, C9: 100n, Capacitor_SMD:C_0603_1608Metric, symbol Device:C
- added Q1: BSS214NW, Package_TO_SOT_SMD:SOT-323_SC-70, symbol Transistor_FET:BSS214NW
Connections:
- net +12V: now also C8.1
- net +5V: now also C10.1
- net -12V: now also C9.2
- net GND: now also C10.2, C8.2, C9.1, Q1.2 (S)
- net SOLOED: now also Q1.1 (G)
- net ~{GLOBAL_SOLO}: now also Q1.3 (D)
Other:
- note added: "JM recommends BSS816NW"
- moved on the sheet: C6, C7, U2E, U4E
