File: mixer/mixer.kicad_pcb (KiCad board)
At the start: 2 copper layers, 12 parts, among them J1 AUX_OUT, J2 AUX_IN_R, J3 AUX_IN_L, J4 MAIN_OUT_R, J5 MAIN_OUT_L, J6 EURORACK_CONN_16, J7 CHANNEL_IN, U3 DG403

Commit message: working out some parts
Parts:
- added RV1: A1M_AUX_SEND, synth:Potentiometer_Alpha_RD901F-40-00D_Single_Vertical, F.Cu at (131.1, 102.1)
- added RV7: A100K_MASTER_FADER, synth:Potentiometer_Alpha_RD902F-40-00D_Dual_Vertical_CircularHoles, F.Cu at (157.5, 158.0)
- added SW1: AUX_PRE_POST_FADER_SLIDESW, synth:Dailywell SPDT Sub-Mini Slide SW, F.Cu at (134.0, 107.1)
- added SW2: MONO_PBSW, Button_Switch_THT:SW_PUSH_6mm, F.Cu at (126.9, 182.5)
- added SW3: SOLO_PBSW, Button_Switch_THT:SW_PUSH_6mm, F.Cu at (136.8, 182.4)
- added U9: ATtiny85-20S, Package_SO:SOIC-8_5.3x5.3mm_P1.27mm, F.Cu at (189.5, 104.8)
- RV2: footprint Potentiometer_THT:Potentiometer_Alpha_RD902F-40-00D_Dual_Vertical -> synth:Potentiometer_Alpha_RD902F-40-00D_Dual_Vertical_CircularHoles
- RV5: value A1M_GAIN -> B1M_GAIN; footprint Potentiometer_THT:Potentiometer_Alpha_RD901F-40-00D_Single_Vertical -> _project:3352W
- RV6: footprint Potentiometer_THT:Potentiometer_Alpha_RD902F-40-00D_Dual_Vertical_CircularHoles -> synth:Potentiometer_Alpha_RD902F-40-00D_Dual_Vertical_CircularHoles
- moved J5 70.3 mm to (160.0, 88.3), turned to -90 degrees
- moved J3 68.2 mm to (160.0, 118.7), turned to -90 degrees
- moved J4 57.1 mm to (160.0, 78.1), turned to -90 degrees
- moved J2 53.3 mm to (160.0, 108.6), turned to -90 degrees
- moved J6 47.0 mm to (228.6, 142.9)
- moved J1 38.5 mm to (160.0, 98.4), turned to -90 degrees
- moved RV2 35.5 mm to (157.5, 139.1)
- moved RV5 21.0 mm to (136.3, 79.8)
- moved RV4 8.25 mm to (132.9, 171.4)
- moved RV6 7.87 mm to (131.9, 123.0)
- moved J7 4.45 mm to (130.2, 79.8)

Commit message: making progress on the outline
Parts:
- removed U9: ATtiny85-20S, Package_SO:SOIC-8_5.3x5.3mm_P1.27mm
- added C1: 10u, Capacitor_SMD:C_0603_1608Metric, F.Cu at (251.7, 143.8)
- added C2: 10u, Capacitor_SMD:C_0603_1608Metric, F.Cu at (251.7, 146.3)
- added C3: 10u, Capacitor_SMD:C_0603_1608Metric, F.Cu at (251.7, 148.8)
- added C4: 100n, Capacitor_SMD:C_0603_1608Metric, F.Cu at (273.8, 108.2)
- added C5: 100n, Capacitor_SMD:C_0603_1608Metric, F.Cu at (-45.0, 147.3)
- added C6: 100n, Capacitor_SMD:C_0603_1608Metric, F.Cu at (-29.5, 73.2)
- added C7: 100n, Capacitor_SMD:C_0603_1608Metric, F.Cu at (-34.7, 113.2)
- added C8: 100n, Capacitor_SMD:C_0603_1608Metric, F.Cu at (86.6, 23.4)
- added C9: 100n, Capacitor_SMD:C_0603_1608Metric, F.Cu at (-33.1, 52.3)
- added D1: M_LED_RED, LED_THT:LED_D2.0mm_W4.8mm_H2.5mm_FlatTop, F.Cu at (88.9, 152.9)
- added D2: S_LED_ORANGE, LED_THT:LED_D2.0mm_W4.8mm_H2.5mm_FlatTop, F.Cu at (88.9, 160.5)
- added D3: M_LED_RED, LED_THT:LED_D2.0mm_W4.8mm_H2.5mm_FlatTop, F.Cu at (104.1, 152.9)
- added D4: S_LED_ORANGE, LED_THT:LED_D2.0mm_W4.8mm_H2.5mm_FlatTop, F.Cu at (104.1, 160.5)
- added J10: C_BOARD_IN_1, Connector_PinSocket_2.54mm:PinSocket_2x04_P2.54mm_Horizontal, B.Cu at (139.7, 61.0)
- added J11: C_BOARD_IN_2, Connector_PinSocket_2.54mm:PinSocket_2x04_P2.54mm_Horizontal, B.Cu at (139.7, 160.0)
- added J12: M_BOARD_IN_1, Connector_PinSocket_2.54mm:PinSocket_2x04_P2.54mm_Horizontal, F.Cu at (259.1, 20.3)
- added J13: M_BOARD_IN_2, Connector_PinSocket_2.54mm:PinSocket_2x04_P2.54mm_Horizontal, F.Cu at (267.2, 168.9)
- added J14: C_BOARD_OUT_1, Connector_PinHeader_2.54mm:PinHeader_2x04_P2.54mm_Horizontal, B.Cu at (149.9, 61.0)
- added J15: C_BOARD_OUT_2, Connector_PinHeader_2.54mm:PinHeader_2x04_P2.54mm_Horizontal, B.Cu at (149.9, 160.0)
- added J8: AVR-ISP-6, _project:IVR_PADS, F.Cu at (-43.5, 165.9)
- added J9: CHANNEL_IN, synth:Jack_3.5mm_QingPu_WQP-PJ398SM_Vertical_CircularHoles, F.Cu at (101.6, 57.4)
- added R1: 10k, Resistor_SMD:R_0603_1608Metric, F.Cu at (271.0, 22.9)
- added R10: 10k, Resistor_SMD:R_0603_1608Metric, B.Cu at (85.1, 53.3)
- added R11: 10k, Resistor_SMD:R_0603_1608Metric, B.Cu at (88.9, 53.3)
- added R12: 10k, Resistor_SMD:R_0603_1608Metric, F.Cu at (-24.9, 153.4)
- added R13: 100k, Resistor_SMD:R_0603_1608Metric, F.Cu at (98.8, 33.9)
- added R14: 100k, Resistor_SMD:R_0603_1608Metric, F.Cu at (94.2, 33.1)
- added R15: 100k, Resistor_SMD:R_0603_1608Metric, F.Cu at (94.2, 35.6)
- added R16: 100k, Resistor_SMD:R_0603_1608Metric, F.Cu at (75.5, 22.9)
- added R17: 100k, Resistor_SMD:R_0603_1608Metric, F.Cu at (75.5, 25.4)
- added R18: 100k, Resistor_SMD:R_0603_1608Metric, F.Cu at (75.5, 27.9)
- added R19: 100k, Resistor_SMD:R_0603_1608Metric, F.Cu at (74.9, 38.0)
- added R2: 33k, Resistor_SMD:R_0603_1608Metric, F.Cu at (265.7, 116.9)
- added R20: 100k, Resistor_SMD:R_0603_1608Metric, F.Cu at (79.4, 34.6)
- added R21: 100k, Resistor_SMD:R_0603_1608Metric, F.Cu at (79.4, 37.1)
- added R22: 100k, Resistor_SMD:R_0603_1608Metric, F.Cu at (98.2, 38.1)
- added R23: 100k, Resistor_SMD:R_0603_1608Metric, F.Cu at (79.5, 25.4)
- added R24: 100k, Resistor_SMD:R_0603_1608Metric, F.Cu at (74.9, 34.4)
- added R25: 10k, Resistor_SMD:R_0603_1608Metric, F.Cu at (96.3, 168.2)
- added R26: 10k, Resistor_SMD:R_0603_1608Metric, F.Cu at (96.3, 170.7)
- added R27: 1k, Resistor_SMD:R_0603_1608Metric, F.Cu at (96.3, 173.3)
- added R28: 1k, Resistor_SMD:R_0603_1608Metric, F.Cu at (96.3, 175.8)
- added R29: 10k, Resistor_SMD:R_0603_1608Metric, F.Cu at (-21.8, 83.8)
- added R3: 33k, Resistor_SMD:R_0603_1608Metric, F.Cu at (265.7, 119.4)
- added R30: 10k, Resistor_SMD:R_0603_1608Metric, F.Cu at (-21.8, 86.3)
- added R31: 10k, Resistor_SMD:R_0603_1608Metric, F.Cu at (-25.2, 159.0)
- added R4: 33k, Resistor_SMD:R_0603_1608Metric, F.Cu at (283.7, 116.9)
- added R5: 33k, Resistor_SMD:R_0603_1608Metric, F.Cu at (283.7, 119.4)
- added R6: 10k, Resistor_SMD:R_0603_1608Metric, B.Cu at (81.3, 151.1)
- added R7: 10k, Resistor_SMD:R_0603_1608Metric, B.Cu at (81.3, 157.0)
- added R8: 1k, Resistor_SMD:R_0603_1608Metric, B.Cu at (81.3, 153.9)
- added R9: 1k, Resistor_SMD:R_0603_1608Metric, B.Cu at (81.3, 160.0)
- added RV10: B100K_PAN, synth:Potentiometer_Alpha_RD902F-40-00D_Dual_Vertical_CircularHoles, F.Cu at (99.6, 90.4)
- added RV3: B1M_GAIN, _project:3352W, F.Cu at (91.4, 56.3)
- added RV8: A100K_CHANNEL_FADER, Potentiometer_THT:Potentiometer_Bourns_PTA3043_Single_Slide, F.Cu at (97.8, 146.5)
- added RV9: A1M_AUX_SEND, synth:Potentiometer_Alpha_RD901F-40-00D_Single_Vertical, F.Cu at (99.6, 70.6)
- added SW4: MUTE_PBSW, Button_Switch_THT:SW_PUSH_6mm, F.Cu at (93.3, 149.4)
- added SW5: SOLO_PBSW, Button_Switch_THT:SW_PUSH_6mm, F.Cu at (93.3, 157.0)
- added SW6: AUX_PRE_POST_FADER_SLIDESW, synth:Dailywell SPDT Sub-Mini Slide SW, F.Cu at (99.6, 82.3)
- added U1: TL074, Package_SO:SOIC-14_3.9x8.7mm_P1.27mm, F.Cu at (272.9, 116.1)
- added U2: TL074, Package_SO:SOIC-14_3.9x8.7mm_P1.27mm, F.Cu at (-29.8, 80.3)
- added U4: TL074, Package_SO:SOIC-14_3.9x8.7mm_P1.27mm, F.Cu at (-34.4, 119.1)
- added U5: TL072, Package_SO:SOIC-8_3.9x4.9mm_P1.27mm, F.Cu at (-33.3, 57.0)
- added U6: ATtiny24-20SS, Package_SO:SOIC-14_3.9x8.7mm_P1.27mm, F.Cu at (-45.0, 156.5)
- added U7: TL074, Package_SO:SOIC-14_3.9x8.7mm_P1.27mm, F.Cu at (86.4, 30.0)
- J1: value AUX_OUT -> EURORACK_CONN_16; footprint synth:Jack_3.5mm_QingPu_WQP-PJ398SM_Vertical_CircularHoles -> synth:EURORACK_16_IDC; moved to B.Cu
- J2: value AUX_IN_R -> AUX_OUT
- J3: value AUX_IN_L -> AUX_IN_R
- J4: value MAIN_OUT_R -> AUX_IN_L
- J5: value MAIN_OUT_L -> MAIN_OUT_R
- J6: value EURORACK_CONN_16 -> MAIN_OUT_L; footprint synth:EURORACK_16_IDC -> synth:Jack_3.5mm_QingPu_WQP-PJ398SM_Vertical_CircularHoles
- RV1: value A1M_AUX_SEND -> A1M - AUX_RETURN_LEVEL; footprint synth:Potentiometer_Alpha_RD901F-40-00D_Single_Vertical -> synth:Potentiometer_Alpha_RD902F-40-00D_Dual_Vertical_CircularHoles
- RV2: value A1M - AUX_RETURN_LEVEL -> A100K_MASTER_VOL
- RV5: value B1M_GAIN -> A1M_AUX_SEND; footprint _project:3352W -> synth:Potentiometer_Alpha_RD901F-40-00D_Single_Vertical
- RV7: value A100K_MASTER_FADER -> B1M_GAIN; footprint synth:Potentiometer_Alpha_RD902F-40-00D_Dual_Vertical_CircularHoles -> _project:3352W
- SW1: value AUX_PRE_POST_FADER_SLIDESW -> MUTE_PBSW; footprint synth:Dailywell SPDT Sub-Mini Slide SW -> Button_Switch_THT:SW_PUSH_6mm
- SW2: value MONO_PBSW -> SOLO_PBSW
- SW3: value SOLO_PBSW -> AUX_PRE_POST_FADER_SLIDESW; footprint Button_Switch_THT:SW_PUSH_6mm -> synth:Dailywell SPDT Sub-Mini Slide SW
- moved U3 233.9 mm to (-32.9, 154.3)
- moved RV7 114.6 mm to (91.4, 64.4), turned to 180 degrees
- moved SW3 113.5 mm to (83.3, 82.3), turned to 0 degrees
- moved RV1 112.6 mm to (241.3, 78.7)
- moved J1 111.5 mm to (263.7, 139.7), turned to 180 degrees
- moved J6 87.0 mm to (238.7, 56.5)
- moved J4 86.7 mm to (238.8, 114.3)
- moved J3 78.9 mm to (238.8, 124.5)
- moved J2 78.9 mm to (238.8, 104.1)
- moved SW1 70.1 mm to (78.0, 149.4)
- moved J5 62.5 mm to (218.4, 66.0)
- moved RV2 62.5 mm to (215.9, 116.8)
- moved RV6 58.5 mm to (83.3, 90.4)
- moved RV4 57.0 mm to (81.6, 146.5)
- moved SW2 55.1 mm to (78.0, 157.0), turned to 0 degrees
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Connections:
- J2 pad T: AUX_RETURN_R -> /Master Module/M_AUX_IN
- J2 pad TN: GND -> unconnected-(J2-PadTN)
- J3 pad T: AUX_RETURN_L -> /Master Module/AUX_RETURN_R
- J3 pad TN: GND -> /Master Module/AUX_RETURN_L
- J4 pad T: Net-(J4-PadT) -> /Master Module/AUX_RETURN_L
- J4 pad TN: unconnected-(J4-PadTN) -> GND
- J7 pad T: C_IN -> Net-(J7-PadT)
- RV1 pad 1: C_AUX -> GND
- RV1 pad 3: GND -> /Master Module/AUX_RETURN_L
- RV2 pad 1: GND -> Net-(U1D--)
- RV2 pad 2: Net-(U1A-+) (its old number) -> Net-(J5-PadT)
- RV2 pad 3: AUX_RETURN_L -> Net-(J5-PadT)
- RV2 pad 4: GND -> Net-(U1C--)
- RV2 pad 5: Net-(U1B-+) -> Net-(J6-PadT)
- RV2 pad 6: AUX_RETURN_R -> Net-(J6-PadT)
- RV4 pad 1: Net-(SW1-A) -> GND
- RV4 pad 3: GND -> Net-(SW3-A)
- RV5 pad 1: Net-(R5-Pad2) -> Net-(SW3-B)
- RV5 pad 2: Net-(U3A-D1) -> Net-(U5A-+)
- RV5 pad 3: Net-(U3A-D1) -> GND
- RV6 pad 3: C_FADER -> Net-(SW3-C)
- RV6 pad 4: C_FADER -> Net-(SW3-C)
- RV7 pad 2: Net-(J4-PadT) -> Net-(U3B-D4)
- RV7 pad 3: Net-(J4-PadT) -> Net-(U3B-D4)
- SW1 pad 1: Net-(SW1-A) -> +5V
- SW1 pad 2: C_AUX -> /Channel Module/C1_MUTE
- SW2 pad 2: Net-(J8-MOSI) -> /Channel Module/C1_SOLO
- SW3 pad 1: +5V -> Net-(SW3-A)
- SW3 pad 2: Net-(J8-MISO) -> Net-(SW3-B)
- U3 pad 1: Net-(U3A-D1) -> unconnected-(U3A-D1-Pad1)
- U3 pad 10: (no net) -> /Channel Module/C2_MUTED
- U3 pad 11: (no net) -> +12V
- U3 pad 12: (no net) -> +5V
- U3 pad 13: (no net) -> GND
- U3 pad 14: (no net) -> -12V
- U3 pad 15: MUTED -> /Channel Module/C1_MUTED
- U3 pad 16: Net-(SW1-A) -> unconnected-(U3A-S1-Pad16)
- U3 pad 2: (no net) -> unconnected-(U3C-N.C.-Pad2)
- U3 pad 3: unconnected-(U3A-D3-Pad3) -> Net-(U3A-D3)
- U3 pad 4: unconnected-(U3A-S3-Pad4) -> Net-(SW3-A)
- U3 pad 5: (no net) -> Net-(SW6-A)
- U3 pad 6: (no net) -> Net-(U3B-D4)
- U3 pad 7: (no net) -> unconnected-(U3C-N.C.-Pad7)
- U3 pad 8: (no net) -> unconnected-(U3B-D2-Pad8)
- U3 pad 9: (no net) -> unconnected-(U3B-S2-Pad9)
Routing:
- net Net-(SW3-A): track 0.00 -> 22.0 mm
- net Net-(SW3-C): track 0.00 -> 21.7 mm
- net /Channel Module/C1_SOLO: track 0.00 -> 12.7 mm
- net /Channel Module/C1_MUTE: track 0.00 -> 12.5 mm
- net Net-(D1-K): track 0.00 -> 7.48 mm
- net Net-(D2-K): track 0.00 -> 7.01 mm
- net Net-(R11-Pad2): track 0.00 -> 5.95 mm
- net Net-(SW3-B): track 0.00 -> 5.22 mm
- net Net-(U2A--): track 0.00 -> 4.49 mm
- net Net-(J7-PadT): track 0.00 -> 3.82 mm
- net Net-(U3A-D3): track 0.00 -> 2.54 mm

Commit message: maybe tone after all?
Parts:
- added RV10: B100K_PAN, synth:Potentiometer_Alpha_RD902F-40-00D_Dual_Vertical_CircularHoles, F.Cu at (102.2, 98.6)
- moved RV1 64.1 mm to (215.0, 137.2)
- moved C8 55.9 mm to (142.5, 23.4)
- moved R13 55.9 mm to (154.7, 33.9)
- moved R22 55.9 mm to (154.1, 38.1)
- moved U7 55.9 mm to (142.3, 30.0)
- moved R14 55.9 mm to (150.1, 33.1)
- moved R15 55.9 mm to (150.1, 35.6)
- moved R16 55.9 mm to (131.4, 22.9)
- moved R17 55.9 mm to (131.4, 25.4)
- moved R18 55.9 mm to (131.4, 27.9)
- moved R20 55.9 mm to (135.3, 34.6)
- moved R21 55.9 mm to (135.3, 37.1)
- moved R23 55.9 mm to (135.4, 25.4)
- moved R19 55.9 mm to (130.8, 38.0)
- moved R24 55.9 mm to (130.8, 34.4)
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Routing:
- added copper zone on B.Cu, net GND
- added copper zone on F.Cu, net GND

Commit message: layed out parts
Parts:
- removed C8, C9: 100n, Capacitor_SMD:C_0603_1608Metric
- removed J15: C_BOARD_OUT_2, Connector_PinHeader_2.54mm:PinHeader_2x04_P2.54mm_Horizontal
- removed R13, R16, R19, R22, R23, R24: 100k, Resistor_SMD:R_0603_1608Metric
- removed R4: 33k, Resistor_SMD:R_0603_1608Metric
- removed the RV10 at (102.2, 98.6)
- removed U5: TL072, Package_SO:SOIC-8_3.9x4.9mm_P1.27mm
- removed U7: TL074, Package_SO:SOIC-14_3.9x8.7mm_P1.27mm
- J10: value C_BOARD_IN_1 -> C_BOARD_IN; footprint Connector_PinSocket_2.54mm:PinSocket_2x04_P2.54mm_Horizontal -> Connector_PinHeader_1.27mm:PinHeader_1x08_P1.27mm_Vertical
- J11: value C_BOARD_IN_2 -> INTERCONNECT1; footprint Connector_PinSocket_2.54mm:PinSocket_2x04_P2.54mm_Horizontal -> Connector_PinHeader_1.27mm:PinHeader_1x08_P1.27mm_Vertical; moved to F.Cu
- J12: value M_BOARD_IN_1 -> M_BOARD_IN; footprint Connector_PinSocket_2.54mm:PinSocket_2x04_P2.54mm_Horizontal -> Connector_PinSocket_1.27mm:PinSocket_1x08_P1.27mm_Vertical; moved to B.Cu
- J13: value M_BOARD_IN_2 -> INTERCONNECT2; footprint Connector_PinSocket_2.54mm:PinSocket_2x04_P2.54mm_Horizontal -> Connector_PinHeader_1.27mm:PinHeader_1x08_P1.27mm_Vertical
- J14: value C_BOARD_OUT_1 -> C_BOARD_OUT; footprint Connector_PinHeader_2.54mm:PinHeader_2x04_P2.54mm_Horizontal -> Connector_PinSocket_1.27mm:PinSocket_1x08_P1.27mm_Vertical
- R17, R18, R20, R21: value 100k -> 33k
- R3: value 33k -> 100k
- RV1: value A1M - AUX_RETURN_LEVEL -> B100K - AUX_RETURN_LEVEL
- RV10, RV6: value B100K_PAN -> A100K_PAN
- RV5, RV9: value A1M_AUX_SEND -> B1M_AUX_SEND
- U2, U3, U4, U6: moved to B.Cu
- moved J13 213.2 mm to (108.5, 26.7), turned to 180 degrees
- moved J12 151.0 mm to (138.9, 111.8)
- moved J11 141.4 mm to (92.7, 26.7), turned to 180 degrees
- moved U2 138.4 mm to (68.6, 177.5)
- moved R29 129.5 mm to (100.0, 39.9)
- moved R30 129.5 mm to (100.0, 42.4)
- moved J1 120.0 mm to (143.6, 137.5)
- moved U6 113.3 mm to (66.7, 137.7)
- moved J8 110.1 mm to (66.3, 157.2)
- moved C7 108.1 mm to (58.4, 168.1)
- moved U3 107.0 mm to (68.3, 189.2), turned to 180 degrees
- moved C5 107.0 mm to (62.0, 146.8)
- moved U4 101.4 mm to (66.7, 125.5)
- moved C6 99.2 mm to (56.9, 121.9)
- moved R14 96.3 mm to (65.2, 78.5)
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Connections:
- J10 pad 1: /Channel Module/C_MIX_IN_R -> -12V
- J10 pad 2: /Channel Module/C_MIX_IN_R -> GND
- J10 pad 3: /Channel Module/C_MIX_IN_L -> +5V
- J10 pad 4: /Channel Module/C_MIX_IN_L -> +12V
- J10 pad 5: /Channel Module/C_AUX_IN -> /Channel Module/~{GLOBAL_SOLO}
- J10 pad 6: /Channel Module/C_AUX_IN -> /Channel Module/C_BUS_AUX
- J10 pad 7: /Channel Module/~{GLOBAL_SOLO} -> /Channel Module/C_BUS_L
- J10 pad 8: /Channel Module/~{GLOBAL_SOLO} -> /Channel Module/C_BUS_R
- J11 pad 1: +12V -> Net-(J11-Pin_1)
- J11 pad 2: +12V -> Net-(J11-Pin_2)
- J11 pad 3: +5V -> Net-(J11-Pin_3)
- J11 pad 4: +5V -> Net-(J11-Pin_4)
- J11 pad 5: GND -> Net-(J11-Pin_5)
- J11 pad 6: GND -> Net-(J11-Pin_6)
- J11 pad 7: -12V -> Net-(J11-Pin_7)
- J11 pad 8: -12V -> Net-(J11-Pin_8)
- J12 pad 1: /Master Module/M_MIX_IN_R -> -12V
- J12 pad 2: /Master Module/M_MIX_IN_R -> GND
- J12 pad 3: /Master Module/M_MIX_IN_L -> +5V
- J12 pad 4: /Master Module/M_MIX_IN_L -> +12V
- J12 pad 5: /Master Module/M_AUX_IN -> /Master Module/~{GLOBAL_SOLO}
- J12 pad 7: /Master Module/~{GLOBAL_SOLO} -> /Master Module/M_MIX_IN_L
- J12 pad 8: /Master Module/~{GLOBAL_SOLO} -> /Master Module/M_MIX_IN_R
- J13 pad 1: +12V -> Net-(J11-Pin_1)
- J13 pad 2: +12V -> Net-(J11-Pin_2)
- J13 pad 3: +5V -> Net-(J11-Pin_3)
- J13 pad 4: +5V -> Net-(J11-Pin_4)
- J13 pad 5: GND -> Net-(J11-Pin_5)
- J13 pad 6: GND -> Net-(J11-Pin_6)
- J13 pad 7: -12V -> Net-(J11-Pin_7)
- J13 pad 8: -12V -> Net-(J11-Pin_8)
- J14 pad 1: /Channel Module/C_OUT_R -> -12V
- J14 pad 2: /Channel Module/C_OUT_R -> GND
- J14 pad 3: /Channel Module/C_OUT_L -> +5V
- J14 pad 4: /Channel Module/C_OUT_L -> +12V
- J14 pad 5: /Channel Module/C_AUX_OUT -> /Channel Module/~{GLOBAL_SOLO}
- J14 pad 6: /Channel Module/C_AUX_OUT -> /Channel Module/C_BUS_AUX
- J14 pad 7: /Channel Module/~{GLOBAL_SOLO} -> /Channel Module/C_BUS_L
- J14 pad 8: /Channel Module/~{GLOBAL_SOLO} -> /Channel Module/C_BUS_R
- J2 pad T: /Master Module/M_AUX_IN -> Net-(J2-PadT)
- R14 pad 2: Net-(U7C--) -> /Channel Module/C_BUS_AUX
- R15 pad 2: Net-(U7C--) -> /Channel Module/C_BUS_AUX
- R17 pad 2: Net-(U7A--) -> /Channel Module/C_BUS_R
- R18 pad 2: Net-(U7A--) -> /Channel Module/C_BUS_R
- R2 pad 1: Net-(U1B--) -> Net-(R2-Pad1)
- R2 pad 2: Net-(U1D--) -> /Master Module/M_MIX_IN_R
- R20 pad 2: Net-(U7B--) -> /Channel Module/C_BUS_L
- R21 pad 2: Net-(U7B--) -> /Channel Module/C_BUS_L
- R3 pad 1: /Master Module/M_MIX_IN_R -> /Master Module/M_AUX_IN
- R3 pad 2: Net-(U1D--) -> Net-(J2-PadT)
- R5 pad 1: Net-(U1A--) -> Net-(R5-Pad1)
- R5 pad 2: Net-(U1C--) -> /Master Module/M_MIX_IN_L
- RV1 pad 2: Net-(U1A-+) -> Net-(R5-Pad1)
- RV1 pad 5: Net-(U1B-+) -> Net-(R2-Pad1)
- RV2 pad 1: Net-(U1D--) -> /Master Module/M_MIX_IN_R
- RV2 pad 4: Net-(U1C--) -> /Master Module/M_MIX_IN_L
- RV5 pad 2: Net-(U5A-+) -> /Channel Module/Channel1/C_AUX_OUT
- RV9 pad 2: Net-(U5B-+) -> /Channel Module/Channel2/C_AUX_OUT
- U1 pad 1: Net-(U1A--) -> Net-(J2-PadT)
- U1 pad 13: Net-(U1D--) -> /Master Module/M_MIX_IN_R
- U1 pad 2: Net-(U1A--) -> /Master Module/M_AUX_IN
- U1 pad 3: Net-(U1A-+) -> GND
- U1 pad 5: Net-(U1B-+) -> (no net)
- U1 pad 6: Net-(U1B--) -> (no net)
- U1 pad 7: Net-(U1B--) -> (no net)
- U1 pad 9: Net-(U1C--) -> /Master Module/M_MIX_IN_L
Routing:
- net Net-(SW3-A): track 22.0 -> 0.00 mm
- net Net-(SW3-C): track 21.7 -> 0.00 mm
- net Net-(J11-Pin_8): track 0.00 -> 15.7 mm
- net Net-(J11-Pin_7): track 0.00 -> 15.7 mm
- net Net-(J11-Pin_6): track 0.00 -> 15.7 mm
- net Net-(J11-Pin_5): track 0.00 -> 15.7 mm
- net Net-(J11-Pin_4): track 0.00 -> 15.7 mm
- net Net-(J11-Pin_3): track 0.00 -> 15.7 mm
- net Net-(J11-Pin_2): track 0.00 -> 15.7 mm
- net Net-(J11-Pin_1): track 0.00 -> 15.7 mm
- net /Channel Module/C1_SOLO: track 12.7 -> 0.00 mm
- net /Channel Module/C1_MUTE: track 12.5 -> 0.00 mm
- net Net-(D1-K): track 7.48 -> 0.00 mm
- net Net-(D2-K): track 7.01 -> 0.00 mm
- net Net-(R11-Pad2): track 5.95 -> 0.00 mm
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Other:
- board outline added: 80.8 x 144.5 mm

Commit message: layout master board
Parts:
- C5, C6, C7, J8, R12, R14, R15, R17, R18, R20, R21, R25, R26, R27, R28, R29, R30, R31: moved to B.Cu
- J10: footprint Connector_PinHeader_1.27mm:PinHeader_1x08_P1.27mm_Vertical -> Connector_PinSocket_1.27mm:PinSocket_1x08_P1.27mm_Vertical
- RV4, RV8: footprint Potentiometer_THT:Potentiometer_Bourns_PTA3043_Single_Slide -> _project:Potentiometer_Bourns_PTA3043_Single_Slide
- moved R28 191.4 mm to (-22.2, 25.4)
- moved R27 187.5 mm to (-22.2, 27.9)
- moved R26 183.6 mm to (-22.2, 30.4)
- moved R25 179.8 mm to (-22.2, 33.0)
- moved C7 172.0 mm to (-51.2, 35.6)
- moved R1 169.9 mm to (141.7, 133.1), turned to 90 degrees
- moved R29 169.6 mm to (-18.5, 161.3)
- moved R30 166.1 mm to (-18.5, 158.8)
- moved J8 165.4 mm to (-88.1, 97.9)
- moved U2 159.1 mm to (-89.1, 156.2)
- moved U3 159.1 mm to (-89.4, 167.9)
- moved U6 155.3 mm to (-88.4, 129.5)
- moved U4 153.2 mm to (-85.9, 111.8)
- moved C5 150.3 mm to (-56.5, 54.4)
- moved R11 149.1 mm to (-59.2, 36.1)
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Routing:
- net Net-(J6-PadT): track 0.00 -> 117.1 mm, vias 0 -> 1
- net Net-(J5-PadT): track 0.00 -> 109.6 mm, vias 0 -> 1
- net /Master Module/M_MIX_IN_L: track 0.00 -> 76.0 mm, vias 0 -> 1
- net +12V: track 0.00 -> 69.0 mm, vias 0 -> 2
- net Net-(J2-PadT): track 0.00 -> 62.8 mm
- net -12V: track 0.00 -> 55.9 mm, vias 0 -> 2
- net +5V: track 0.00 -> 49.6 mm, vias 0 -> 1
- net /Master Module/M_AUX_IN: track 0.00 -> 38.7 mm
- net /Master Module/AUX_RETURN_L: track 0.00 -> 37.1 mm, vias 0 -> 1
- net /Master Module/M_MIX_IN_R: track 0.00 -> 34.2 mm, vias 0 -> 1
- net /Master Module/AUX_RETURN_R: track 0.00 -> 28.7 mm, vias 0 -> 1
- net /Master Module/~{GLOBAL_SOLO}: track 0.00 -> 28.5 mm
- net Net-(R5-Pad1): track 0.00 -> 15.6 mm
- net Net-(R2-Pad1): track 0.00 -> 10.4 mm
- net GND: track 0.00 -> 10.0 mm, vias 0 -> 5
- added copper zone on In1.Cu, net GND
- removed copper zone on B.Cu, net GND
- removed copper zone on F.Cu, net GND
Other:
- copper layers 2 -> 4

Commit message: first pass route
Parts:
- added C10: 100n, Capacitor_SMD:C_0603_1608Metric, B.Cu at (78.9, 120.0)
- added C8: 100n, Capacitor_SMD:C_0603_1608Metric, B.Cu at (78.9, 123.1)
- added C9: 100n, Capacitor_SMD:C_0603_1608Metric, B.Cu at (78.9, 117.0)
- added Q1: BSS214NW, Package_TO_SOT_SMD:SOT-323_SC-70, B.Cu at (90.8, 138.7)
- moved U2 191.7 mm to (99.6, 122.0), turned to 180 degrees
- moved U4 186.9 mm to (99.5, 135.1), turned to 180 degrees
- moved C7 184.1 mm to (99.5, 141.2), turned to 180 degrees
- moved U3 181.0 mm to (84.8, 118.9)
- moved J8 178.0 mm to (87.1, 128.8)
- moved R28 175.9 mm to (99.1, 152.9), turned to 90 degrees
- moved R26 174.5 mm to (102.1, 152.9), turned to 90 degrees
- moved U6 173.3 mm to (84.8, 134.6)
- moved R27 169.9 mm to (93.0, 152.9), turned to 90 degrees
- moved R25 168.4 mm to (96.0, 152.9), turned to 90 degrees
- moved R7 162.5 mm to (89.9, 152.9), turned to 90 degrees
- moved R18 160.3 mm to (103.9, 114.8), turned to 90 degrees
- moved R9 159.4 mm to (86.9, 152.9), turned to 90 degrees
- moved C5 159.1 mm to (78.7, 138.2), turned to 180 degrees
- moved C6 158.1 mm to (99.6, 128.0), turned to 180 degrees
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Connections:
- R10 pad 2: Net-(U2A--) -> Net-(U4D--)
- R11 pad 1: Net-(U2A--) -> Net-(U4D--)
- R29 pad 2: Net-(U2C--) -> Net-(U4A--)
- R30 pad 1: Net-(U2C--) -> Net-(U4A--)
- RV10 pad 2: Net-(U4D-+) -> Net-(U2A-+)
- RV10 pad 5: Net-(U4C-+) -> Net-(U2B-+)
- RV4 pad 2: Net-(U2B-+) -> Net-(U4C-+)
- RV6 pad 2: Net-(U4B-+) -> Net-(U2D-+)
- RV6 pad 5: Net-(U4A-+) -> Net-(U2C-+)
- RV8 pad 2: Net-(U2D-+) -> Net-(U4B-+)
- U2 pad 1: Net-(U3A-D3) -> /Channel Module/Channel2/C_PAN_L
- U2 pad 10: GND -> Net-(U2C-+)
- U2 pad 13: Net-(SW6-C) -> /Channel Module/Channel1/C_PAN_L
- U2 pad 14: Net-(SW6-C) -> /Channel Module/Channel1/C_PAN_L
- U2 pad 2: Net-(U2A--) -> /Channel Module/Channel2/C_PAN_L
- U2 pad 3: GND -> Net-(U2A-+)
- U2 pad 6: Net-(SW3-C) -> /Channel Module/Channel2/C_PAN_R
- U2 pad 7: Net-(SW3-C) -> /Channel Module/Channel2/C_PAN_R
- U2 pad 8: Net-(U3B-D4) -> /Channel Module/Channel1/C_PAN_R
- U2 pad 9: Net-(U2C--) -> /Channel Module/Channel1/C_PAN_R
- U4 pad 1: /Channel Module/Channel1/C_PAN_R -> Net-(U3B-D4)
- U4 pad 12: Net-(U4D-+) -> GND
- U4 pad 13: /Channel Module/Channel2/C_PAN_L -> Net-(U4D--)
- U4 pad 14: /Channel Module/Channel2/C_PAN_L -> Net-(U3A-D3)
- U4 pad 2: /Channel Module/Channel1/C_PAN_R -> Net-(U4A--)
- U4 pad 3: Net-(U4A-+) -> GND
- U4 pad 6: /Channel Module/Channel1/C_PAN_L -> Net-(SW6-C)
- U4 pad 7: /Channel Module/Channel1/C_PAN_L -> Net-(SW6-C)
- U4 pad 8: /Channel Module/Channel2/C_PAN_R -> Net-(SW3-C)
- U4 pad 9: /Channel Module/Channel2/C_PAN_R -> Net-(SW3-C)
Routing:
- net +5V: track 49.6 -> 203.1 mm, vias 1 -> 4
- net +12V: track 69.0 -> 178.4 mm, vias 2 -> 5
- net Net-(U3A-D3): track 0.00 -> 85.3 mm, vias 0 -> 2
- net Net-(U4A--): track 0.00 -> 84.9 mm, vias 0 -> 2
- net Net-(U3B-D4): track 0.00 -> 83.5 mm, vias 0 -> 1
- net Net-(U4D--): track 0.00 -> 79.2 mm, vias 0 -> 2
- net -12V: track 55.9 -> 125.1 mm, vias 2 -> 5
- net Net-(SW3-C): track 0.00 -> 68.7 mm, vias 0 -> 1
- net Net-(SW6-C): track 0.00 -> 65.6 mm, vias 0 -> 1
- net /Channel Module/~{GLOBAL_SOLO}: track 0.00 -> 55.3 mm, vias 0 -> 1
- net /Channel Module/C2_SOLO: track 0.00 -> 46.0 mm, vias 0 -> 1
- net Net-(SW6-A): track 0.00 -> 43.6 mm, vias 0 -> 1
- net /Channel Module/C2_SOLO_LED: track 0.00 -> 42.6 mm, vias 0 -> 2
- net /Channel Module/C_BUS_R: track 0.00 -> 40.4 mm
- net Net-(SW3-A): track 0.00 -> 40.0 mm
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Other:
- board text added: "2x OP-AMP"
- board text added: "6 OP-AMP"

Commit message: cleanup 1
Parts:
- moved R12 3.74 mm to (81.8, 111.5), turned to 90 degrees
Routing:
- net Net-(U3A-D3): track 85.3 -> 130.1 mm
- net +5V: track 203.1 -> 186.0 mm
- net GND: track 37.1 -> 22.6 mm, vias 14 -> 20
- net /Channel Module/C2_SOLO_LED: track 42.6 -> 46.2 mm
- net Net-(U4C-+): track 16.0 -> 19.1 mm
- net /Channel Module/C1_SOLO: track 23.9 -> 26.7 mm, vias 2 -> 1
- net /Channel Module/C1_MUTE: track 28.0 -> 25.5 mm, vias 1 -> 0
- net /Channel Module/C1_MUTED: track 23.3 -> 25.6 mm
- net Net-(U3B-D4): track 83.5 -> 81.3 mm
- net Net-(U2C-+): track 36.9 -> 35.0 mm
- net /Channel Module/~{GLOBAL_SOLO}: track 55.3 -> 56.3 mm
- net /Channel Module/C_BUS_R: track 40.4 -> 41.4 mm
- net /Channel Module/C_BUS_L: track 30.4 -> 31.4 mm
- net /Channel Module/C2_SOLO: track 46.0 -> 45.0 mm
- net Net-(U4A--): track 84.9 -> 84.1 mm
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- added copper zone on B.Cu, net GND
- added copper zone on F.Cu, net GND
- added copper zone on In2.Cu, net GND
Other:
- board text removed: "2x OP-AMP"
- board text removed: "6 OP-AMP"

Commit message: cleanup 2
Parts:
- moved R5 13.1 mm to (142.2, 97.0)
- moved R2 2.59 mm to (139.2, 97.0)
- moved Q1 1.80 mm to (90.9, 136.9)
Routing:
- net /Master Module/M_MIX_IN_R: track 34.2 -> 53.3 mm
- net /Master Module/M_MIX_IN_L: track 75.4 -> 58.1 mm
- net /Master Module/M_AUX_IN: track 33.9 -> 45.0 mm
- net /Master Module/AUX_RETURN_R: track 28.7 -> 36.4 mm, vias 1 -> 0
- net Net-(J2-PadT): track 61.5 -> 67.6 mm
- net Net-(R5-Pad1): track 15.6 -> 9.86 mm
- net Net-(U4B-+): track 12.0 -> 16.3 mm
- net GND: track 22.6 -> 18.5 mm, vias 20 -> 21
- net /Channel Module/Channel1/C_AUX_OUT: track 12.6 -> 8.72 mm, vias 1 -> 0
- net Net-(U3A-D3): track 130.1 -> 133.5 mm
- net +12V: track 178.4 -> 181.5 mm
- net /Master Module/AUX_RETURN_L: track 37.1 -> 34.2 mm, vias 1 -> 0
- net /Channel Module/~{GLOBAL_SOLO}: track 56.3 -> 58.9 mm
- net /Channel Module/C1_SOLO_LED: track 28.8 -> 31.1 mm
- net /Channel Module/C_BUS_R: track 41.4 -> 43.6 mm
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Other:
- board text added: "+"
