File: mixer/mixer.kicad_pcb (KiCad board)
At the start: 4 copper layers, 80.8 x 144.5 mm, 74 parts, among them J1 EURORACK_CONN_16, J10 C_BOARD_IN, J11 INTERCONNECT1, J12 M_BOARD_IN, J13 INTERCONNECT2, J14 C_BOARD_OUT, J2 AUX_OUT, J3 AUX_IN_R, J4 AUX_IN_L, J5 MAIN_OUT_R, J6 MAIN_OUT_L, J7 CHANNEL_IN, J8 AVR-ISP-6, J9 CHANNEL_IN, Q1 BSS214NW, SW1 MUTE_PBSW, SW2 SOLO_PBSW, SW3 AUX_PRE_POST_FADER_SLIDESW, SW4 MUTE_PBSW, SW5 SOLO_PBSW, SW6 AUX_PRE_POST_FADER_SLIDESW, U1 TL074, U2 TL074, U3 DG403, U4 TL074, U6 ATtiny24-20SS

Commit message: start on panel
Parts:
- added FID10: C_MUTE_1, _project:MUTE_CUTOUT, F.Cu at (29.2, 159.0)
- added FID11: C_SOLO_2, _project:SOLO_CUTOUT, F.Cu at (52.1, 159.0)
- added FID12: C_MUTE_2, _project:MUTE_CUTOUT, F.Cu at (44.5, 159.0)
- added FID5: C_BTN1, synth:toggle_sw_hole, F.Cu at (29.2, 152.7)
- added FID6: C_BTN2, synth:toggle_sw_hole, F.Cu at (36.8, 152.7)
- added FID7: C_BTN3, synth:toggle_sw_hole, F.Cu at (44.5, 152.7)
- added FID8: C_BTN4, synth:toggle_sw_hole, F.Cu at (52.1, 152.7)
- added FID9: C_SOLO_1, _project:SOLO_CUTOUT, F.Cu at (36.8, 159.0)
- added J15: C_IN1, synth:thonkiconn_hole, F.Cu at (30.5, 57.4)
- added J16: C_IN2, synth:thonkiconn_hole, F.Cu at (50.8, 57.4)
- added J17: C_AUXSEND1, synth:knob_hole, F.Cu at (33.0, 70.6)
- added J18: C_PAN1, synth:knob_hole, F.Cu at (33.0, 90.4)
- added J19: C_AUXSEND2, synth:knob_hole, F.Cu at (48.3, 70.6)
- added J20: C_PAN2, synth:knob_hole, F.Cu at (48.3, 90.4)
- added J21: M_OUT_L, synth:thonkiconn_hole, F.Cu at (199.4, 56.4)
- added J22: M_AUXSEND, synth:thonkiconn_hole, F.Cu at (199.4, 76.7)
- added J23: M_AUX_AMOUNT, synth:knob_hole, F.Cu at (199.4, 88.9)
- added J24: M_OUT_R, synth:thonkiconn_hole, F.Cu at (199.4, 66.5)
- added J25: M_AUX_RETURN_L, synth:thonkiconn_hole, F.Cu at (199.4, 101.6)
- added J26: M_AUX_RETURN_L, synth:thonkiconn_hole, F.Cu at (199.4, 111.8)
- added J27: M_MASTER, synth:knob_hole, F.Cu at (199.4, 124.5)
Routing:
- net /Master Module/M_MIX_IN_L: track 58.1 -> 56.7 mm
- net Net-(J6-PadT): track 117.0 -> 115.8 mm
Other:
- board size 80.8 x 144.5 mm -> 182.9 x 154.9 mm

Commit message: rework master board for space and symmetry
Parts:
- C1, C2, C3, C4, R1, R2, R3, R5, U1: moved to B.Cu
- moved R2 26.6 mm to (154.7, 118.6)
- moved R5 23.9 mm to (152.4, 118.6)
- moved J23 18.3 mm to (198.1, 107.2)
- moved RV1 18.3 mm to (147.3, 107.2), turned to 90 degrees
- moved C1 18.0 mm to (152.4, 144.8), turned to 0 degrees
- moved J26 15.0 mm to (198.1, 96.8)
- moved J3 15.0 mm to (147.3, 96.8)
- moved J25 15.0 mm to (198.1, 86.6)
- moved J4 15.0 mm to (147.3, 86.6)
- moved R1 14.5 mm to (140.5, 118.6)
- moved R3 12.5 mm to (156.0, 144.5), turned to 90 degrees
- moved C2 11.7 mm to (152.4, 142.0), turned to 0 degrees
- moved C4 10.4 mm to (152.4, 147.6), turned to 180 degrees
- moved U1 10.4 mm to (152.4, 153.7), turned to 180 degrees
- moved C3 7.62 mm to (152.4, 139.2), turned to 180 degrees
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Connections:
- RV1 pad 2: Net-(R5-Pad1) -> Net-(R2-Pad1)
- RV1 pad 3: /Master Module/AUX_RETURN_L -> /Master Module/AUX_RETURN_R
- RV1 pad 5: Net-(R2-Pad1) -> Net-(R5-Pad1)
- RV1 pad 6: /Master Module/AUX_RETURN_R -> /Master Module/AUX_RETURN_L
Routing:
- net /Master Module/M_MIX_IN_R: track 53.3 -> 79.2 mm, vias 1 -> 2
- net /Master Module/M_MIX_IN_L: track 56.7 -> 78.9 mm, vias 1 -> 3
- net /Master Module/M_AUX_IN: track 45.0 -> 64.9 mm, vias 0 -> 2
- net /Master Module/AUX_RETURN_R: track 36.4 -> 18.9 mm
- net /Master Module/~{GLOBAL_SOLO}: track 28.5 -> 11.5 mm
- net Net-(J6-PadT): track 115.8 -> 103.7 mm
- net /Master Module/AUX_RETURN_L: track 34.2 -> 46.2 mm
- net Net-(J2-PadT): track 67.6 -> 76.7 mm, vias 0 -> 1
- net -12V: track 125.1 -> 132.6 mm
- net Net-(J5-PadT): track 109.6 -> 103.1 mm
- net +5V: track 187.1 -> 193.0 mm, vias 4 -> 5
- net Net-(R5-Pad1): track 9.86 -> 7.09 mm
- net Net-(R2-Pad1): track 9.77 -> 12.2 mm
Other:
- outline, holes or cut-outs redrawn

Commit message: rework channel board for space
Parts:
- moved R14 11.4 mm to (89.7, 85.1)
- moved R15 11.4 mm to (92.7, 85.1)
- moved J18 6.10 mm to (33.0, 96.5)
- moved J20 6.10 mm to (48.3, 96.5)
- moved RV10 6.10 mm to (99.1, 96.5), turned to -90 degrees
- moved RV6 6.10 mm to (83.8, 96.5), turned to -90 degrees
Routing:
- net Net-(U3A-D3): track 133.5 -> 88.8 mm
- net Net-(U2B-+): track 24.9 -> 39.8 mm
- net Net-(U2C-+): track 35.0 -> 48.0 mm, vias 2 -> 1
- net Net-(U2D-+): track 29.4 -> 41.5 mm, vias 3 -> 1
- net Net-(U2A-+): track 24.8 -> 33.7 mm
- net /Channel Module/Channel2/C_AUX_OUT: track 20.4 -> 11.6 mm
- net Net-(SW6-A): track 43.6 -> 46.7 mm
- net /Channel Module/Channel1/C_AUX_OUT: track 8.72 -> 11.1 mm
- net /Channel Module/C_BUS_AUX: track 38.2 -> 40.3 mm, vias 0 -> 2
- net /Channel Module/~{GLOBAL_SOLO}: track 58.9 -> 58.1 mm
- net Net-(SW3-A): track 40.7 -> 40.0 mm
- net Net-(U3B-D4): track 81.3 -> 82.0 mm, vias 1 -> 2
- net /Channel Module/Channel1/C_PAN_R: track 13.6 -> 13.9 mm, vias 0 -> 2

Commit message: panel design
Parts:
- moved J3 10.2 mm to (147.3, 86.6)
- moved J4 10.2 mm to (147.3, 96.8)
Connections:
- J3 pad TN: /Master Module/AUX_RETURN_L -> GND
- J4 pad TN: GND -> /Master Module/AUX_RETURN_R
Routing:
- net /Master Module/AUX_RETURN_R: track 18.9 -> 43.0 mm
- net /Master Module/AUX_RETURN_L: track 46.2 -> 22.7 mm
Other:
- outline, holes or cut-outs redrawn
Changed lines of the file:
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@@
 		(sheetname "/Panel/")
 		(sheetfile "panel.kicad_sch")
-		(attr through_hole allow_missing_courtyard)
+		(attr through_hole exclude_from_bom allow_missing_courtyard)
 		(fp_circle
 			(center 0 0)
@@
 		(locked yes)
 		(layer "F.Cu")
-		(at 147.32 96.774 90)
+		(at 147.32 86.614 90)
 		(descr "TRS 3.5mm, vertical, Thonkiconn, PCB mount, (http://www.qingpu-electronics.com/en/products/WQP-PJ398SM-362.html)")
 		(tags "WQP-PJ398SM WQP-PJ301M-12 TRS 3.5mm mono vertical jack thonkiconn qingpu")
@@
 			(layers "*.Cu" "*.Mask")
 			(remove_unused_layers no)
-			(net 25 "/Master Module/AUX_RETURN_L")
+			(net 1 "GND")
 			(pintype "passive")
 		)
@@
 		(sheetname "/Panel/")
 		(sheetfile "panel.kicad_sch")
-		(attr through_hole allow_missing_courtyard)
+		(attr through_hole exclude_from_bom allow_missing_courtyard)
 		(fp_circle
 			(center 0 0)
@@
 		(sheetname "/Panel/")
 		(sheetfile "panel.kicad_sch")
-		(attr through_hole allow_missing_courtyard)
+		(attr through_hole exclude_from_bom allow_missing_courtyard)
 		(fp_circle
 			(center 0 0)
@@
 		(sheetname "/Panel/")
 		(sheetfile "panel.kicad_sch")
-		(attr through_hole allow_missing_courtyard)
+		(attr through_hole exclude_from_bom allow_missing_courtyard)
 		(fp_circle
 			(center 0 0)
@@
 		(locked yes)
 		(layer "F.Cu")
-		(at 147.32 86.614 90)
+		(at 147.32 96.774 90)
 		(descr "TRS 3.5mm, vertical, Thonkiconn, PCB mount, (http://www.qingpu-electronics.com/en/products/WQP-PJ398SM-362.html)")
 		(tags "WQP-PJ398SM WQP-PJ301M-12 TRS 3.5mm mono vertical jack thonkiconn qingpu")
@@
 			(layers "*.Cu" "*.Mask")
 			(remove_unused_layers no)
-			(net 1 "GND")
+			(net 26 "/Master Module/AUX_RETURN_R")
 			(pintype "passive")
 		)
@@
 	(gr_rect
 		(start 137.414 51.054)
-		(end 157.226 160.782)
+		(end 157.226 160.655)
 		(stroke
 			(width 0.05)
@@
 		)
 		(fill no)
-		(locked yes)
 		(layer "Edge.Cuts")
 	)
 	(gr_rect
-		(start 47.518 109.468)
-		(end 50.018 140.468)
+		(start 46.248 109.468)
+		(end 50.272 140.468)
 		(stroke
 			(width 0.1)
@@
 	(gr_rect
 		(start 76.454 51.054)
-		(end 106.426 160.782)
+		(end 106.426 160.655)
 		(stroke
 			(width 0.05)
@@
 		)
 		(fill no)
-		(locked yes)
 		(layer "Edge.Cuts")
 	)
@@
 	)
 	(gr_rect
-		(start 32.532 109.468)
+		(start 31.008 109.468)
 		(end 35.032 140.468)
 		(stroke
@@
 	)
 	(gr_rect
-		(start 187.96 41.656)
+		(start 187.96 42.672)
 		(end 208.28 170.18)
 		(stroke
@@
 	(gr_rect
 		(start 137.16 50.8)
-		(end 157.508 161)
+		(end 157.508 160.8)
 		(stroke
 			(width 0.1)
@@
 		)
 		(fill no)
-		(locked yes)
 		(layer "User.1")
 	)
@@
 		)
 		(fill no)
-		(locked yes)
 		(layer "User.1")
 	)
 	(gr_rect
 		(start 76.2 50.8)
-		(end 106.68 160.8328)
+		(end 106.68 160.8)
 		(stroke
 			(width 0.1)
@@
 		)
 		(fill no)
-		(locked yes)
 		(layer "User.1")
 	)
 	(gr_rect
-		(start 187.96 41.65)
-		(end 208.308 170.15)
+		(start 25.4 41.541)
+		(end 55.88 170.041)
 		(stroke
 			(width 0.1)
@@
 	)
 	(gr_rect
-		(start 25.4 42.684)
-		(end 55.88 171.184)
+		(start 187.946 41.541)
+		(end 208.294 170.041)
+		(stroke
+			(width 0.1)
+			(type solid)
+		)
+		(fill no)
+		(layer "User.1")
+	)
+	(gr_rect
+		(start 187.96 50.8)
+		(end 208.308 160.8)
 		(stroke
 			(width 0.1)
@@
 		)
 		(fill no)
-		(locked yes)
 		(layer "User.1")
 	)
@@
 			(type default)
 		)
-		(locked yes)
 		(layer "User.3")
 	)
@@
 	)
 	(segment
-		(start 149.82 117.188)
-		(end 148.546 115.914)
+		(start 151.384 115.624)
+		(end 151.384 112.903)
 		(width 0.25)
 		(layer "F.Cu")
@@
 	)
 	(segment
-		(start 148.546 90.308)
-		(end 152.24 86.614)
+		(start 149.86 99.154)
+		(end 152.24 96.774)
 		(width 0.25)
 		(layer "F.Cu")
@@
 	)
 	(segment
-		(start 148.546 115.914)
-		(end 148.546 90.308)
+		(start 149.86 111.379)
+		(end 149.86 99.154)
 		(width 0.25)
 		(layer "F.Cu")
@@
 	)
 	(segment
-		(start 143.94 94.914)
-		(end 152.24 86.614)
+		(start 149.82 117.188)
+		(end 151.384 115.624)
 		(width 0.25)
-		(layer "B.Cu")
+		(layer "F.Cu")
 		(net 25)
 	)
 	(segment
-		(start 143.94 96.774)
-		(end 143.94 94.914)
+		(start 151.384 112.903)
+		(end 149.86 111.379)
 		(width 0.25)
-		(layer "B.Cu")
+		(layer "F.Cu")
 		(net 25)
 	)
 	(segment
-		(start 149.82 99.194)
-		(end 152.24 96.774)
+		(start 149.479 89.375)
+		(end 152.24 86.614)
+		(width 0.25)
+		(layer "F.Cu")
+		(net 26)
+	)
+	(segment
+		(start 149.479 114.347)
+		(end 149.479 89.375)
 		(width 0.25)
 		(layer "F.Cu")
@@
 	(segment
 		(start 149.82 114.688)
-		(end 149.82 99.194)
+		(end 149.479 114.347)
 		(width 0.25)
 		(layer "F.Cu")
@@
 	)
 	(segment
+		(start 143.94 96.774)
+		(end 143.94 94.914)
+		(width 0.25)
+		(layer "B.Cu")
+		(net 26)
+	)
+	(segment
+		(start 143.94 94.914)
+		(end 152.24 86.614)
+		(width 0.25)
+		(layer "B.Cu")
+		(net 26)
+	)
+	(segment
 		(start 143.002 117.976)
 		(end 144.82 119.794)
@@
 		(net 1)
 		(net_name "GND")
-		(layer "F.Cu")
+		(layers "F.Cu" "B.Cu" "In1.Cu" "In2.Cu")
 		(hatch edge 0.5)
-		(priority 1)
 		(connect_pads
 			(clearance 0.2)
 		)
-		(min_thickness 0.25)
+		(min_thickness 0.2)
 		(filled_areas_thickness no)
 		(fill yes
-			(thermal_gap 0.5)
-			(thermal_bridge_width 0.5)
+			(thermal_gap 0.2)
+			(thermal_bridge_width 0.2)
 		)
 		(polygon
 			(pts
-				(xy 25.4 171.196) (xy 55.88 171.196) (xy 55.88 42.672) (xy 25.4 42.672)
+				(xy 76.2 50.8) (xy 106.68 50.8) (xy 106.68 160.782) (xy 76.2 160.782)
 			)
 		)
@@
 		(layers "F.Cu" "B.Cu" "In1.Cu" "In2.Cu")
 		(hatch edge 0.5)
+		(priority 2)
 		(connect_pads
 			(clearance 0.2)
@@
 		(polygon
 			(pts
-				(xy 76.2 50.8) (xy 106.68 50.8) (xy 106.68 160.782) (xy 76.2 160.782)
+				(xy 137.16 50.8) (xy 157.48 50.8) (xy 157.48 160.782) (xy 137.16 160.782)
 			)
 		)
@@
 		(net 1)
 		(net_name "GND")
-		(layers "F.Cu" "B.Cu" "In1.Cu" "In2.Cu")
+		(layer "B.Cu")
 		(hatch edge 0.5)
-		(priority 2)
+		(priority 1)
 		(connect_pads
 			(clearance 0.2)
 		)
-		(min_thickness 0.2)
+		(min_thickness 0.25)
 		(filled_areas_thickness no)
 		(fill yes
-			(thermal_gap 0.2)
-			(thermal_bridge_width 0.2)
+			(thermal_gap 0.5)
+			(thermal_bridge_width 0.5)
 		)
 		(polygon
 			(pts
-				(xy 137.16 50.8) (xy 157.48 50.8) (xy 157.48 161.036) (xy 137.16 161.036)
+				(xy 187.96 170.18) (xy 208.28 170.18) (xy 208.28 42.672) (xy 187.96 42.672)
+			)
+		)
+	)
+	(zone
+		(net 1)
+		(net_name "GND")
+		(layer "B.Cu")
+		(hatch edge 0.5)
+		(priority 1)
+		(connect_pads
+			(clearance 0.2)
+		)
+		(min_thickness 0.25)
+		(filled_areas_thickness no)
+		(fill yes
+			(thermal_gap 0.5)
+			(thermal_bridge_width 0.5)
+		)
+		(polygon
+			(pts
+				(xy 25.4 171.196) (xy 55.88 171.196) (xy 55.88 42.672) (xy 25.4 42.672)
 			)
 		)

Commit message: place screws
Parts:
- added FID1: C_SCREW_B, synth:eurorack_screw_hole, F.Cu at (40.6, 166.0)
- added FID2: C_SCREW_T, synth:eurorack_screw_hole, F.Cu at (40.6, 45.5)
- added FID3: M_SCREW_T, synth:eurorack_screw_hole, F.Cu at (198.1, 45.5)
- added FID4: M_SCREW_B, synth:eurorack_screw_hole, F.Cu at (198.1, 166.0)
Other:
- board size 182.9 x 154.9 mm -> 182.9 x 153.8 mm
- board text added: "TODO: confirm all cutout sizes"

Commit message: update graphics
Parts:
- FID10, FID12: footprint _project:MUTE_CUTOUT -> _project:MUTE_CUTOUT_ALT
- FID11, FID9: footprint _project:SOLO_CUTOUT -> _project:SOLO_CUTOUT_ALT
Other:
- board text added: "TODO: fix graphics alignment"
- board text added: "TODO: run final drc"
