File: mixer/master.kicad_sch (KiCad schematic)
At the start: 14 parts, among them J1 AUX_OUT, J2 AUX_IN_R, J3 AUX_IN_L, J4 MAIN_OUT_R, J5 MAIN_OUT_L, U1 TL074

Commit message: working out some parts
Parts:
- removed RV1: A100K_MASTER_FADER_R, symbol Device:R_Potentiometer
- removed RV3: A100K_MASTER_FADER_L, symbol Device:R_Potentiometer
- added RV7: A100K_MASTER_FADER, synth:Potentiometer_Alpha_RD902F-40-00D_Dual_Vertical_CircularHoles, symbol Device:R_Potentiometer_Dual_Separate
- RV2: footprint Potentiometer_THT:Potentiometer_Alpha_RD902F-40-00D_Dual_Vertical -> synth:Potentiometer_Alpha_RD902F-40-00D_Dual_Vertical_CircularHoles
Connections:
- net at J5.T, U1.8: now also RV7.5, RV7.6
- net at R3.2, R4.2, U1.9 (-): now also RV7.4
- net at R1.2, R2.2, U1.13 (-): now also RV7.1
- net at J4.T, U1.14: now also RV7.2, RV7.3
Changed lines of the file:
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@@
 			)
 		)
-		(property "Footprint" "Potentiometer_THT:Potentiometer_Alpha_RD902F-40-00D_Dual_Vertical"
+		(property "Footprint" "synth:Potentiometer_Alpha_RD902F-40-00D_Dual_Vertical_CircularHoles"
 			(at 72.39 133.35 0)
 			(effects
@@
 	)
 	(symbol
-		(lib_id "Device:R_Potentiometer")
-		(at 128.27 125.73 90)
-		(unit 1)
-		(exclude_from_sim no)
-		(in_bom yes)
-		(on_board yes)
-		(dnp no)
-		(property "Reference" "RV3"
-			(at 128.27 128.016 90)
-			(effects
-				(font
-					(size 1.27 1.27)
-				)
-			)
-		)
-		(property "Value" "A100K_MASTER_FADER_L"
-			(at 128.27 130.556 90)
-			(effects
-				(font
-					(size 1.27 1.27)
-				)
-			)
-		)
-		(property "Footprint" ""
-			(at 128.27 125.73 0)
-			(effects
-				(font
-					(size 1.27 1.27)
-				)
-				(hide yes)
-			)
-		)
-		(property "Datasheet" "~"
-			(at 128.27 125.73 0)
-			(effects
-				(font
-					(size 1.27 1.27)
-				)
-				(hide yes)
-			)
-		)
-		(property "Description" "Potentiometer"
-			(at 128.27 125.73 0)
-			(effects
-				(font
-					(size 1.27 1.27)
-				)
-				(hide yes)
-			)
-		)
-		(pin "3"
-		)
-		(pin "2"
-		)
-		(pin "1"
-		)
-		(instances
-			(project "mixer"
-				(path "/7887173d-29cc-4936-b1a7-ffeb730ae153/33e847a2-c80a-4a2a-9bd4-e640d7127b7a"
-					(reference "RV3")
-					(unit 1)
-				)
-			)
-		)
-	)
-	(symbol
 		(lib_id "synth:AudioJack_SwitchT")
 		(at 60.96 36.83 0)
@@
 					(reference "U1")
 					(unit 2)
-				)
-			)
-		)
-	)
-	(symbol
-		(lib_id "Device:R_Potentiometer")
-		(at 128.27 90.17 90)
-		(unit 1)
-		(exclude_from_sim no)
-		(in_bom yes)
-		(on_board yes)
-		(dnp no)
-		(property "Reference" "RV1"
-			(at 128.27 92.456 90)
-			(effects
-				(font
-					(size 1.27 1.27)
-				)
-			)
-		)
-		(property "Value" "A100K_MASTER_FADER_R"
-			(at 128.27 94.996 90)
-			(effects
-				(font
-					(size 1.27 1.27)
-				)
-			)
-		)
-		(property "Footprint" ""
-			(at 128.27 90.17 0)
-			(effects
-				(font
-					(size 1.27 1.27)
-				)
-				(hide yes)
-			)
-		)
-		(property "Datasheet" "~"
-			(at 128.27 90.17 0)
-			(effects
-				(font
-					(size 1.27 1.27)
-				)
-				(hide yes)
-			)
-		)
-		(property "Description" "Potentiometer"
-			(at 128.27 90.17 0)
-			(effects
-				(font
-					(size 1.27 1.27)
-				)
-				(hide yes)
-			)
-		)
-		(pin "3"
-		)
-		(pin "2"
-		)
-		(pin "1"
-		)
-		(instances
-			(project "mixer"
-				(path "/7887173d-29cc-4936-b1a7-ffeb730ae153/33e847a2-c80a-4a2a-9bd4-e640d7127b7a"
-					(reference "RV1")
-					(unit 1)
 				)
 			)
@@
 	)
 	(symbol
+		(lib_id "Device:R_Potentiometer_Dual_Separate")
+		(at 128.27 90.17 90)
+		(unit 1)
+		(exclude_from_sim no)
+		(in_bom yes)
+		(on_board yes)
+		(dnp no)
+		(fields_autoplaced yes)
+		(property "Reference" "RV7"
+			(at 128.27 93.98 90)
+			(effects
+				(font
+					(size 1.27 1.27)
+				)
+			)
+		)
+		(property "Value" "A100K_MASTER_FADER"
+			(at 128.27 96.52 90)
+			(effects
+				(font
+					(size 1.27 1.27)
+				)
+			)
+		)
+		(property "Footprint" "synth:Potentiometer_Alpha_RD902F-40-00D_Dual_Vertical_CircularHoles"
+			(at 128.27 90.17 0)
+			(effects
+				(font
+					(size 1.27 1.27)
+				)
+				(hide yes)
+			)
+		)
+		(property "Datasheet" "~"
+			(at 128.27 90.17 0)
+			(effects
+				(font
+					(size 1.27 1.27)
+				)
+				(hide yes)
+			)
+		)
+		(property "Description" "Dual potentiometer, separate units"
+			(at 128.27 90.17 0)
+			(effects
+				(font
+					(size 1.27 1.27)
+				)
+				(hide yes)
+			)
+		)
+		(pin "3"
+		)
+		(pin "1"
+		)
+		(pin "6"
+		)
+		(pin "5"
+		)
+		(pin "4"
+		)
+		(pin "2"
+		)
+		(instances
+			(project ""
+				(path "/7887173d-29cc-4936-b1a7-ffeb730ae153/33e847a2-c80a-4a2a-9bd4-e640d7127b7a"
+					(reference "RV7")
+					(unit 1)
+				)
+			)
+		)
+	)
+	(symbol
 		(lib_id "power:GND")
 		(at 114.3 109.22 0)
@@
 					(reference "#PWR04")
 					(unit 1)
+				)
+			)
+		)
+	)
+	(symbol
+		(lib_id "Device:R_Potentiometer_Dual_Separate")
+		(at 128.27 125.73 90)
+		(unit 2)
+		(exclude_from_sim no)
+		(in_bom yes)
+		(on_board yes)
+		(dnp no)
+		(fields_autoplaced yes)
+		(property "Reference" "RV7"
+			(at 128.27 129.54 90)
+			(effects
+				(font
+					(size 1.27 1.27)
+				)
+			)
+		)
+		(property "Value" "A100K_MASTER_FADER"
+			(at 128.27 132.08 90)
+			(effects
+				(font
+					(size 1.27 1.27)
+				)
+			)
+		)
+		(property "Footprint" "synth:Potentiometer_Alpha_RD902F-40-00D_Dual_Vertical_CircularHoles"
+			(at 128.27 125.73 0)
+			(effects
+				(font
+					(size 1.27 1.27)
+				)
+				(hide yes)
+			)
+		)
+		(property "Datasheet" "~"
+			(at 128.27 125.73 0)
+			(effects
+				(font
+					(size 1.27 1.27)
+				)
+				(hide yes)
+			)
+		)
+		(property "Description" "Dual potentiometer, separate units"
+			(at 128.27 125.73 0)
+			(effects
+				(font
+					(size 1.27 1.27)
+				)
+				(hide yes)
+			)
+		)
+		(pin "3"
+		)
+		(pin "1"
+		)
+		(pin "6"
+		)
+		(pin "5"
+		)
+		(pin "4"
+		)
+		(pin "2"
+		)
+		(instances
+			(project ""
+				(path "/7887173d-29cc-4936-b1a7-ffeb730ae153/33e847a2-c80a-4a2a-9bd4-e640d7127b7a"
+					(reference "RV7")
+					(unit 2)
 				)
 			)
@@
 			)
 		)
-		(property "Footprint" "Potentiometer_THT:Potentiometer_Alpha_RD902F-40-00D_Dual_Vertical"
+		(property "Footprint" "synth:Potentiometer_Alpha_RD902F-40-00D_Dual_Vertical_CircularHoles"
 			(at 67.31 85.09 0)
 			(effects

Commit message: 2 channel chain
Parts:
- added C1, C2, C3: 10u, symbol Device:C
- added J1: EURORACK_CONN_16, synth:EURORACK_16_IDC, symbol synth:EURORACK_CONN_16
- added R1: 10k, symbol Device:R
- RV2: renamed from RV7; value A100K_MASTER_FADER -> A100K_MASTER_VOL
- renumbered C1 to C4, J1 to J2, J2 to J3, J3 to J4, J4 to J5, J5 to J6, R1 to R2, R2 to R3, R3 to R4, R4 to R5, RV2 to RV1
Connections:
- net +12V: now also C2.1, J1.9 (12V_P)
- net -12V: now also C3.2, J1.1 (12V_N)
- net AUX_RETURN_L: now also J3.TN
- net GND: now also C1.2, C2.2, C3.1, J1.3 (GND); no longer J3.TN
- new net +5V: C1.1, J1.11 (5V), R1.1
- new net ~{GLOBAL_SOLO}: R1.2
Other:
- note removed: "High end mixers: +10db to -70db"
- note removed: "RA2045F - Alpha 20mm sliders https://www.thonk.co.uk/wp-content/uploads/2019/05/RA_c3_a2_c2_96_c2_a1_c3_a2_c2_96_c2_a145F-2303679.pdf Bourns equiv: PTA2043 PTA2043-20..A.. Digikey: Bourns, largest audio = 100k Mouser: Alphas are all linear, similar bourns selection to digikey Dual-gang are completely unavailable Switch to Dual pot instead of two sliders? May want 30mm instead of 20mm travel - PTA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"
- note removed: "TODO: test both a gain of 10db (100k/3.1 ~=> 33k) and 5-6db (~=> 56k)"
- moved on the sheet: J2, J3, J4, J5, J6, R2, R3, R4, R5, RV1A, RV1B, RV2A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

Commit message: making progress on the outline
Parts:
- C1, C2, C3, C4: footprint (none) -> Capacitor_SMD:C_0603_1608Metric
- R1, R2, R3, R4, R5: footprint (none) -> Resistor_SMD:R_0603_1608Metric
- U1: footprint (none) -> Package_SO:SOIC-14_3.9x8.7mm_P1.27mm
Changed lines of the file:
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@@
 			)
 		)
-		(property "Footprint" ""
+		(property "Footprint" "Resistor_SMD:R_0603_1608Metric"
 			(at 83.312 34.29 90)
 			(effects
@@
 			)
 		)
-		(property "Footprint" ""
+		(property "Footprint" "Capacitor_SMD:C_0603_1608Metric"
 			(at 275.2852 35.56 0)
 			(effects
@@
 			)
 		)
-		(property "Footprint" ""
+		(property "Footprint" "Resistor_SMD:R_0603_1608Metric"
 			(at 152.4 128.778 90)
 			(effects
@@
 			)
 		)
-		(property "Footprint" ""
+		(property "Footprint" "Package_SO:SOIC-14_3.9x8.7mm_P1.27mm"
 			(at 170.18 109.22 0)
 			(effects
@@
 			)
 		)
-		(property "Footprint" ""
+		(property "Footprint" "Capacitor_SMD:C_0603_1608Metric"
 			(at 33.9852 43.18 0)
 			(effects
@@
 			)
 		)
-		(property "Footprint" ""
+		(property "Footprint" "Resistor_SMD:R_0603_1608Metric"
 			(at 152.4 141.478 90)
 			(effects
@@
 			)
 		)
-		(property "Footprint" ""
+		(property "Footprint" "Resistor_SMD:R_0603_1608Metric"
 			(at 152.4 93.218 90)
 			(effects
@@
 			)
 		)
-		(property "Footprint" ""
+		(property "Footprint" "Capacitor_SMD:C_0603_1608Metric"
 			(at 20.0152 31.75 0)
 			(effects
@@
 			)
 		)
-		(property "Footprint" ""
+		(property "Footprint" "Package_SO:SOIC-14_3.9x8.7mm_P1.27mm"
 			(at 130.81 88.9 0)
 			(effects
@@
 			)
 		)
-		(property "Footprint" ""
+		(property "Footprint" "Package_SO:SOIC-14_3.9x8.7mm_P1.27mm"
 			(at 170.18 144.78 0)
 			(effects
@@
 			)
 		)
-		(property "Footprint" ""
+		(property "Footprint" "Resistor_SMD:R_0603_1608Metric"
 			(at 152.4 105.918 90)
 			(effects
@@
 			)
 		)
-		(property "Footprint" ""
+		(property "Footprint" "Package_SO:SOIC-14_3.9x8.7mm_P1.27mm"
 			(at 262.89 29.21 0)
 			(effects
@@
 			)
 		)
-		(property "Footprint" ""
+		(property "Footprint" "Package_SO:SOIC-14_3.9x8.7mm_P1.27mm"
 			(at 134.62 137.16 0)
 			(effects
@@
 			)
 		)
-		(property "Footprint" ""
+		(property "Footprint" "Capacitor_SMD:C_0603_1608Metric"
 			(at 33.9852 31.75 0)
 			(effects

Commit message: layed out parts
Parts:
- removed R4: 33k, Resistor_SMD:R_0603_1608Metric, symbol Device:R
- removed unit 2 of U1
- R3: value 33k -> 100k
- RV1: value A1M - AUX_RETURN_LEVEL -> B100K - AUX_RETURN_LEVEL
Connections:
- net GND: now also U1.3 (+)
- net M_AUX_IN: now also R3.1, U1.2 (-); no longer J2.T
- net M_MIX_IN_L: now also R5.2, RV2.4, U1.9 (-)
- net M_MIX_IN_R: now also R2.2, RV2.1, U1.13 (-); no longer R3.1
- net at RV1.2: now also R5.1; no longer U1.3 (+)
- net at R2.1: now also RV1.5
- new net: J2.T, R3.2, U1.1
Other:
- note added: "100k/33k = max gain 3.03 (9.6db)"
- note added: "100k||33k approximate audio taper"
- moved on the sheet: J2, J3, J4, RV1A, RV1B

Commit message: rework master board for space and symmetry
Connections:
- net AUX_RETURN_L: now also RV1.6; no longer RV1.3
- net AUX_RETURN_R: now also RV1.3; no longer RV1.6
- net at RV1.2: now also R2.1; no longer R5.1
- net at RV1.5: now also R5.1; no longer R2.1
Other:
- moved on the sheet: RV1A, RV1B
Changed lines of the file:
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@@
 	(symbol
 		(lib_id "Device:R_Potentiometer_Dual_Separate")
-		(at 135.89 139.7 0)
+		(at 130.81 91.44 0)
 		(mirror x)
 		(unit 1)
@@
 		(dnp no)
 		(property "Reference" "RV1"
-			(at 133.35 140.9701 0)
+			(at 128.27 92.7101 0)
 			(effects
 				(font
@@
 		)
 		(property "Value" "B100K - AUX_RETURN_LEVEL"
-			(at 133.35 138.4301 0)
+			(at 128.27 90.1701 0)
 			(effects
 				(font
@@
 		)
 		(property "Footprint" "synth:Potentiometer_Alpha_RD902F-40-00D_Dual_Vertical_CircularHoles"
-			(at 135.89 139.7 0)
+			(at 130.81 91.44 0)
 			(effects
 				(font
@@
 		)
 		(property "Datasheet" "~"
-			(at 135.89 139.7 0)
+			(at 130.81 91.44 0)
 			(effects
 				(font
@@
 		)
 		(property "Description" "Dual potentiometer, separate units"
-			(at 135.89 139.7 0)
+			(at 130.81 91.44 0)
 			(effects
 				(font
@@
 	(symbol
 		(lib_id "Device:R_Potentiometer_Dual_Separate")
-		(at 130.81 91.44 0)
+		(at 135.89 139.7 0)
 		(mirror x)
 		(unit 2)
@@
 		(dnp no)
 		(property "Reference" "RV1"
-			(at 128.27 92.7101 0)
+			(at 133.35 140.9701 0)
 			(effects
 				(font
@@
 		)
 		(property "Value" "B100K - AUX_RETURN_LEVEL"
-			(at 128.27 90.1701 0)
+			(at 133.35 138.4301 0)
 			(effects
 				(font
@@
 		)
 		(property "Footprint" "synth:Potentiometer_Alpha_RD902F-40-00D_Dual_Vertical_CircularHoles"
-			(at 130.81 91.44 0)
+			(at 135.89 139.7 0)
 			(effects
 				(font
@@
 		)
 		(property "Datasheet" "~"
-			(at 130.81 91.44 0)
+			(at 135.89 139.7 0)
 			(effects
 				(font
@@
 		)
 		(property "Description" "Dual potentiometer, separate units"
-			(at 130.81 91.44 0)
-			(effects
-				(font
+			(at 135.89 139.7 0)
+			(effects
+				(font

Commit message: panel design
Connections:
- net AUX_RETURN_L: no longer J3.TN
- net AUX_RETURN_R: now also J4.TN
- net GND: now also J3.TN; no longer J4.TN
Changed lines of the file:
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@@
-	)
-	(junction
-		(at 116.84 130.81)
-		(diameter 0)
-		(color 0 0 0 0)
 	)
 	(junction
@@
 	)
 	(junction
+		(at 118.11 82.55)
+		(diameter 0)
+		(color 0 0 0 0)
+	)
+	(junction
 		(at 161.29 104.14)
 		(diameter 0)
@@
 	(wire
 		(pts
-			(xy 105.41 133.35) (xy 107.95 133.35)
+			(xy 105.41 133.35) (xy 118.11 133.35)
 		)
 		(stroke
@@
 	(wire
 		(pts
-			(xy 116.84 130.81) (xy 135.89 130.81)
+			(xy 105.41 82.55) (xy 118.11 82.55)
 		)
 		(stroke
@@
 	(wire
 		(pts
-			(xy 105.41 85.09) (xy 116.84 85.09)
-		)
-		(stroke
-			(width 0)
-			(type default)
-		)
-	)
-	(wire
-		(pts
 			(xy 33.02 20.32) (xy 33.02 24.13)
 		)
@@
 	(wire
 		(pts
+			(xy 118.11 133.35) (xy 118.11 82.55)
+		)
+		(stroke
+			(width 0)
+			(type default)
+		)
+	)
+	(wire
+		(pts
 			(xy 179.07 125.73) (xy 179.07 129.54)
 		)
@@
 	(wire
 		(pts
-			(xy 105.41 130.81) (xy 116.84 130.81)
+			(xy 105.41 85.09) (xy 107.95 85.09)
+		)
+		(stroke
+			(width 0)
+			(type default)
+		)
+	)
+	(wire
+		(pts
+			(xy 105.41 130.81) (xy 135.89 130.81)
 		)
 		(stroke
@@
 	(wire
 		(pts
-			(xy 116.84 85.09) (xy 116.84 130.81)
+			(xy 118.11 82.55) (xy 130.81 82.55)
 		)
 		(stroke
@@
 		(pts
 			(xy 179.07 129.54) (xy 181.61 129.54)
-		)
-		(stroke
-			(width 0)
-			(type default)
-		)
-	)
-	(wire
-		(pts
-			(xy 105.41 82.55) (xy 130.81 82.55)
 		)
 		(stroke
@@
 	(symbol
 		(lib_id "power:GND")
-		(at 107.95 133.35 90)
+		(at 107.95 85.09 90)
 		(unit 1)
 		(exclude_from_sim no)
@@
 		(fields_autoplaced yes)
 		(property "Reference" "#PWR020"
-			(at 114.3 133.35 0)
+			(at 114.3 85.09 0)
 			(effects
 				(font
@@
 		)
 		(property "Value" "GND"
-			(at 111.76 133.3499 90)
+			(at 111.76 85.0899 90)
 			(effects
 				(font
@@
 		)
 		(property "Footprint" ""
-			(at 107.95 133.35 0)
+			(at 107.95 85.09 0)
 			(effects
 				(font
@@
 		)
 		(property "Datasheet" ""
-			(at 107.95 133.35 0)
+			(at 107.95 85.09 0)
 			(effects
 				(font
@@
 		)
 		(property "Description" "Power symbol creates a global label with name \"GND\" , ground"
-			(at 107.95 133.35 0)
-			(effects
-				(font
+			(at 107.95 85.09 0)
+			(effects
+				(font
