File: mixer/mixer.kicad_sch (KiCad schematic)
At the start: 5 parts, among them J6 EURORACK_CONN_16

Commit message: 2 channel chain
Parts:
- removed C2, C3, C4: 10u, symbol Device:C
- removed J6: EURORACK_CONN_16, synth:EURORACK_16_IDC, symbol synth:EURORACK_CONN_16
- removed R16: 10k, symbol Device:R
Other:
- removed sheet Channel
- added sheet Channel Module (channels.kicad_sch)
- sheet Master Module ports: added M_AUX_IN, M_MIX_IN_L, M_MIX_IN_R, ~{GLOBAL_SOLO}; removed none
- note added: "High end mixers: +10db to -70db"
- note added: "N of these units can be dasy chained together"
- note added: "RA2045F - Alpha 20mm sliders https://www.thonk.co.uk/wp-content/uploads/2019/05/RA_c3_a2_c2_96_c2_a1_c3_a2_c2_96_c2_a145F-2303679.pdf Bourns equiv: PTA2043 PTA2043-20..A.. Digikey: Bourns, largest audio = 100k Mouser: Alphas are all linear, similar bourns selection to digikey Dual-gang are completely unavailable Switch to Dual pot instead of two sliders? May want 30mm instead of 20mm travel - PTA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"
- note added: "TODO: test both a gain of 10db (100k/3.1 ~=> 33k) and 5-6db (~=> 56k)"

Commit message: making progress on the outline
Parts:
- added J10: C_BOARD_IN_1, Connector_PinSocket_2.54mm:PinSocket_2x04_P2.54mm_Horizontal, symbol Connector_Generic:Conn_01x08
- added J11: C_BOARD_IN_2, Connector_PinSocket_2.54mm:PinSocket_2x04_P2.54mm_Horizontal, symbol Connector_Generic:Conn_01x08
- added J12: M_BOARD_IN_1, Connector_PinSocket_2.54mm:PinSocket_2x04_P2.54mm_Horizontal, symbol Connector_Generic:Conn_01x08
- added J13: M_BOARD_IN_2, Connector_PinSocket_2.54mm:PinSocket_2x04_P2.54mm_Horizontal, symbol Connector_Generic:Conn_01x08
- added J14: C_BOARD_OUT_1, Connector_PinHeader_2.54mm:PinHeader_2x04_P2.54mm_Horizontal, symbol Connector_Generic:Conn_01x08
- added J15: C_BOARD_OUT_2, Connector_PinHeader_2.54mm:PinHeader_2x04_P2.54mm_Horizontal, symbol Connector_Generic:Conn_01x08
Connections:
- net +12V: now also J11.1 (Pin_1), J11.2 (Pin_2), J13.1 (Pin_1), J13.2 (Pin_2), J15.1 (Pin_1), J15.2 (Pin_2)
- net +5V: now also J11.3 (Pin_3), J11.4 (Pin_4), J13.3 (Pin_3), J13.4 (Pin_4), J15.3 (Pin_3), J15.4 (Pin_4)
- net -12V: now also J11.7 (Pin_7), J11.8 (Pin_8), J13.7 (Pin_7), J13.8 (Pin_8), J15.7 (Pin_7), J15.8 (Pin_8)
- net Channel Module/C_AUX_IN: now also J10.5 (Pin_5), J10.6 (Pin_6)
- net Channel Module/C_AUX_OUT: now also J14.5 (Pin_5), J14.6 (Pin_6)
- net Channel Module/C_MIX_IN_L: now also J10.3 (Pin_3), J10.4 (Pin_4)
- net Channel Module/C_MIX_IN_R: now also J10.1 (Pin_1), J10.2 (Pin_2)
- net Channel Module/C_OUT_L: now also J14.3 (Pin_3), J14.4 (Pin_4)
- net Channel Module/C_OUT_R: now also J14.1 (Pin_1), J14.2 (Pin_2)
- net Channel Module/~{GLOBAL_SOLO}: now also J10.7 (Pin_7), J10.8 (Pin_8), J14.7 (Pin_7), J14.8 (Pin_8)
- net GND: now also J11.5 (Pin_5), J11.6 (Pin_6), J13.5 (Pin_5), J13.6 (Pin_6), J15.5 (Pin_5), J15.6 (Pin_6)
- net Master Module/M_AUX_IN: now also J12.5 (Pin_5), J12.6 (Pin_6)
- net Master Module/M_MIX_IN_L: now also J12.3 (Pin_3), J12.4 (Pin_4)
- net Master Module/M_MIX_IN_R: now also J12.1 (Pin_1), J12.2 (Pin_2)
- net Master Module/~{GLOBAL_SOLO}: now also J12.7 (Pin_7), J12.8 (Pin_8)

Commit message: layed out parts
Parts:
- removed J15: C_BOARD_OUT_2, Connector_PinHeader_2.54mm:PinHeader_2x04_P2.54mm_Horizontal, symbol Connector_Generic:Conn_01x08
- J10: value C_BOARD_IN_1 -> C_BOARD_IN; footprint Connector_PinSocket_2.54mm:PinSocket_2x04_P2.54mm_Horizontal -> Connector_PinHeader_1.27mm:PinHeader_1x08_P1.27mm_Vertical
- J11: value C_BOARD_IN_2 -> INTERCONNECT1; footprint Connector_PinSocket_2.54mm:PinSocket_2x04_P2.54mm_Horizontal -> Connector_PinHeader_1.27mm:PinHeader_1x08_P1.27mm_Vertical
- J12: value M_BOARD_IN_1 -> M_BOARD_IN; footprint Connector_PinSocket_2.54mm:PinSocket_2x04_P2.54mm_Horizontal -> Connector_PinSocket_1.27mm:PinSocket_1x08_P1.27mm_Vertical
- J13: value M_BOARD_IN_2 -> INTERCONNECT2; footprint Connector_PinSocket_2.54mm:PinSocket_2x04_P2.54mm_Horizontal -> Connector_PinHeader_1.27mm:PinHeader_1x08_P1.27mm_Vertical
- J14: value C_BOARD_OUT_1 -> C_BOARD_OUT; footprint Connector_PinHeader_2.54mm:PinHeader_2x04_P2.54mm_Horizontal -> Connector_PinSocket_1.27mm:PinSocket_1x08_P1.27mm_Vertical
Connections:
- net +12V: now also J10.4 (Pin_4), J12.4 (Pin_4), J14.4 (Pin_4); no longer J11.1 (Pin_1), J11.2 (Pin_2), J13.1 (Pin_1), J13.2 (Pin_2)
- net +5V: now also J10.3 (Pin_3), J12.3 (Pin_3), J14.3 (Pin_3); no longer J11.3 (Pin_3), J11.4 (Pin_4), J13.3 (Pin_3), J13.4 (Pin_4)
- net -12V: now also J10.1 (Pin_1), J12.1 (Pin_1), J14.1 (Pin_1); no longer J11.7 (Pin_7), J11.8 (Pin_8), J13.7 (Pin_7), J13.8 (Pin_8)
- net Channel Module/~{GLOBAL_SOLO}: now also J10.5 (Pin_5), J14.5 (Pin_5); no longer J10.7 (Pin_7), J10.8 (Pin_8), J14.7 (Pin_7), J14.8 (Pin_8)
- net GND: now also J10.2 (Pin_2), J12.2 (Pin_2), J14.2 (Pin_2); no longer J11.5 (Pin_5), J11.6 (Pin_6), J13.5 (Pin_5), J13.6 (Pin_6)
- net Master Module/M_AUX_IN: no longer J12.5 (Pin_5)
- net Master Module/M_MIX_IN_L: now also J12.7 (Pin_7); no longer J12.3 (Pin_3), J12.4 (Pin_4)
- net Master Module/M_MIX_IN_R: now also J12.8 (Pin_8); no longer J12.1 (Pin_1), J12.2 (Pin_2)
- net Master Module/~{GLOBAL_SOLO}: now also J12.5 (Pin_5); no longer J12.7 (Pin_7), J12.8 (Pin_8)
- net Channel Module/C_AUX_IN renamed Channel Module/C_BUS_AUX
- net Channel Module/C_BUS_AUX: now also J14.6 (Pin_6); no longer J10.5 (Pin_5)
- removed net Channel Module/C_AUX_OUT: J14.5 (Pin_5), J14.6 (Pin_6)
- removed net Channel Module/C_MIX_IN_L: J10.3 (Pin_3), J10.4 (Pin_4)
- removed net Channel Module/C_MIX_IN_R: J10.1 (Pin_1), J10.2 (Pin_2)
- removed net Channel Module/C_OUT_L: J14.3 (Pin_3), J14.4 (Pin_4)
- removed net Channel Module/C_OUT_R: J14.1 (Pin_1), J14.2 (Pin_2)
- new net: J11.1 (Pin_1), J13.1 (Pin_1)
- new net: J11.2 (Pin_2), J13.2 (Pin_2)
- new net: J11.3 (Pin_3), J13.3 (Pin_3)
- new net: J11.4 (Pin_4), J13.4 (Pin_4)
- new net: J11.5 (Pin_5), J13.5 (Pin_5)
- new net: J11.6 (Pin_6), J13.6 (Pin_6)
- new net: J11.7 (Pin_7), J13.7 (Pin_7)
- new net: J11.8 (Pin_8), J13.8 (Pin_8)
- new net Channel Module/C_BUS_L: J10.7 (Pin_7), J14.7 (Pin_7)
- new net Channel Module/C_BUS_R: J10.8 (Pin_8), J14.8 (Pin_8)
Other:
- sheet Channel Module ports: added C_BUS_AUX, C_BUS_L, C_BUS_R; removed C_AUX_IN, C_AUX_OUT, C_MIX_IN_L, C_MIX_IN_R, C_OUT_L, C_OUT_R
- moved on the sheet: J10, J12, J14

Commit message: layout master board
Parts:
- J10: footprint Connector_PinHeader_1.27mm:PinHeader_1x08_P1.27mm_Vertical -> Connector_PinSocket_1.27mm:PinSocket_1x08_P1.27mm_Vertical
Changed lines of the file:
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@@
 			)
 		)
-		(property "Footprint" "Connector_PinHeader_1.27mm:PinHeader_1x08_P1.27mm_Vertical"
+		(property "Footprint" "Connector_PinSocket_1.27mm:PinSocket_1x08_P1.27mm_Vertical"
 			(at 72.39 72.39 0)
 			(effects

Commit message: start on panel
Other:
- added sheet Panel (panel.kicad_sch)
Changed lines of the file:
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@@
+		)
+	)
+	(sheet
+		(at 218.44 132.08)
+		(size 52.07 27.94)
+		(exclude_from_sim no)
+		(in_bom yes)
+		(on_board yes)
+		(dnp no)
+		(fields_autoplaced yes)
+		(stroke
+			(width 0.1524)
+			(type solid)
+		)
+		(fill
+			(color 0 0 0 0.0000)
+		)
+		(property "Sheetname" "Panel"
+			(at 218.44 131.3684 0)
+			(effects
+				(font
+					(size 1.27 1.27)
+				)
+				(justify left bottom)
+			)
+		)
+		(property "Sheetfile" "panel.kicad_sch"
+			(at 218.44 160.6046 0)
+			(effects
+				(font
+					(size 1.27 1.27)
+				)
+				(justify left top)
+			)
+		)
+		(instances
+			(project "mixer"
+				(path "/7887173d-29cc-4936-b1a7-ffeb730ae153"
+					(page "6")
+				)
+			)
 		)
 	)

Commit message: cleanup 3
Other:
- note removed: "TODO: test both a gain of 10db (100k/3.1 ~=> 33k) and 5-6db (~=> 56k)"
- moved on the sheet: J11, J13
Changed lines of the file:
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@@
-		)
-	)
-	(text "TODO: test both a gain of 10db (100k/3.1 ~=> 33k) and 5-6db (~=> 56k)"
-		(exclude_from_sim no)
-		(at 78.486 139.954 0)
-		(effects
-			(font
-				(size 1.27 1.27)
-			)
 		)
 	)
@@
 	(text "N of these units can be dasy chained together"
 		(exclude_from_sim no)
-		(at 114.3 50.038 0)
+		(at 42.672 71.628 0)
 		(effects
 			(font
@@
 	(wire
 		(pts
-			(xy 153.67 24.13) (xy 156.21 24.13)
+			(xy 156.21 40.64) (xy 158.75 40.64)
 		)
 		(stroke
@@
 	(wire
 		(pts
-			(xy 153.67 31.75) (xy 156.21 31.75)
+			(xy 156.21 48.26) (xy 158.75 48.26)
 		)
 		(stroke
@@
 	(wire
 		(pts
-			(xy 153.67 29.21) (xy 156.21 29.21)
+			(xy 156.21 45.72) (xy 158.75 45.72)
 		)
 		(stroke
@@
 	(wire
 		(pts
-			(xy 153.67 36.83) (xy 156.21 36.83)
+			(xy 156.21 53.34) (xy 158.75 53.34)
 		)
 		(stroke
@@
 	(wire
 		(pts
-			(xy 153.67 26.67) (xy 156.21 26.67)
+			(xy 156.21 43.18) (xy 158.75 43.18)
 		)
 		(stroke
@@
 	(wire
 		(pts
-			(xy 153.67 21.59) (xy 156.21 21.59)
+			(xy 156.21 38.1) (xy 158.75 38.1)
 		)
 		(stroke
@@
 	(wire
 		(pts
-			(xy 153.67 34.29) (xy 156.21 34.29)
+			(xy 156.21 50.8) (xy 158.75 50.8)
 		)
 		(stroke
@@
 	(wire
 		(pts
-			(xy 153.67 19.05) (xy 156.21 19.05)
+			(xy 156.21 35.56) (xy 158.75 35.56)
 		)
 		(stroke
@@
 		(dnp no)
 		(property "Reference" "J14"
-			(at 156.718 69.342 90)
+			(at 155.956 69.342 90)
 			(effects
 				(font
@@
 		)
 		(property "Value" "C_BOARD_OUT"
-			(at 154.178 69.342 90)
+			(at 153.67 65.278 90)
 			(effects
 				(font
@@
 		(dnp no)
 		(property "Reference" "J12"
-			(at 158.242 69.342 90)
+			(at 159.512 69.596 90)
 			(effects
 				(font
@@
 		)
 		(property "Value" "M_BOARD_IN"
-			(at 160.782 69.342 90)
+			(at 161.036 65.278 90)
 			(effects
 				(font
@@
 		(dnp no)
 		(property "Reference" "J10"
-			(at 66.802 69.342 90)
+			(at 67.818 69.342 90)
 			(effects
 				(font
@@
 		)
 		(property "Value" "C_BOARD_IN"
-			(at 69.342 69.342 90)
+			(at 69.596 65.278 90)
 			(effects
 				(font
@@
 	(symbol
 		(lib_id "Connector_Generic:Conn_01x08")
-		(at 148.59 29.21 180)
+		(at 151.13 45.72 180)
 		(unit 1)
 		(exclude_from_sim no)
@@
 		(dnp no)
 		(property "Reference" "J11"
-			(at 143.002 26.162 90)
+			(at 145.542 42.672 90)
 			(effects
 				(font
@@
 		)
 		(property "Value" "INTERCONNECT1"
-			(at 145.288 22.352 90)
+			(at 147.828 38.862 90)
 			(effects
 				(font
@@
 		)
 		(property "Footprint" "Connector_PinHeader_1.27mm:PinHeader_1x08_P1.27mm_Vertical"
-			(at 148.59 29.21 0)
+			(at 151.13 45.72 0)
 			(effects
 				(font
@@
 		)
 		(property "Datasheet" "~"
-			(at 148.59 29.21 0)
+			(at 151.13 45.72 0)
 			(effects
 				(font
@@
 		)
 		(property "Description" "Generic connector, single row, 01x08, script generated (kicad-library-utils/schlib/autogen/connector/)"
-			(at 148.59 29.21 0)
+			(at 151.13 45.72 0)
 			(effects
 				(font
@@
 	(symbol
 		(lib_id "Connector_Generic:Conn_01x08")
-		(at 161.29 29.21 0)
+		(at 163.83 45.72 0)
 		(mirror x)
 		(unit 1)
@@
 		(dnp no)
 		(property "Reference" "J13"
-			(at 166.878 26.162 90)
+			(at 169.418 42.672 90)
 			(effects
 				(font
@@
 		)
 		(property "Value" "INTERCONNECT2"
-			(at 164.338 26.162 90)
+			(at 166.624 36.83 90)
 			(effects
 				(font
@@
 		)
 		(property "Footprint" "Connector_PinHeader_1.27mm:PinHeader_1x08_P1.27mm_Vertical"
-			(at 161.29 29.21 0)
+			(at 163.83 45.72 0)
 			(effects
 				(font
@@
 		)
 		(property "Datasheet" "~"
-			(at 161.29 29.21 0)
+			(at 163.83 45.72 0)
 			(effects
 				(font
@@
 		)
 		(property "Description" "Generic connector, single row, 01x08, script generated (kicad-library-utils/schlib/autogen/connector/)"
-			(at 161.29 29.21 0)
-			(effects
-				(font
+			(at 163.83 45.72 0)
+			(effects
+				(font
