File: mixer/panel.kicad_sch (KiCad schematic)
At the start: 21 parts, among them J15 C_IN1, J16 C_IN2, J17 C_AUXSEND1, J18 C_PAN1, J19 C_AUXSEND2, J20 C_PAN2, J21 M_OUT_L, J22 M_AUXSEND, J23 M_AUX_AMOUNT, J24 M_OUT_R, J25 M_AUX_RETURN_L, J26 M_AUX_RETURN_L, J27 M_MASTER

Commit message: place screws
Parts:
- added FID1: C_SCREW_B, synth:eurorack_screw_hole, symbol synth:PanelItem
- added FID2: C_SCREW_T, synth:eurorack_screw_hole, symbol synth:PanelItem
- added FID3: M_SCREW_T, synth:eurorack_screw_hole, symbol synth:PanelItem
- added FID4: M_SCREW_B, synth:eurorack_screw_hole, symbol synth:PanelItem
Connections:
- net GND: now also FID1.1, FID2.1, FID3.1, FID4.1

Commit message: update graphics
Parts:
- FID10, FID12: footprint _project:MUTE_CUTOUT -> _project:MUTE_CUTOUT_ALT
- FID11, FID9: footprint _project:SOLO_CUTOUT -> _project:SOLO_CUTOUT_ALT
Changed lines of the file:
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@@
 			)
 		)
-		(property "Footprint" "_project:MUTE_CUTOUT"
+		(property "Footprint" "_project:MUTE_CUTOUT_ALT"
 			(at 44.45 148.59 0)
 			(effects
@@
 			)
 		)
-		(property "Footprint" "_project:MUTE_CUTOUT"
+		(property "Footprint" "_project:MUTE_CUTOUT_ALT"
 			(at 63.5 148.59 0)
 			(effects
@@
 			)
 		)
-		(property "Footprint" "_project:SOLO_CUTOUT"
+		(property "Footprint" "_project:SOLO_CUTOUT_ALT"
 			(at 44.45 140.97 0)
 			(effects
@@
 			)
 		)
-		(property "Footprint" "_project:SOLO_CUTOUT"
+		(property "Footprint" "_project:SOLO_CUTOUT_ALT"
 			(at 63.5 140.97 0)
 			(effects

Commit message: cleanup 3
Parts:
- FID10, FID12: footprint _project:MUTE_CUTOUT_ALT -> _project:MUTE_CUTOUT
- FID11, FID9: footprint _project:SOLO_CUTOUT_ALT -> _project:SOLO_CUTOUT
Changed lines of the file:
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@@
 			)
 		)
-		(property "Footprint" "_project:MUTE_CUTOUT_ALT"
+		(property "Footprint" "_project:MUTE_CUTOUT"
 			(at 44.45 148.59 0)
 			(effects
@@
 			)
 		)
-		(property "Footprint" "_project:MUTE_CUTOUT_ALT"
+		(property "Footprint" "_project:MUTE_CUTOUT"
 			(at 63.5 148.59 0)
 			(effects
@@
 			)
 		)
-		(property "Footprint" "_project:SOLO_CUTOUT_ALT"
+		(property "Footprint" "_project:SOLO_CUTOUT"
 			(at 44.45 140.97 0)
 			(effects
@@
 			)
 		)
-		(property "Footprint" "_project:SOLO_CUTOUT_ALT"
+		(property "Footprint" "_project:SOLO_CUTOUT"
 			(at 63.5 140.97 0)
 			(effects
